Commit message: add dual_xarm_moveit control

File: xarm_description/urdf/xarm5/xarm5.ros2_control.xacro (robot description, xacro)
@@ -13,5 +13,5 @@
       <hardware>
         <plugin>${ros2_control_plugin}</plugin>
-        <param name="hw_ns">${hw_ns}</param>
+        <param name="hw_ns">${prefix}${hw_ns}</param>
       </hardware>
       <joint name="${prefix}joint1">

File: xarm_description/urdf/xarm5/xarm5.urdf.xacro (robot description, xacro)
@@ -7,14 +7,14 @@
     joint4_lower_limit:=${-1.69297}  joint4_upper_limit:=${pi}
     joint5_lower_limit:=${-2.0*pi}  joint5_upper_limit:=${2.0*pi}">
-    <material name="Black">
+    <material name="${prefix}Black">
       <color rgba="0.0 0.0 0.0 1.0"/>
     </material>
-    <material name="Red">
+    <material name="${prefix}Red">
       <color rgba="0.8 0.0 0.0 1.0"/>
     </material>
-    <material name="White">
+    <material name="${prefix}White">
       <color rgba="1.0 1.0 1.0 1.0"/>
     </material>
-    <material name="Silver">
+    <material name="${prefix}Silver">
       <color rgba="0.753 0.753 0.753 1.0"/>
     </material>
@@ -43,5 +43,5 @@
             filename="package://xarm_description/meshes/xarm5/visual/base_link.STL" />
         </geometry>
-        <material name="White" />
+        <material name="${prefix}White" />
       </visual>
       <collision>
@@ -79,5 +79,5 @@
             filename="package://xarm_description/meshes/xarm5/visual/link1.STL" />
         </geometry>
-        <material name="White" />
+        <material name="${prefix}White" />
       </visual>
       <collision>
@@ -136,5 +136,5 @@
             filename="package://xarm_description/meshes/xarm5/visual/link2.STL" />
         </geometry>
-        <material name="White" />
+        <material name="${prefix}White" />
       </visual>
       <collision>
@@ -193,5 +193,5 @@
             filename="package://xarm_description/meshes/xarm5/visual/link3.STL" />
         </geometry>
-        <material name="White" />
+        <material name="${prefix}White" />
       </visual>
       <collision>
@@ -250,5 +250,5 @@
             filename="package://xarm_description/meshes/xarm5/visual/link4.STL" />
         </geometry>
-        <material name="White" />
+        <material name="${prefix}White" />
       </visual>
       <collision>
@@ -307,5 +307,5 @@
             filename="package://xarm_description/meshes/xarm5/visual/link5.STL" />
         </geometry>
-        <material name="Silver" />
+        <material name="${prefix}Silver" />
       </visual>
       <collision>

File: xarm_description/urdf/xarm5/xarm5_robot_macro.xacro (robot description, xacro)
@@ -18,5 +18,5 @@
       <link name="world" />
     </xacro:if>
-    <joint name="world_joint" type="fixed">
+    <joint name="${prefix}world_joint" type="fixed">
       <parent link="${attach_to}" />
       <child link = "${prefix}link_base" />

File: xarm_description/urdf/xarm6/xarm6.ros2_control.xacro (robot description, xacro)
@@ -14,5 +14,5 @@
       <hardware>
         <plugin>${ros2_control_plugin}</plugin>
-        <param name="hw_ns">${hw_ns}</param>
+        <param name="hw_ns">${prefix}${hw_ns}</param>
         <!-- fake -->
         <!-- <plugin>fake_components/GenericSystem</plugin> -->

File: xarm_description/urdf/xarm7/xarm7.ros2_control.xacro (robot description, xacro)
@@ -15,5 +15,5 @@
       <hardware>
         <plugin>${ros2_control_plugin}</plugin>
-        <param name="hw_ns">${hw_ns}</param>
+        <param name="hw_ns">${prefix}${hw_ns}</param>
       </hardware>
       <joint name="${prefix}joint1">

File: xarm_description/urdf/xarm7/xarm7.urdf.xacro (robot description, xacro)
@@ -9,14 +9,14 @@
     joint6_lower_limit:=${-1.69297}  joint6_upper_limit:=${pi}
     joint7_lower_limit:=${-2.0*pi}  joint7_upper_limit:=${2.0*pi}">
-    <material name="Black">
+    <material name="${prefix}Black">
       <color rgba="0.0 0.0 0.0 1.0"/>
     </material>
-    <material name="Red">
+    <material name="${prefix}Red">
       <color rgba="0.8 0.0 0.0 1.0"/>
     </material>
-    <material name="White">
+    <material name="${prefix}White">
       <color rgba="1.0 1.0 1.0 1.0"/>
     </material>
-    <material name="Silver">
+    <material name="${prefix}Silver">
       <color rgba="0.753 0.753 0.753 1.0"/>
     </material>
@@ -45,5 +45,5 @@
           filename="package://xarm_description/meshes/xarm7/visual/link_base.STL" />
       </geometry>
-      <material name="White" />
+      <material name="${prefix}White" />
     </visual>
     <collision>
@@ -81,5 +81,5 @@
           filename="package://xarm_description/meshes/xarm7/visual/link1.STL" />
       </geometry>
-      <material name="White" />
+      <material name="${prefix}White" />
     </visual>
     <collision>
@@ -138,5 +138,5 @@
           filename="package://xarm_description/meshes/xarm7/visual/link2.STL" />
       </geometry>
-      <material name="White" />
+      <material name="${prefix}White" />
     </visual>
     <collision>
@@ -195,5 +195,5 @@
           filename="package://xarm_description/meshes/xarm7/visual/link3.STL" />
       </geometry>
-      <material name="White" />
+      <material name="${prefix}White" />
     </visual>
     <collision>
@@ -252,5 +252,5 @@
           filename="package://xarm_description/meshes/xarm7/visual/link4.STL" />
       </geometry>
-      <material name="White" />
+      <material name="${prefix}White" />
     </visual>
     <collision>
@@ -309,5 +309,5 @@
           filename="package://xarm_description/meshes/xarm7/visual/link5.STL" />
       </geometry>
-      <material name="White" />
+      <material name="${prefix}White" />
     </visual>
     <collision>
@@ -366,5 +366,5 @@
           filename="package://xarm_description/meshes/xarm7/visual/link6.STL" />
       </geometry>
-      <material name="White" />
+      <material name="${prefix}White" />
     </visual>
     <collision>
@@ -423,5 +423,5 @@
           filename="package://xarm_description/meshes/xarm7/visual/link7.STL" />
       </geometry>
-      <material name="Silver" />
+      <material name="${prefix}Silver" />
     </visual>
     <collision>

File: xarm_description/urdf/xarm_device_macro.xacro (robot description, xacro)
@@ -2,10 +2,12 @@
 <robot xmlns:xacro="http://ros.org/wiki/xacro" name="xarm_device">
   <xacro:macro name="xarm_device" params="prefix:='' namespace:='xarm' limited:='false' effort_control:='false'
-    velocity_control:='false' add_gripper:='false' add_vacuum_gripper:='false' dof:=7 ros2_control_plugin:='xarm_control/XArmHW' ">
+    velocity_control:='false' add_gripper:='false' add_vacuum_gripper:='false' dof:=7 ros2_control_plugin:='xarm_control/XArmHW'
+    attach_to:='world' xyz:='0 0 0' rpy:='0 0 0' ">
     <xacro:if value="${dof == 5}">
       <xacro:include filename="$(find xarm_description)/urdf/xarm5/xarm5_robot_macro.xacro" />
       <xacro:xarm5_robot prefix="${prefix}" namespace="${namespace}" limited="${limited}"
         effort_control="${effort_control}" velocity_control="${velocity_control}"
-        ros2_control_plugin="${ros2_control_plugin}" />
+        ros2_control_plugin="${ros2_control_plugin}"
+        attach_to="${attach_to}" xyz="${xyz}" rpy="${rpy}" />
     </xacro:if>
     <xacro:if value="${dof == 6}">
@@ -13,5 +15,6 @@
       <xacro:xarm6_robot prefix="${prefix}" namespace="${namespace}" limited="${limited}"
         effort_control="${effort_control}" velocity_control="${velocity_control}"
-        ros2_control_plugin="${ros2_control_plugin}" />
+        ros2_control_plugin="${ros2_control_plugin}"
+        attach_to="${attach_to}" xyz="${xyz}" rpy="${rpy}" />
     </xacro:if>
     <xacro:unless value="${dof == 5 or dof == 6}">
@@ -19,13 +22,14 @@
       <xacro:xarm7_robot prefix="${prefix}" namespace="${namespace}" limited="${limited}"
         effort_control="${effort_control}" velocity_control="${velocity_control}"
-        ros2_control_plugin="${ros2_control_plugin}" />
+        ros2_control_plugin="${ros2_control_plugin}"
+        attach_to="${attach_to}" xyz="${xyz}" rpy="${rpy}" />
     </xacro:unless>
     <xacro:if value="${add_gripper}">
       <xacro:include filename="$(find xarm_description)/urdf/gripper/xarm_gripper_model.xacro" />
-      <xacro:load_gripper attach_to="${prefix}link_eef" effort_control="${effort_control}" velocity_control="${velocity_control}" />
+      <xacro:load_gripper prefix="${prefix}" attach_to="${prefix}link_eef" effort_control="${effort_control}" velocity_control="${velocity_control}" />
     </xacro:if>
     <xacro:if value="${add_vacuum_gripper}">
       <xacro:include filename="$(find xarm_description)/urdf/vacuum_gripper/xarm_vacuum_gripper.urdf.xacro" />
-      <xacro:xarm_vacuum_gripper_urdf attach_to="${prefix}link_eef" effort_control="${effort_control}" velocity_control="${velocity_control}" />
+      <xacro:xarm_vacuum_gripper_urdf prefix="${prefix}" attach_to="${prefix}link_eef" effort_control="${effort_control}" velocity_control="${velocity_control}" />
     </xacro:if>
   </xacro:macro>
