Commit message: remove moveit_fake_controller

File: xarm_description/urdf/gripper/xarm_gripper_model.xacro (robot description, xacro)
@@ -5,10 +5,12 @@
   <xacro:include filename="$(find xarm_description)/urdf/common/common.gazebo.xacro" />
   <!-- xarm_gripper -->
+  <xacro:include filename="$(find xarm_description)/urdf/gripper/xarm_gripper.ros2_control.xacro" />
   <xacro:include filename="$(find xarm_description)/urdf/gripper/xarm_gripper.urdf.xacro" />
   <xacro:include filename="$(find xarm_description)/urdf/gripper/xarm_gripper.transmission.xacro" />
   <xacro:include filename="$(find xarm_description)/urdf/gripper/xarm_gripper.gazebo.xacro" />
-  <xacro:macro name="load_gripper" params="prefix:='' attach_to:='' ns:='xarm' xyz:='0 0 0' rpy:='0 0 0' effort_control:='false' velocity_control:='false' ">
+  <xacro:macro name="load_gripper" params="prefix:='' attach_to:='' ns:='xarm' xyz:='0 0 0' rpy:='0 0 0' effort_control:='false' velocity_control:='false' ros2_control_plugin:='xarm_control/FakeXArmHW' ">
     <!-- gazebo plugin -->
     <!-- <xacro:gazebo_ros_control_plugin namespace="${ns}"/> -->
+    <xacro:xarm_gripper_ros2_control prefix="${prefix}" ros2_control_plugin="${ros2_control_plugin}" />
     <xacro:xarm_gripper_urdf prefix="${prefix}" attach_to="${attach_to}" xyz="${xyz}" rpy="${rpy}" />
     <xacro:xarm_gripper_transmission prefix="${prefix}" hard_interface="${'EffortJointInterface' if effort_control else 'VelocityJointInterface' if velocity_control else 'PositionJointInterface'}" />

File: xarm_description/urdf/xarm_device_macro.xacro (robot description, xacro)
@@ -27,5 +27,5 @@
     <xacro:if value="${add_gripper}">
       <xacro:include filename="$(find xarm_description)/urdf/gripper/xarm_gripper_model.xacro" />
-      <xacro:load_gripper prefix="${prefix}" attach_to="${prefix}link_eef" effort_control="${effort_control}" velocity_control="${velocity_control}" />
+      <xacro:load_gripper prefix="${prefix}" attach_to="${prefix}link_eef" effort_control="${effort_control}" velocity_control="${velocity_control}" ros2_control_plugin="${ros2_control_plugin}" />
     </xacro:if>
     <xacro:if value="${add_vacuum_gripper}">
