Commit message: modify urdf mesh filename

File: xarm_description/urdf/gripper/xarm_gripper.urdf.xacro (robot description, xacro)
@@ -33,6 +33,6 @@
         rpy="0 0 0" />
       <geometry>
-        <mesh
-          filename="package://xarm_description/meshes/gripper/base_link.STL" />
+        <!-- <mesh filename="package://xarm_description/meshes/gripper/base_link.STL" /> -->
+        <mesh filename="file:///$(find xarm_description)/meshes/gripper/base_link.STL"/>
       </geometry>
       <!-- <material
@@ -50,6 +50,6 @@
         rpy="0 0 0" />
       <geometry>
-        <mesh
-          filename="package://xarm_description/meshes/gripper/base_link.STL" />
+        <!-- <mesh filename="package://xarm_description/meshes/gripper/base_link.STL" /> -->
+        <mesh filename="file:///$(find xarm_description)/meshes/gripper/base_link.STL"/>
       </geometry>
     </collision>
@@ -76,18 +76,18 @@
         rpy="0 0 0" />
       <geometry>
-        <mesh
-          filename="package://xarm_description/meshes/gripper/left_outer_knuckle.STL" />
-      </geometry>
-      <material name="Silver">
-        <color rgba="0.753 0.753 0.753 1.0"/>
-      </material>
-    </visual>
-    <collision>
-      <origin
-        xyz="0 0 0"
-        rpy="0 0 0" />
-      <geometry>
-        <mesh
-          filename="package://xarm_description/meshes/gripper/left_outer_knuckle.STL" />
+        <!-- <mesh filename="package://xarm_description/meshes/gripper/left_outer_knuckle.STL" /> -->
+        <mesh filename="file:///$(find xarm_description)/meshes/gripper/left_outer_knuckle.STL"/>
+      </geometry>
+      <material name="Silver">
+        <color rgba="0.753 0.753 0.753 1.0"/>
+      </material>
+    </visual>
+    <collision>
+      <origin
+        xyz="0 0 0"
+        rpy="0 0 0" />
+      <geometry>
+        <!-- <mesh filename="package://xarm_description/meshes/gripper/left_outer_knuckle.STL" /> -->
+        <mesh filename="file:///$(find xarm_description)/meshes/gripper/left_outer_knuckle.STL"/>
       </geometry>
     </collision>
@@ -132,18 +132,18 @@
         rpy="0 0 0" />
       <geometry>
-        <mesh
-          filename="package://xarm_description/meshes/gripper/left_finger.STL" />
-      </geometry>
-      <material name="Silver">
-        <color rgba="0.753 0.753 0.753 1.0"/>
-      </material>
-    </visual>
-    <collision>
-      <origin
-        xyz="0 0 0"
-        rpy="0 0 0" />
-      <geometry>
-        <mesh
-          filename="package://xarm_description/meshes/gripper/left_finger.STL" />
+        <!-- <mesh filename="package://xarm_description/meshes/gripper/left_finger.STL" /> -->
+        <mesh filename="file:///$(find xarm_description)/meshes/gripper/left_finger.STL"/>
+      </geometry>
+      <material name="Silver">
+        <color rgba="0.753 0.753 0.753 1.0"/>
+      </material>
+    </visual>
+    <collision>
+      <origin
+        xyz="0 0 0"
+        rpy="0 0 0" />
+      <geometry>
+        <!-- <mesh filename="package://xarm_description/meshes/gripper/left_finger.STL" /> -->
+        <mesh filename="file:///$(find xarm_description)/meshes/gripper/left_finger.STL"/>
       </geometry>
     </collision>
@@ -189,18 +189,18 @@
         rpy="0 0 0" />
       <geometry>
-        <mesh
-          filename="package://xarm_description/meshes/gripper/left_inner_knuckle.STL" />
-      </geometry>
-      <material name="Silver">
-        <color rgba="0.753 0.753 0.753 1.0"/>
-      </material>
-    </visual>
-    <collision>
-      <origin
-        xyz="0 0 0"
-        rpy="0 0 0" />
-      <geometry>
-        <mesh
-          filename="package://xarm_description/meshes/gripper/left_inner_knuckle.STL" />
+        <!-- <mesh filename="package://xarm_description/meshes/gripper/left_inner_knuckle.STL" /> -->
+        <mesh filename="file:///$(find xarm_description)/meshes/gripper/left_inner_knuckle.STL"/>
+      </geometry>
+      <material name="Silver">
+        <color rgba="0.753 0.753 0.753 1.0"/>
+      </material>
+    </visual>
+    <collision>
+      <origin
+        xyz="0 0 0"
+        rpy="0 0 0" />
+      <geometry>
+        <!-- <mesh filename="package://xarm_description/meshes/gripper/left_inner_knuckle.STL" /> -->
+        <mesh filename="file:///$(find xarm_description)/meshes/gripper/left_inner_knuckle.STL"/>
       </geometry>
     </collision>
@@ -246,18 +246,18 @@
         rpy="0 0 0" />
       <geometry>
-        <mesh
-          filename="package://xarm_description/meshes/gripper/right_outer_knuckle.STL" />
-      </geometry>
-      <material name="Silver">
-        <color rgba="0.753 0.753 0.753 1.0"/>
-      </material>
-    </visual>
-    <collision>
-      <origin
-        xyz="0 0 0"
-        rpy="0 0 0" />
-      <geometry>
-        <mesh
-          filename="package://xarm_description/meshes/gripper/right_outer_knuckle.STL" />
+        <!-- <mesh filename="package://xarm_description/meshes/gripper/right_outer_knuckle.STL" /> -->
+        <mesh filename="file:///$(find xarm_description)/meshes/gripper/right_outer_knuckle.STL"/>
+      </geometry>
+      <material name="Silver">
+        <color rgba="0.753 0.753 0.753 1.0"/>
+      </material>
+    </visual>
+    <collision>
+      <origin
+        xyz="0 0 0"
+        rpy="0 0 0" />
+      <geometry>
+        <!-- <mesh filename="package://xarm_description/meshes/gripper/right_outer_knuckle.STL" /> -->
+        <mesh filename="file:///$(find xarm_description)/meshes/gripper/right_outer_knuckle.STL"/>
       </geometry>
     </collision>
@@ -303,18 +303,18 @@
         rpy="0 0 0" />
       <geometry>
-        <mesh
-          filename="package://xarm_description/meshes/gripper/right_finger.STL" />
-      </geometry>
-      <material name="Silver">
-        <color rgba="0.753 0.753 0.753 1.0"/>
-      </material>
-    </visual>
-    <collision>
-      <origin
-        xyz="0 0 0"
-        rpy="0 0 0" />
-      <geometry>
-        <mesh
-          filename="package://xarm_description/meshes/gripper/right_finger.STL" />
+        <!-- <mesh filename="package://xarm_description/meshes/gripper/right_finger.STL" /> -->
+        <mesh filename="file:///$(find xarm_description)/meshes/gripper/right_finger.STL"/>
+      </geometry>
+      <material name="Silver">
+        <color rgba="0.753 0.753 0.753 1.0"/>
+      </material>
+    </visual>
+    <collision>
+      <origin
+        xyz="0 0 0"
+        rpy="0 0 0" />
+      <geometry>
+        <!-- <mesh filename="package://xarm_description/meshes/gripper/right_finger.STL" /> -->
+        <mesh filename="file:///$(find xarm_description)/meshes/gripper/right_finger.STL"/>
       </geometry>
     </collision>
@@ -360,18 +360,18 @@
         rpy="0 0 0" />
       <geometry>
-        <mesh
-          filename="package://xarm_description/meshes/gripper/right_inner_knuckle.STL" />
-      </geometry>
-      <material name="Silver">
-        <color rgba="0.753 0.753 0.753 1.0"/>
-      </material>
-    </visual>
-    <collision>
-      <origin
-        xyz="0 0 0"
-        rpy="0 0 0" />
-      <geometry>
-        <mesh
-          filename="package://xarm_description/meshes/gripper/right_inner_knuckle.STL" />
+        <!-- <mesh filename="package://xarm_description/meshes/gripper/right_inner_knuckle.STL" /> -->
+        <mesh filename="file:///$(find xarm_description)/meshes/gripper/right_inner_knuckle.STL"/>
+      </geometry>
+      <material name="Silver">
+        <color rgba="0.753 0.753 0.753 1.0"/>
+      </material>
+    </visual>
+    <collision>
+      <origin
+        xyz="0 0 0"
+        rpy="0 0 0" />
+      <geometry>
+        <!-- <mesh filename="package://xarm_description/meshes/gripper/right_inner_knuckle.STL" /> -->
+        <mesh filename="file:///$(find xarm_description)/meshes/gripper/right_inner_knuckle.STL"/>
       </geometry>
     </collision>

File: xarm_description/urdf/vacuum_gripper/xarm_vacuum_gripper.urdf.xacro (robot description, xacro)
@@ -33,6 +33,6 @@
         rpy="0 0 0" />
       <geometry>
-        <mesh
-          filename="package://xarm_description/meshes/vacuum_gripper/visual/vacuum_gripper.STL" />
+        <!-- <mesh filename="package://xarm_description/meshes/vacuum_gripper/visual/vacuum_gripper.STL" /> -->
+        <mesh filename="file:///$(find xarm_description)/meshes/vacuum_gripper/visual/vacuum_gripper.STL"/>
       </geometry>
       <material name="White">
@@ -45,6 +45,6 @@
         rpy="0 0 0" />
       <geometry>
-        <mesh
-          filename="package://xarm_description/meshes/vacuum_gripper/collision/vacuum_gripper.STL" />
+        <!-- <mesh filename="package://xarm_description/meshes/vacuum_gripper/collision/vacuum_gripper.STL" /> -->
+        <mesh filename="file:///$(find xarm_description)/meshes/vacuum_gripper/collision/vacuum_gripper.STL"/>
       </geometry>
     </collision>

File: xarm_description/urdf/xarm5/xarm5.urdf.xacro (robot description, xacro)
@@ -40,16 +40,16 @@
           rpy="0 0 0" />
         <geometry>
-          <mesh
-            filename="package://xarm_description/meshes/xarm5/visual/base_link.STL" />
-        </geometry>
-        <material name="${prefix}White" />
-      </visual>
-      <collision>
-        <origin
-          xyz="0 0 0"
-          rpy="0 0 0" />
-        <geometry>
-          <mesh
-            filename="package://xarm_description/meshes/xarm5/visual/base_link.STL" />
+          <!-- <mesh filename="package://xarm_description/meshes/xarm5/visual/base_link.STL" /> -->
+          <mesh filename="file:///$(find xarm_description)/meshes/xarm5/visual/base_link.STL"/>
+        </geometry>
+        <material name="${prefix}White" />
+      </visual>
+      <collision>
+        <origin
+          xyz="0 0 0"
+          rpy="0 0 0" />
+        <geometry>
+          <!-- <mesh filename="package://xarm_description/meshes/xarm5/visual/base_link.STL" /> -->
+          <mesh filename="file:///$(find xarm_description)/meshes/xarm5/visual/base_link.STL"/>
         </geometry>
       </collision>
@@ -76,16 +76,16 @@
           rpy="0 0 0" />
         <geometry>
-          <mesh
-            filename="package://xarm_description/meshes/xarm5/visual/link1.STL" />
-        </geometry>
-        <material name="${prefix}White" />
-      </visual>
-      <collision>
-        <origin
-          xyz="0 0 0"
-          rpy="0 0 0" />
-        <geometry>
-          <mesh
-            filename="package://xarm_description/meshes/xarm5/visual/link1.STL" />
+          <!-- <mesh filename="package://xarm_description/meshes/xarm5/visual/link1.STL" /> -->
+          <mesh filename="file:///$(find xarm_description)/meshes/xarm5/visual/link1.STL"/>
+        </geometry>
+        <material name="${prefix}White" />
+      </visual>
+      <collision>
+        <origin
+          xyz="0 0 0"
+          rpy="0 0 0" />
+        <geometry>
+          <!-- <mesh filename="package://xarm_description/meshes/xarm5/visual/link1.STL" /> -->
+          <mesh filename="file:///$(find xarm_description)/meshes/xarm5/visual/link1.STL"/>
         </geometry>
       </collision>
@@ -133,16 +133,16 @@
           rpy="0 0 0" />
         <geometry>
-          <mesh
-            filename="package://xarm_description/meshes/xarm5/visual/link2.STL" />
-        </geometry>
-        <material name="${prefix}White" />
-      </visual>
-      <collision>
-        <origin
-          xyz="0 0 0"
-          rpy="0 0 0" />
-        <geometry>
-          <mesh
-            filename="package://xarm_description/meshes/xarm5/visual/link2.STL" />
+          <!-- <mesh filename="package://xarm_description/meshes/xarm5/visual/link2.STL" /> -->
+          <mesh filename="file:///$(find xarm_description)/meshes/xarm5/visual/link2.STL"/>
+        </geometry>
+        <material name="${prefix}White" />
+      </visual>
+      <collision>
+        <origin
+          xyz="0 0 0"
+          rpy="0 0 0" />
+        <geometry>
+          <!-- <mesh filename="package://xarm_description/meshes/xarm5/visual/link2.STL" /> -->
+          <mesh filename="file:///$(find xarm_description)/meshes/xarm5/visual/link2.STL"/>
         </geometry>
       </collision>
@@ -190,16 +190,16 @@
           rpy="0 0 0" />
         <geometry>
-          <mesh
-            filename="package://xarm_description/meshes/xarm5/visual/link3.STL" />
-        </geometry>
-        <material name="${prefix}White" />
-      </visual>
-      <collision>
-        <origin
-          xyz="0 0 0"
-          rpy="0 0 0" />
-        <geometry>
-          <mesh
-            filename="package://xarm_description/meshes/xarm5/visual/link3.STL" />
+          <!-- <mesh filename="package://xarm_description/meshes/xarm5/visual/link3.STL" /> -->
+          <mesh filename="file:///$(find xarm_description)/meshes/xarm5/visual/link3.STL"/>
+        </geometry>
+        <material name="${prefix}White" />
+      </visual>
+      <collision>
+        <origin
+          xyz="0 0 0"
+          rpy="0 0 0" />
+        <geometry>
+          <!-- <mesh filename="package://xarm_description/meshes/xarm5/visual/link3.STL" /> -->
+          <mesh filename="file:///$(find xarm_description)/meshes/xarm5/visual/link3.STL"/>
         </geometry>
       </collision>
@@ -247,16 +247,16 @@
           rpy="0 0 0" />
         <geometry>
-          <mesh
-            filename="package://xarm_description/meshes/xarm5/visual/link4.STL" />
-        </geometry>
-        <material name="${prefix}White" />
-      </visual>
-      <collision>
-        <origin
-          xyz="0 0 0"
-          rpy="0 0 0" />
-        <geometry>
-          <mesh
-            filename="package://xarm_description/meshes/xarm5/visual/link4.STL" />
+          <!-- <mesh filename="package://xarm_description/meshes/xarm5/visual/link4.STL" /> -->
+          <mesh filename="file:///$(find xarm_description)/meshes/xarm5/visual/link4.STL"/>
+        </geometry>
+        <material name="${prefix}White" />
+      </visual>
+      <collision>
+        <origin
+          xyz="0 0 0"
+          rpy="0 0 0" />
+        <geometry>
+          <!-- <mesh filename="package://xarm_description/meshes/xarm5/visual/link4.STL" /> -->
+          <mesh filename="file:///$(find xarm_description)/meshes/xarm5/visual/link4.STL"/>
         </geometry>
       </collision>
@@ -304,6 +304,6 @@
           rpy="0 0 0" />
         <geometry>
-          <mesh
-            filename="package://xarm_description/meshes/xarm5/visual/link5.STL" />
+          <!-- <mesh filename="package://xarm_description/meshes/xarm5/visual/link5.STL" /> -->
+          <mesh filename="file:///$(find xarm_description)/meshes/xarm5/visual/link5.STL"/>
         </geometry>
         <material name="${prefix}Silver" />
@@ -314,6 +314,6 @@
           rpy="0 0 0" />
         <geometry>
-          <mesh
-            filename="package://xarm_description/meshes/xarm5/visual/link5.STL" />
+          <!-- <mesh filename="package://xarm_description/meshes/xarm5/visual/link5.STL" /> -->
+          <mesh filename="file:///$(find xarm_description)/meshes/xarm5/visual/link5.STL"/>
         </geometry>
       </collision>

File: xarm_description/urdf/xarm6/xarm6.urdf.xacro (robot description, xacro)
@@ -23,12 +23,14 @@
       <visual>
         <geometry>
-          <mesh filename="package://xarm_description/meshes/xarm6/visual/base.stl"/>
-        </geometry>
-        <origin xyz="0 0 0" rpy="0 0 0"/>
-        <material name="${prefix}White" />
-      </visual>
-      <collision>
-        <geometry>
-          <mesh filename="package://xarm_description/meshes/xarm6/visual/base.stl"/>
+          <!-- <mesh filename="package://xarm_description/meshes/xarm6/visual/base.stl"/> -->
+          <mesh filename="file:///$(find xarm_description)/meshes/xarm6/visual/base.stl"/>
+        </geometry>
+        <origin xyz="0 0 0" rpy="0 0 0"/>
+        <material name="${prefix}White" />
+      </visual>
+      <collision>
+        <geometry>
+          <!-- <mesh filename="package://xarm_description/meshes/xarm6/visual/base.stl"/> -->
+          <mesh filename="file:///$(find xarm_description)/meshes/xarm6/visual/base.stl"/>
         </geometry>
         <origin xyz="0 0 0" rpy="0 0 0"/>
@@ -49,12 +51,14 @@
       <visual>
         <geometry>
-          <mesh filename="package://xarm_description/meshes/xarm6/visual/link1.stl"/>
-        </geometry>
-        <origin xyz="0 0 0" rpy="0 0 0"/>
-        <material name="${prefix}White" />
-      </visual>
-      <collision>
-        <geometry>
-          <mesh filename="package://xarm_description/meshes/xarm6/visual/link1.stl"/>
+          <!-- <mesh filename="package://xarm_description/meshes/xarm6/visual/link1.stl"/> -->
+          <mesh filename="file:///$(find xarm_description)/meshes/xarm6/visual/link1.stl"/>
+        </geometry>
+        <origin xyz="0 0 0" rpy="0 0 0"/>
+        <material name="${prefix}White" />
+      </visual>
+      <collision>
+        <geometry>
+          <!-- <mesh filename="package://xarm_description/meshes/xarm6/visual/link1.stl"/> -->
+          <mesh filename="file:///$(find xarm_description)/meshes/xarm6/visual/link1.stl"/>
         </geometry>
         <origin xyz="0 0 0" rpy="0 0 0"/>
@@ -87,12 +91,14 @@
       <visual>
         <geometry>
-          <mesh filename="package://xarm_description/meshes/xarm6/visual/link2.stl"/>
-        </geometry>
-        <origin xyz="0 0 0" rpy="0 0 0"/>
-        <material name="${prefix}White" />
-      </visual>
-      <collision>
-        <geometry>
-          <mesh filename="package://xarm_description/meshes/xarm6/visual/link2.stl"/>
+          <!-- <mesh filename="package://xarm_description/meshes/xarm6/visual/link2.stl"/> -->
+          <mesh filename="file:///$(find xarm_description)/meshes/xarm6/visual/link2.stl"/>
+        </geometry>
+        <origin xyz="0 0 0" rpy="0 0 0"/>
+        <material name="${prefix}White" />
+      </visual>
+      <collision>
+        <geometry>
+          <!-- <mesh filename="package://xarm_description/meshes/xarm6/visual/link2.stl"/> -->
+          <mesh filename="file:///$(find xarm_description)/meshes/xarm6/visual/link2.stl"/>
         </geometry>
         <origin xyz="0 0 0" rpy="0 0 0"/>
@@ -128,12 +134,14 @@
       <visual>
         <geometry>
-          <mesh filename="package://xarm_description/meshes/xarm6/visual/link3.stl"/>
-        </geometry>
-        <origin xyz="0 0 0" rpy="0 0 0"/>
-        <material name="${prefix}White" />
-      </visual>
-      <collision>
-        <geometry>
-          <mesh filename="package://xarm_description/meshes/xarm6/visual/link3.stl"/>
+          <!-- <mesh filename="package://xarm_description/meshes/xarm6/visual/link3.stl"/> -->
+          <mesh filename="file:///$(find xarm_description)/meshes/xarm6/visual/link3.stl"/>
+        </geometry>
+        <origin xyz="0 0 0" rpy="0 0 0"/>
+        <material name="${prefix}White" />
+      </visual>
+      <collision>
+        <geometry>
+          <!-- <mesh filename="package://xarm_description/meshes/xarm6/visual/link3.stl"/> -->
+          <mesh filename="file:///$(find xarm_description)/meshes/xarm6/visual/link3.stl"/>
         </geometry>
         <origin xyz="0 0 0" rpy="0 0 0"/>
@@ -169,12 +177,14 @@
       <visual>
         <geometry>
-          <mesh filename="package://xarm_description/meshes/xarm6/visual/link4.stl"/>
-        </geometry>
-        <origin xyz="0 0 0" rpy="0 0 0"/>
-        <material name="${prefix}White" />
-      </visual>
-      <collision>
-        <geometry>
-          <mesh filename="package://xarm_description/meshes/xarm6/visual/link4.stl"/>
+          <!-- <mesh filename="package://xarm_description/meshes/xarm6/visual/link4.stl"/> -->
+          <mesh filename="file:///$(find xarm_description)/meshes/xarm6/visual/link4.stl"/>
+        </geometry>
+        <origin xyz="0 0 0" rpy="0 0 0"/>
+        <material name="${prefix}White" />
+      </visual>
+      <collision>
+        <geometry>
+          <!-- <mesh filename="package://xarm_description/meshes/xarm6/visual/link4.stl"/> -->
+          <mesh filename="file:///$(find xarm_description)/meshes/xarm6/visual/link4.stl"/>
         </geometry>
         <origin xyz="0 0 0" rpy="0 0 0"/>
@@ -207,12 +217,14 @@
       <visual>
         <geometry>
-          <mesh filename="package://xarm_description/meshes/xarm6/visual/link5.stl"/>
-        </geometry>
-        <origin xyz="0 0 0" rpy="0 0 0"/>
-        <material name="${prefix}White" />
-      </visual>
-      <collision>
-        <geometry>
-          <mesh filename="package://xarm_description/meshes/xarm6/visual/link5.stl"/>
+          <!-- <mesh filename="package://xarm_description/meshes/xarm6/visual/link5.stl"/> -->
+          <mesh filename="file:///$(find xarm_description)/meshes/xarm6/visual/link5.stl"/>
+        </geometry>
+        <origin xyz="0 0 0" rpy="0 0 0"/>
+        <material name="${prefix}White" />
+      </visual>
+      <collision>
+        <geometry>
+          <!-- <mesh filename="package://xarm_description/meshes/xarm6/visual/link5.stl"/> -->
+          <mesh filename="file:///$(find xarm_description)/meshes/xarm6/visual/link5.stl"/>
         </geometry>
         <origin xyz="0 0 0" rpy="0 0 0"/>
@@ -248,5 +260,6 @@
       <visual>
         <geometry>
-          <mesh filename="package://xarm_description/meshes/xarm6/visual/link6.stl"/>
+          <!-- <mesh filename="package://xarm_description/meshes/xarm6/visual/link6.stl"/> -->
+          <mesh filename="file:///$(find xarm_description)/meshes/xarm6/visual/link6.stl"/>
         </geometry>
         <origin xyz="0 0 0" rpy="0 0 0"/>
@@ -255,5 +268,6 @@
       <collision>
         <geometry>
-          <mesh filename="package://xarm_description/meshes/xarm6/visual/link6.stl"/>
+          <!-- <mesh filename="package://xarm_description/meshes/xarm6/visual/link6.stl"/> -->
+          <mesh filename="file:///$(find xarm_description)/meshes/xarm6/visual/link6.stl"/>
         </geometry>
         <origin xyz="0 0 0" rpy="0 0 0"/>
