Commit message: modify urdf mesh filename

File: xarm_description/urdf/xarm7/xarm7.urdf.xacro (robot description, xacro)
@@ -42,16 +42,16 @@
         rpy="0 0 0" />
       <geometry>
-        <mesh
-          filename="package://xarm_description/meshes/xarm7/visual/link_base.STL" />
-      </geometry>
-      <material name="${prefix}White" />
-    </visual>
-    <collision>
-      <origin
-        xyz="0 0 0"
-        rpy="0 0 0" />
-      <geometry>
-        <mesh
-          filename="package://xarm_description/meshes/xarm7/visual/link_base.STL" />
+        <!-- <mesh filename="package://xarm_description/meshes/xarm7/visual/link_base.STL" /> -->
+        <mesh filename="file:///$(find xarm_description)/meshes/xarm7/visual/link_base.STL"/>
+      </geometry>
+      <material name="${prefix}White" />
+    </visual>
+    <collision>
+      <origin
+        xyz="0 0 0"
+        rpy="0 0 0" />
+      <geometry>
+        <!-- <mesh filename="package://xarm_description/meshes/xarm7/visual/link_base.STL" /> -->
+        <mesh filename="file:///$(find xarm_description)/meshes/xarm7/visual/link_base.STL"/>
       </geometry>
     </collision>
@@ -78,16 +78,16 @@
         rpy="0 0 0" />
       <geometry>
-        <mesh
-          filename="package://xarm_description/meshes/xarm7/visual/link1.STL" />
-      </geometry>
-      <material name="${prefix}White" />
-    </visual>
-    <collision>
-      <origin
-        xyz="0 0 0"
-        rpy="0 0 0" />
-      <geometry>
-        <mesh
-          filename="package://xarm_description/meshes/xarm7/visual/link1.STL" />
+        <!-- <mesh filename="package://xarm_description/meshes/xarm7/visual/link1.STL" /> -->
+        <mesh filename="file:///$(find xarm_description)/meshes/xarm7/visual/link1.STL"/>
+      </geometry>
+      <material name="${prefix}White" />
+    </visual>
+    <collision>
+      <origin
+        xyz="0 0 0"
+        rpy="0 0 0" />
+      <geometry>
+        <!-- <mesh filename="package://xarm_description/meshes/xarm7/visual/link1.STL" /> -->
+        <mesh filename="file:///$(find xarm_description)/meshes/xarm7/visual/link1.STL"/>
       </geometry>
     </collision>
@@ -135,16 +135,16 @@
         rpy="0 0 0" />
       <geometry>
-        <mesh
-          filename="package://xarm_description/meshes/xarm7/visual/link2.STL" />
-      </geometry>
-      <material name="${prefix}White" />
-    </visual>
-    <collision>
-      <origin
-        xyz="0 0 0"
-        rpy="0 0 0" />
-      <geometry>
-        <mesh
-          filename="package://xarm_description/meshes/xarm7/visual/link2.STL" />
+        <!-- <mesh filename="package://xarm_description/meshes/xarm7/visual/link2.STL" /> -->
+        <mesh filename="file:///$(find xarm_description)/meshes/xarm7/visual/link2.STL"/>
+      </geometry>
+      <material name="${prefix}White" />
+    </visual>
+    <collision>
+      <origin
+        xyz="0 0 0"
+        rpy="0 0 0" />
+      <geometry>
+        <!-- <mesh filename="package://xarm_description/meshes/xarm7/visual/link2.STL" /> -->
+        <mesh filename="file:///$(find xarm_description)/meshes/xarm7/visual/link2.STL"/>
       </geometry>
     </collision>
@@ -192,16 +192,16 @@
         rpy="0 0 0" />
       <geometry>
-        <mesh
-          filename="package://xarm_description/meshes/xarm7/visual/link3.STL" />
-      </geometry>
-      <material name="${prefix}White" />
-    </visual>
-    <collision>
-      <origin
-        xyz="0 0 0"
-        rpy="0 0 0" />
-      <geometry>
-        <mesh
-          filename="package://xarm_description/meshes/xarm7/visual/link3.STL" />
+        <!-- <mesh filename="package://xarm_description/meshes/xarm7/visual/link3.STL" /> -->
+        <mesh filename="file:///$(find xarm_description)/meshes/xarm7/visual/link3.STL"/>
+      </geometry>
+      <material name="${prefix}White" />
+    </visual>
+    <collision>
+      <origin
+        xyz="0 0 0"
+        rpy="0 0 0" />
+      <geometry>
+        <!-- <mesh filename="package://xarm_description/meshes/xarm7/visual/link3.STL" /> -->
+        <mesh filename="file:///$(find xarm_description)/meshes/xarm7/visual/link3.STL"/>
       </geometry>
     </collision>
@@ -249,16 +249,16 @@
         rpy="0 0 0" />
       <geometry>
-        <mesh
-          filename="package://xarm_description/meshes/xarm7/visual/link4.STL" />
-      </geometry>
-      <material name="${prefix}White" />
-    </visual>
-    <collision>
-      <origin
-        xyz="0 0 0"
-        rpy="0 0 0" />
-      <geometry>
-        <mesh
-          filename="package://xarm_description/meshes/xarm7/visual/link4.STL" />
+        <!-- <mesh filename="package://xarm_description/meshes/xarm7/visual/link4.STL" /> -->
+        <mesh filename="file:///$(find xarm_description)/meshes/xarm7/visual/link4.STL"/>
+      </geometry>
+      <material name="${prefix}White" />
+    </visual>
+    <collision>
+      <origin
+        xyz="0 0 0"
+        rpy="0 0 0" />
+      <geometry>
+        <!-- <mesh filename="package://xarm_description/meshes/xarm7/visual/link4.STL" /> -->
+        <mesh filename="file:///$(find xarm_description)/meshes/xarm7/visual/link4.STL"/>
       </geometry>
     </collision>
@@ -306,16 +306,16 @@
         rpy="0 0 0" />
       <geometry>
-        <mesh
-          filename="package://xarm_description/meshes/xarm7/visual/link5.STL" />
-      </geometry>
-      <material name="${prefix}White" />
-    </visual>
-    <collision>
-      <origin
-        xyz="0 0 0"
-        rpy="0 0 0" />
-      <geometry>
-        <mesh
-          filename="package://xarm_description/meshes/xarm7/visual/link5.STL" />
+        <!-- <mesh filename="package://xarm_description/meshes/xarm7/visual/link5.STL" /> -->
+        <mesh filename="file:///$(find xarm_description)/meshes/xarm7/visual/link5.STL"/>
+      </geometry>
+      <material name="${prefix}White" />
+    </visual>
+    <collision>
+      <origin
+        xyz="0 0 0"
+        rpy="0 0 0" />
+      <geometry>
+        <!-- <mesh filename="package://xarm_description/meshes/xarm7/visual/link5.STL" /> -->
+        <mesh filename="file:///$(find xarm_description)/meshes/xarm7/visual/link5.STL"/>
       </geometry>
     </collision>
@@ -363,16 +363,16 @@
         rpy="0 0 0" />
       <geometry>
-        <mesh
-          filename="package://xarm_description/meshes/xarm7/visual/link6.STL" />
-      </geometry>
-      <material name="${prefix}White" />
-    </visual>
-    <collision>
-      <origin
-        xyz="0 0 0"
-        rpy="0 0 0" />
-      <geometry>
-        <mesh
-          filename="package://xarm_description/meshes/xarm7/visual/link6.STL" />
+        <!-- <mesh filename="package://xarm_description/meshes/xarm7/visual/link6.STL" /> -->
+        <mesh filename="file:///$(find xarm_description)/meshes/xarm7/visual/link6.STL"/>
+      </geometry>
+      <material name="${prefix}White" />
+    </visual>
+    <collision>
+      <origin
+        xyz="0 0 0"
+        rpy="0 0 0" />
+      <geometry>
+        <!-- <mesh filename="package://xarm_description/meshes/xarm7/visual/link6.STL" /> -->
+        <mesh filename="file:///$(find xarm_description)/meshes/xarm7/visual/link6.STL"/>
       </geometry>
     </collision>
@@ -420,6 +420,6 @@
         rpy="0 0 0" />
       <geometry>
-        <mesh
-          filename="package://xarm_description/meshes/xarm7/visual/link7.STL" />
+        <!-- <mesh filename="package://xarm_description/meshes/xarm7/visual/link7.STL" /> -->
+        <mesh filename="file:///$(find xarm_description)/meshes/xarm7/visual/link7.STL"/>
       </geometry>
       <material name="${prefix}Silver" />
@@ -430,6 +430,6 @@
         rpy="0 0 0" />
       <geometry>
-        <mesh
-          filename="package://xarm_description/meshes/xarm7/visual/link7.STL" />
+        <!-- <mesh filename="package://xarm_description/meshes/xarm7/visual/link7.STL" /> -->
+        <mesh filename="file:///$(find xarm_description)/meshes/xarm7/visual/link7.STL"/>
       </geometry>
     </collision>
