Commit message: Fix URDF file
1. delete gripper/xarm_gripper.xacro (no use)
2. rename gripper/xarm_gripper_model.xacro ->
gripper/xarm_gripper_macro.xacro
3. change the mesh filename in lite (vacuum) gripper urdf

File: xarm_description/urdf/gripper/lite_gripper.urdf.xacro (robot description, xacro)
@@ -33,6 +33,5 @@
         rpy="0 0 0" />
       <geometry>
-        <mesh
-          filename="package://xarm_description/meshes/lite6/visual/gripper_lite.stl" />
+        <mesh filename="file:///$(find xarm_description)/meshes/lite6/visual/gripper_lite.stl"/>
       </geometry>
       <material name="White">
@@ -45,6 +44,5 @@
         rpy="0 0 0" />
       <geometry>
-        <mesh
-          filename="package://xarm_description/meshes/lite6/collision/gripper_lite.stl" />
+        <mesh filename="file:///$(find xarm_description)/meshes/lite6/collision/gripper_lite.stl"/>
       </geometry>
     </collision>

File: xarm_description/urdf/gripper/xarm_gripper_macro.xacro (robot description, xacro)
@@ -6,5 +6,5 @@
   <xacro:include filename="$(find xarm_description)/urdf/gripper/xarm_gripper.transmission.xacro" />
   <xacro:include filename="$(find xarm_description)/urdf/gripper/xarm_gripper.gazebo.xacro" />
-  <xacro:macro name="load_gripper" params="prefix:='' attach_to:='' ns:='xarm' xyz:='0 0 0' rpy:='0 0 0' effort_control:='false' velocity_control:='false'
+  <xacro:macro name="xarm_gripper_macro" params="prefix:='' attach_to:='' ns:='xarm' xyz:='0 0 0' rpy:='0 0 0' effort_control:='false' velocity_control:='false'
     load_gazebo_plugin:='false' ros2_control_plugin:='xarm_control/FakeXArmHW' ros2_control_params:='' ">
     <!-- gazebo_plugin -->

File: xarm_description/urdf/lite6/lite6_robot_macro.xacro (robot description, xacro)
@@ -28,17 +28,17 @@
         ros2_control_plugin="${ros2_control_plugin}"
         hw_ns="${namespace}"
-        joint1_lower_limit="${-2.0*pi}"   joint1_upper_limit="${2.0*pi}"
+        joint1_lower_limit="${-pi}"   joint1_upper_limit="${pi}"
         joint2_lower_limit="${-2.61799}"  joint2_upper_limit="${2.61799}"
         joint3_lower_limit="${-0.061087}" joint3_upper_limit="${5.235988}"
-        joint4_lower_limit="${-2.0*pi}"   joint4_upper_limit="${2.0*pi}"
+        joint4_lower_limit="${-pi}"   joint4_upper_limit="${pi}"
         joint5_lower_limit="${-2.1642}"   joint5_upper_limit="${2.1642}"
-        joint6_lower_limit="${-2.0*pi}"   joint6_upper_limit="${2.0*pi}"/>
+        joint6_lower_limit="${-pi}"   joint6_upper_limit="${pi}"/>
       <xacro:lite6_urdf prefix="${prefix}"
-        joint1_lower_limit="${-2.0*pi}"   joint1_upper_limit="${2.0*pi}"
+        joint1_lower_limit="${-pi}"   joint1_upper_limit="${pi}"
         joint2_lower_limit="${-2.61799}"  joint2_upper_limit="${2.61799}"
         joint3_lower_limit="${-0.061087}" joint3_upper_limit="${5.235988}"
-        joint4_lower_limit="${-2.0*pi}"   joint4_upper_limit="${2.0*pi}"
+        joint4_lower_limit="${-pi}"   joint4_upper_limit="${pi}"
         joint5_lower_limit="${-2.1642}"   joint5_upper_limit="${2.1642}"
-        joint6_lower_limit="${-2.0*pi}"   joint6_upper_limit="${2.0*pi}"/>
+        joint6_lower_limit="${-pi}"   joint6_upper_limit="${pi}"/>
     </xacro:if>
     <xacro:unless value="${limited}">

File: xarm_description/urdf/vacuum_gripper/lite_vacuum_gripper.urdf.xacro (robot description, xacro)
@@ -33,6 +33,5 @@
         rpy="0 0 0" />
       <geometry>
-        <mesh
-          filename="package://xarm_description/meshes/lite6/visual/vacuum_gripper_lite.stl" />
+        <mesh filename="file:///$(find xarm_description)/meshes/lite6/visual/vacuum_gripper_lite.stl"/>
       </geometry>
       <material name="White">
@@ -45,6 +44,5 @@
         rpy="0 0 0" />
       <geometry>
-        <mesh
-          filename="package://xarm_description/meshes/lite6/collision/vacuum_gripper_lite.stl" />
+        <mesh filename="file:///$(find xarm_description)/meshes/lite6/collision/vacuum_gripper_lite.stl"/>
       </geometry>
     </collision>

File: xarm_description/urdf/xarm_device_macro.xacro (robot description, xacro)
@@ -14,4 +14,5 @@
     geometry_mesh_tcp_rpy:='0 0 0' ">
     <xacro:if value="${dof == 5}">
+      <!-- Load XArm5 Robot Model URDF -->
       <xacro:include filename="$(find xarm_description)/urdf/xarm5/xarm5_robot_macro.xacro" />
       <xacro:xarm5_robot prefix="${prefix}" namespace="${namespace}" limited="${limited}"
@@ -24,4 +25,5 @@
     <xacro:if value="${dof == 6}">
       <xacro:if value="${robot_type == 'lite'}">
+        <!-- Load Lite6 Robot Model URDF -->
         <xacro:include filename="$(find xarm_description)/urdf/lite6/lite6_robot_macro.xacro" />
         <xacro:lite6_robot prefix="${prefix}" namespace="${namespace}" limited="${limited}"
@@ -33,4 +35,5 @@
       </xacro:if>
       <xacro:unless value="${robot_type == 'lite'}">
+        <!-- Load XArm6 Robot Model URDF -->
         <xacro:include filename="$(find xarm_description)/urdf/xarm6/xarm6_robot_macro.xacro" />
         <xacro:xarm6_robot prefix="${prefix}" namespace="${namespace}" limited="${limited}"
@@ -43,4 +46,5 @@
     </xacro:if>
     <xacro:unless value="${dof == 5 or dof == 6}">
+      <!-- Load XArm7 Robot Model URDF -->
       <xacro:include filename="$(find xarm_description)/urdf/xarm7/xarm7_robot_macro.xacro" />
       <xacro:xarm7_robot prefix="${prefix}" namespace="${namespace}" limited="${limited}"
@@ -52,26 +56,31 @@
     </xacro:unless>
     <xacro:if value="${add_gripper}">
-      <xacro:if value="${robot_type == 'xarm'}">
-        <xacro:include filename="$(find xarm_description)/urdf/gripper/xarm_gripper_model.xacro" />
-        <xacro:load_gripper prefix="${prefix}" attach_to="${prefix}link_eef" effort_control="${effort_control}" velocity_control="${velocity_control}"
-          ros2_control_plugin="${ros2_control_plugin}" ros2_control_params="${ros2_control_params}"
-          load_gazebo_plugin="${load_gazebo_plugin}" />
-      </xacro:if>
       <xacro:if value="${robot_type == 'lite'}">
+        <!-- Load Lite Gripper Model URDF -->
         <xacro:include filename="$(find xarm_description)/urdf/gripper/lite_gripper.urdf.xacro" />
         <xacro:uflite_gripper_urdf prefix="${prefix}" attach_to="${prefix}link_eef" />
       </xacro:if>
+      <xacro:unless value="${robot_type == 'lite'}">
+        <!-- Load XArm Gripper Model URDF -->
+        <xacro:include filename="$(find xarm_description)/urdf/gripper/xarm_gripper_macro.xacro" />
+        <xacro:xarm_gripper_macro prefix="${prefix}" attach_to="${prefix}link_eef" effort_control="${effort_control}" velocity_control="${velocity_control}"
+          ros2_control_plugin="${ros2_control_plugin}" ros2_control_params="${ros2_control_params}"
+          load_gazebo_plugin="${load_gazebo_plugin}" />
+      </xacro:unless>
     </xacro:if>
     <xacro:if value="${not add_gripper and add_vacuum_gripper}">
-      <xacro:if value="${robot_type == 'xarm'}">
-        <xacro:include filename="$(find xarm_description)/urdf/vacuum_gripper/xarm_vacuum_gripper.urdf.xacro" />
-        <xacro:xarm_vacuum_gripper_urdf prefix="${prefix}" attach_to="${prefix}link_eef" effort_control="${effort_control}" velocity_control="${velocity_control}" />
-      </xacro:if>
       <xacro:if value="${robot_type == 'lite'}">
+        <!-- Load Lite Vacuum Gripper Model URDF -->
         <xacro:include filename="$(find xarm_description)/urdf/vacuum_gripper/lite_vacuum_gripper.urdf.xacro" />
         <xacro:uflite_vacuum_gripper_urdf prefix="${prefix}" attach_to="${prefix}link_eef" />
       </xacro:if>
+      <xacro:unless value="${robot_type == 'lite'}">
+        <!-- Load XArm Vacuum Gripper Model URDF -->
+        <xacro:include filename="$(find xarm_description)/urdf/vacuum_gripper/xarm_vacuum_gripper.urdf.xacro" />
+        <xacro:xarm_vacuum_gripper_urdf prefix="${prefix}" attach_to="${prefix}link_eef" effort_control="${effort_control}" velocity_control="${velocity_control}" />
+      </xacro:unless>
     </xacro:if>
     <xacro:if value="${not add_gripper and not add_vacuum_gripper and add_other_geometry}">
+      <!-- Load Other Model URDF -->
       <xacro:include filename="$(find xarm_description)/urdf/other/other_geometry.urdf.xacro" />
       <xacro:other_geometry prefix="${prefix}" attach_to="${prefix}link_eef"
