Commit message: Keep the gripper linkage together on gz by declaring mimic joints to ros2_control
The gripper's five follower joints are coupled to drive_joint by URDF
<mimic> tags alone, which leaves enforcement to the physics engine. gz's
default engine, DART, has no mimic constraint support
(gazebosim/gz-physics#432), so it warns and skips them:

  [Err] Attempting to create a mimic constraint for joint
  [left_finger_joint] but the chosen physics engine does not support
  mimic constraints, so no constraint will be created.

The fingers are then unconstrained and drift away from the gripper body.
The Gazebo Classic mimic_joint_plugin that used to cover this has no gz
equivalent (issue #111), so on jazzy there is nothing holding the
linkage together.

Declaring the followers in the ros2_control block moves the coupling a
layer above the physics engine. mimic="true" populates
HardwareInfo::mimic_joints, and gz_ros2_control drives each follower
from drive_joint every update; mock_components implements the same, so
fake hardware behaves consistently. This works on any engine rather than
depending on engine support.

The followers take no command interface, as they are driven by that loop
rather than claimed by a controller.

Real hardware is unaffected: this block is only emitted when the plugin
is not uf_robot_hardware/UFRobotSystemHardware, so the UFACTORY driver
path never sees these joints.

Verified on ROS 2 Jazzy / Gazebo Harmonic with an xArm6 + gripper:
- gz_ros2_control + DART: fingers track drive_joint symmetrically,
  0.070 m apart open and 0.027 m closed, where previously they detached
- mock_components/GenericSystem: gripper component loads active, the
  five joints appear as state interfaces with no command interfaces

File: xarm_description/urdf/gripper/xarm_gripper.ros2_control.xacro (robot description, xacro)
@@ -18,4 +18,34 @@
         <!-- <state_interface name="effort"/> -->
       </joint>
+      <!-- The five follower joints of the gripper's four-bar linkage carry
+           URDF <mimic> tags. Enforcing those is left to the physics engine,
+           and gz's default engine, DART, has no mimic constraint support
+           (gazebosim/gz-physics#432, still open):
+             [Err] Attempting to create a mimic constraint for joint
+             [left_finger_joint] but the chosen physics engine does not
+             support mimic constraints, so no constraint will be created.
+           The fingers then come adrift from the gripper body. The Gazebo
+           Classic mimic_joint_plugin this used to rely on is not available
+           for gz either (see issue #111).
+           Declaring the followers here instead makes ros2_control own the
+           coupling, a layer above the physics engine: mimic="true"
+           populates HardwareInfo::mimic_joints, and gz_ros2_control drives
+           each follower from drive_joint every update. mock_components does
+           the same, so fake hardware stays consistent.
+           Mimic joints deliberately take no command interface; they are
+           driven by that loop, not claimed by a controller. Real hardware is
+           unaffected, since this whole block is only emitted when the plugin
+           is not uf_robot_hardware/UFRobotSystemHardware. -->
+      <xacro:macro name="gripper_mimic_joint" params="name">
+        <joint name="${name}" mimic="true">
+          <state_interface name="position"/>
+          <state_interface name="velocity"/>
+        </joint>
+      </xacro:macro>
+      <xacro:gripper_mimic_joint name="${prefix}left_finger_joint"/>
+      <xacro:gripper_mimic_joint name="${prefix}left_inner_knuckle_joint"/>
+      <xacro:gripper_mimic_joint name="${prefix}right_outer_knuckle_joint"/>
+      <xacro:gripper_mimic_joint name="${prefix}right_finger_joint"/>
+      <xacro:gripper_mimic_joint name="${prefix}right_inner_knuckle_joint"/>
     </ros2_control>
   </xacro:macro>
