Commit message: fix urdf/srdf name and add gazebo_ros2_control

File: xarm_description/urdf/common/common.gazebo.xacro (robot description, xacro)
@@ -1,10 +1,9 @@
 <?xml version="1.0"?>
 <robot xmlns:xacro="http://ros.org/wiki/xacro">
-  <xacro:macro name="gazebo_ros_control_plugin" params="namespace">
+  <xacro:macro name="gazebo_ros_control_plugin" params="prefix:='' dof:=7">
     <gazebo>
       <plugin filename="libgazebo_ros2_control.so" name="gazebo_ros2_control">
-        <robotNamespace>/${namespace}</robotNamespace>
-        <robotSimType>gazebo_ros2_control/GazeboSystem</robotSimType>
-        <legacyModeNS>true</legacyModeNS>
+        <robot_sim_type>gazebo_ros2_control/GazeboSystem</robot_sim_type>
+        <parameters>$(find xarm_controller)/config/xarm${dof}_controllers.yaml</parameters>
       </plugin>
     </gazebo>

File: xarm_description/urdf/dual_xarm_device.urdf.xacro (robot description, xacro)
@@ -1,4 +1,4 @@
 <?xml version='1.0' encoding='utf-8'?>
-<robot xmlns:xacro="http://ros.org/wiki/xacro" name="xarm">
+<robot xmlns:xacro="http://ros.org/wiki/xacro" name="dual_xarm">
   <xacro:arg name="prefix_1" default="L_"/>
   <xacro:arg name="prefix_2" default="R_"/>

File: xarm_description/urdf/xarm5/xarm5_robot_macro.xacro (robot description, xacro)
@@ -12,5 +12,5 @@
     <xacro:if value="${load_gazebo_plugin}">
     <xacro:include filename="$(find xarm_description)/urdf/common/common.gazebo.xacro" />
-    <xacro:gazebo_ros_control_plugin namespace="${namespace}"/>
+    <xacro:gazebo_ros_control_plugin prefix="${prefix}" dof="5"/>
     </xacro:if>
     <!-- add one world link if no 'attach_to' specified  -->

File: xarm_description/urdf/xarm6/xarm6_robot_macro.xacro (robot description, xacro)
@@ -12,5 +12,5 @@
     <xacro:if value="${load_gazebo_plugin}">
     <xacro:include filename="$(find xarm_description)/urdf/common/common.gazebo.xacro" />
-    <xacro:gazebo_ros_control_plugin namespace="${namespace}"/>
+    <xacro:gazebo_ros_control_plugin  prefix="${prefix}" dof="6"/>
     </xacro:if>
     <!-- add one world link if no 'attach_to' specified  -->

File: xarm_description/urdf/xarm7/xarm7_robot_macro.xacro (robot description, xacro)
@@ -12,5 +12,5 @@
     <xacro:if value="${load_gazebo_plugin}">
     <xacro:include filename="$(find xarm_description)/urdf/common/common.gazebo.xacro" />
-    <xacro:gazebo_ros_control_plugin namespace="${namespace}"/>
+    <xacro:gazebo_ros_control_plugin  prefix="${prefix}" dof="7"/>
     </xacro:if>
     <!-- add one world link if no 'attach_to' specified  -->

File: xarm_description/urdf/xarm_device.urdf.xacro (robot description, xacro)
@@ -1,4 +1,4 @@
 <?xml version='1.0' encoding='utf-8'?>
-<robot xmlns:xacro="http://ros.org/wiki/xacro" name="xarm">
+<robot xmlns:xacro="http://ros.org/wiki/xacro" name="xarm$(arg dof)">
   <xacro:arg name="prefix" default=""/>
   <xacro:arg name="hw_ns" default="xarm"/>

File: xarm_moveit_config/srdf/dual_xarm.srdf.xacro (robot description, xacro)
@@ -1,4 +1,4 @@
 <?xml version="1.0" encoding="UTF-8"?>
-<robot xmlns:xacro="http://wiki.ros.org/xacro" name="xarm5_srdf">
+<robot xmlns:xacro="http://wiki.ros.org/xacro" name="dual_xarm">
   <!-- parameters -->
   <xacro:arg name="prefix_1" default="L_" />

File: xarm_moveit_config/srdf/xarm.srdf.xacro (robot description, xacro)
@@ -1,4 +1,4 @@
 <?xml version="1.0" encoding="UTF-8"?>
-<robot xmlns:xacro="http://wiki.ros.org/xacro" name="xarm5_srdf">
+<robot xmlns:xacro="http://wiki.ros.org/xacro" name="xarm$(arg dof)">
   <!-- parameters -->
   <xacro:arg name="add_gripper" default="false"/>

Commit message: Separate xarm/gripper parameters, automatically combine parameters to use

File: xarm_description/urdf/common/common.gazebo.xacro (robot description, xacro)
@@ -1,9 +1,11 @@
 <?xml version="1.0"?>
 <robot xmlns:xacro="http://ros.org/wiki/xacro">
-  <xacro:macro name="gazebo_ros_control_plugin" params="prefix:='' dof:=7">
+  <xacro:macro name="gazebo_ros_control_plugin" params="prefix:='' ros2_control_params:=''">
     <gazebo>
       <plugin filename="libgazebo_ros2_control.so" name="gazebo_ros2_control">
         <robot_sim_type>gazebo_ros2_control/GazeboSystem</robot_sim_type>
-        <parameters>$(find xarm_controller)/config/xarm${dof}_controllers.yaml</parameters>
+        <xacro:if value="${ros2_control_params != ''}">
+          <parameters>${ros2_control_params}</parameters>
+        </xacro:if>
       </plugin>
     </gazebo>

File: xarm_description/urdf/dual_xarm_device.urdf.xacro (robot description, xacro)
@@ -13,15 +13,17 @@
   <xacro:arg name="effort_control" default="false"/>
   <xacro:arg name="velocity_control" default="false"/>
-  <!-- <xacro:arg name="add_gripper" default="false"/>
-  <xacro:arg name="add_vacuum_gripper" default="false"/>
-  <xacro:arg name="dof" default="7"/> -->
   <xacro:arg name="ros2_control_plugin" default="xarm_control/XArmHW"/>
+  <xacro:arg name="ros2_control_params" default="$(find xarm_controller)/config/xarm$(arg dof_1)_controllers.yaml"/>
   <!-- load xarm device -->
   <xacro:include filename="$(find xarm_description)/urdf/xarm_device_macro.xacro" />
   <link name="ground" />
+  <!-- gazebo_plugin -->
+  <xacro:include filename="$(find xarm_description)/urdf/common/common.gazebo.xacro" />
+  <xacro:gazebo_ros_control_plugin ros2_control_params="$(arg ros2_control_params)"/>
   <xacro:xarm_device prefix="$(arg prefix_1)" namespace="$(arg hw_ns)" limited="$(arg limited)"
     effort_control="$(arg effort_control)" velocity_control="$(arg velocity_control)"
     add_gripper="$(arg add_gripper_1)" add_vacuum_gripper="$(arg add_vacuum_gripper_1)" dof="$(arg dof_1)"
     ros2_control_plugin="$(arg ros2_control_plugin)"
+    load_gazebo_plugin="false" ros2_control_params="$(arg ros2_control_params)"
     attach_to="ground" xyz="0 0 0" rpy="0 0 0" />
   <xacro:xarm_device prefix="$(arg prefix_2)" namespace="$(arg hw_ns)" limited="$(arg limited)"
@@ -29,4 +31,5 @@
     add_gripper="$(arg add_gripper_2)" add_vacuum_gripper="$(arg add_vacuum_gripper_2)" dof="$(arg dof_2)"
     ros2_control_plugin="$(arg ros2_control_plugin)"
+    load_gazebo_plugin="false" ros2_control_params="$(arg ros2_control_params)"
     attach_to="ground" xyz="0 1 0" rpy="0 0 0" />
 </robot>

File: xarm_description/urdf/gripper/xarm_gripper_model.xacro (robot description, xacro)
@@ -1,7 +1,4 @@
 <?xml version="1.0"?>
-<robot xmlns:xacro="http://ros.org/wiki/xacro"
-       name="xarm_gripper" >
-  <!-- common stuff -->
-  <xacro:include filename="$(find xarm_description)/urdf/common/common.gazebo.xacro" />
+<robot xmlns:xacro="http://ros.org/wiki/xacro" name="xarm_gripper" >
   <!-- xarm_gripper -->
   <xacro:include filename="$(find xarm_description)/urdf/gripper/xarm_gripper.ros2_control.xacro" />
@@ -9,8 +6,14 @@
   <xacro:include filename="$(find xarm_description)/urdf/gripper/xarm_gripper.transmission.xacro" />
   <xacro:include filename="$(find xarm_description)/urdf/gripper/xarm_gripper.gazebo.xacro" />
-  <xacro:macro name="load_gripper" params="prefix:='' attach_to:='' ns:='xarm' xyz:='0 0 0' rpy:='0 0 0' effort_control:='false' velocity_control:='false' ros2_control_plugin:='xarm_control/FakeXArmHW' ">
-    <!-- gazebo plugin -->
-    <!-- <xacro:gazebo_ros_control_plugin namespace="${ns}"/> -->
-    <xacro:xarm_gripper_ros2_control prefix="${prefix}" ros2_control_plugin="${ros2_control_plugin}" />
+  <xacro:macro name="load_gripper" params="prefix:='' attach_to:='' ns:='xarm' xyz:='0 0 0' rpy:='0 0 0' effort_control:='false' velocity_control:='false'
+    load_gazebo_plugin:='false' ros2_control_plugin:='xarm_control/FakeXArmHW' ros2_control_params:='' ">
+    <!-- gazebo_plugin -->
+    <xacro:if value="${load_gazebo_plugin}">
+      <xacro:include filename="$(find xarm_description)/urdf/common/common.gazebo.xacro" />
+      <xacro:gazebo_ros_control_plugin prefix="${prefix}" ros2_control_params="${ros2_control_params}"/>
+    </xacro:if>
+    <xacro:if value="${ros2_control_plugin != 'xarm_control/XArmHW'}">
+      <xacro:xarm_gripper_ros2_control prefix="${prefix}" ros2_control_plugin="${ros2_control_plugin}" />
+    </xacro:if>
     <xacro:xarm_gripper_urdf prefix="${prefix}" attach_to="${attach_to}" xyz="${xyz}" rpy="${rpy}" />
     <xacro:xarm_gripper_transmission prefix="${prefix}" hard_interface="${'EffortJointInterface' if effort_control else 'VelocityJointInterface' if velocity_control else 'PositionJointInterface'}" />

File: xarm_description/urdf/xarm5/xarm5_robot_macro.xacro (robot description, xacro)
@@ -2,6 +2,6 @@
 <robot xmlns:xacro="http://ros.org/wiki/xacro" name="xarm5" >
   <xacro:macro name="xarm5_robot" params="prefix:='' namespace:='xarm' limited:='false' effort_control:='false'
-    velocity_control:='false' attach_to:='world' xyz:='0 0 0' rpy:='0 0 0' load_gazebo_plugin:='true'
-    ros2_control_plugin:='xarm_control/XArmHW' ">
+    velocity_control:='false' attach_to:='world' xyz:='0 0 0' rpy:='0 0 0' load_gazebo_plugin:='false'
+    ros2_control_plugin:='xarm_control/XArmHW' ros2_control_params:='' ">
     <!-- include xarm5 relative macros: -->
     <xacro:include filename="$(find xarm_description)/urdf/xarm5/xarm5.ros2_control.xacro" />
@@ -11,6 +11,6 @@
     <!-- gazebo_plugin -->
     <xacro:if value="${load_gazebo_plugin}">
-    <xacro:include filename="$(find xarm_description)/urdf/common/common.gazebo.xacro" />
-    <xacro:gazebo_ros_control_plugin prefix="${prefix}" dof="5"/>
+      <xacro:include filename="$(find xarm_description)/urdf/common/common.gazebo.xacro" />
+      <xacro:gazebo_ros_control_plugin prefix="${prefix}" ros2_control_params="${ros2_control_params}"/>
     </xacro:if>
     <!-- add one world link if no 'attach_to' specified  -->

File: xarm_description/urdf/xarm6/xarm6_robot_macro.xacro (robot description, xacro)
@@ -2,6 +2,6 @@
 <robot xmlns:xacro="http://ros.org/wiki/xacro" name="xarm6" >
   <xacro:macro name="xarm6_robot" params="prefix:='' namespace:='xarm' limited:='false' effort_control:='false'
-    velocity_control:='false' attach_to:='world' xyz:='0 0 0' rpy:='0 0 0' load_gazebo_plugin:='true'
-    ros2_control_plugin:='xarm_control/XArmHW' ">
+    velocity_control:='false' attach_to:='world' xyz:='0 0 0' rpy:='0 0 0' load_gazebo_plugin:='false'
+    ros2_control_plugin:='xarm_control/XArmHW' ros2_control_params:='' ">
     <!-- include xarm6 relative macros: -->
     <xacro:include filename="$(find xarm_description)/urdf/xarm6/xarm6.ros2_control.xacro" />
@@ -11,6 +11,6 @@
     <!-- gazebo_plugin -->
     <xacro:if value="${load_gazebo_plugin}">
-    <xacro:include filename="$(find xarm_description)/urdf/common/common.gazebo.xacro" />
-    <xacro:gazebo_ros_control_plugin  prefix="${prefix}" dof="6"/>
+      <xacro:include filename="$(find xarm_description)/urdf/common/common.gazebo.xacro" />
+      <xacro:gazebo_ros_control_plugin  prefix="${prefix}" ros2_control_params="${ros2_control_params}"/>
     </xacro:if>
     <!-- add one world link if no 'attach_to' specified  -->

File: xarm_description/urdf/xarm7/xarm7_robot_macro.xacro (robot description, xacro)
@@ -2,6 +2,6 @@
 <robot xmlns:xacro="http://ros.org/wiki/xacro" name="xarm7" >
   <xacro:macro name="xarm7_robot" params="prefix:='' namespace:='xarm' limited:='false' effort_control:='false'
-    velocity_control:='false' attach_to:='world' xyz:='0 0 0' rpy:='0 0 0' load_gazebo_plugin:='true'
-    ros2_control_plugin:='xarm_control/XArmHW' ">
+    velocity_control:='false' attach_to:='world' xyz:='0 0 0' rpy:='0 0 0' load_gazebo_plugin:='false'
+    ros2_control_plugin:='xarm_control/XArmHW' ros2_control_params:='' ">
     <!-- xarm7 -->
     <xacro:include filename="$(find xarm_description)/urdf/xarm7/xarm7.ros2_control.xacro" />
@@ -11,6 +11,6 @@
     <!-- gazebo_plugin -->
     <xacro:if value="${load_gazebo_plugin}">
-    <xacro:include filename="$(find xarm_description)/urdf/common/common.gazebo.xacro" />
-    <xacro:gazebo_ros_control_plugin  prefix="${prefix}" dof="7"/>
+      <xacro:include filename="$(find xarm_description)/urdf/common/common.gazebo.xacro" />
+      <xacro:gazebo_ros_control_plugin  prefix="${prefix}" ros2_control_params="${ros2_control_params}"/>
     </xacro:if>
     <!-- add one world link if no 'attach_to' specified  -->

File: xarm_description/urdf/xarm_device.urdf.xacro (robot description, xacro)
@@ -10,4 +10,8 @@
   <xacro:arg name="dof" default="7"/>
   <xacro:arg name="ros2_control_plugin" default="xarm_control/XArmHW"/>
+  <xacro:arg name="ros2_control_params" default="$(find xarm_controller)/config/xarm$(arg dof)_controllers.yaml"/>
+  <!-- gazebo_plugin -->
+  <xacro:include filename="$(find xarm_description)/urdf/common/common.gazebo.xacro" />
+  <xacro:gazebo_ros_control_plugin ros2_control_params="$(arg ros2_control_params)"/>
   <!-- load xarm device -->
   <xacro:include filename="$(find xarm_description)/urdf/xarm_device_macro.xacro" />
@@ -15,4 +19,5 @@
     effort_control="$(arg effort_control)" velocity_control="$(arg velocity_control)"
     add_gripper="$(arg add_gripper)" add_vacuum_gripper="$(arg add_vacuum_gripper)" dof="$(arg dof)"
-    ros2_control_plugin="$(arg ros2_control_plugin)"/>
+    ros2_control_plugin="$(arg ros2_control_plugin)"
+    load_gazebo_plugin="false" ros2_control_params="$(arg ros2_control_params)"/>
 </robot>

File: xarm_description/urdf/xarm_device_macro.xacro (robot description, xacro)
@@ -3,5 +3,5 @@
   <xacro:macro name="xarm_device" params="prefix:='' namespace:='xarm' limited:='false' effort_control:='false'
     velocity_control:='false' add_gripper:='false' add_vacuum_gripper:='false' dof:=7 ros2_control_plugin:='xarm_control/XArmHW'
-    attach_to:='world' xyz:='0 0 0' rpy:='0 0 0' ">
+    attach_to:='world' xyz:='0 0 0' rpy:='0 0 0' ros2_control_params:='' load_gazebo_plugin:='false' ">
     <xacro:if value="${dof == 5}">
       <xacro:include filename="$(find xarm_description)/urdf/xarm5/xarm5_robot_macro.xacro" />
@@ -9,5 +9,7 @@
         effort_control="${effort_control}" velocity_control="${velocity_control}"
         ros2_control_plugin="${ros2_control_plugin}"
-        attach_to="${attach_to}" xyz="${xyz}" rpy="${rpy}" />
+        attach_to="${attach_to}" xyz="${xyz}" rpy="${rpy}"
+        ros2_control_params="${ros2_control_params}"
+        load_gazebo_plugin="${load_gazebo_plugin}" />
     </xacro:if>
     <xacro:if value="${dof == 6}">
@@ -16,5 +18,7 @@
         effort_control="${effort_control}" velocity_control="${velocity_control}"
         ros2_control_plugin="${ros2_control_plugin}"
-        attach_to="${attach_to}" xyz="${xyz}" rpy="${rpy}" />
+        attach_to="${attach_to}" xyz="${xyz}" rpy="${rpy}"
+        ros2_control_params="${ros2_control_params}"
+        load_gazebo_plugin="${load_gazebo_plugin}" />
     </xacro:if>
     <xacro:unless value="${dof == 5 or dof == 6}">
@@ -23,9 +27,13 @@
         effort_control="${effort_control}" velocity_control="${velocity_control}"
         ros2_control_plugin="${ros2_control_plugin}"
-        attach_to="${attach_to}" xyz="${xyz}" rpy="${rpy}" />
+        attach_to="${attach_to}" xyz="${xyz}" rpy="${rpy}"
+        ros2_control_params="${ros2_control_params}"
+        load_gazebo_plugin="${load_gazebo_plugin}" />
     </xacro:unless>
     <xacro:if value="${add_gripper}">
       <xacro:include filename="$(find xarm_description)/urdf/gripper/xarm_gripper_model.xacro" />
-      <xacro:load_gripper prefix="${prefix}" attach_to="${prefix}link_eef" effort_control="${effort_control}" velocity_control="${velocity_control}" ros2_control_plugin="${ros2_control_plugin}" />
+      <xacro:load_gripper prefix="${prefix}" attach_to="${prefix}link_eef" effort_control="${effort_control}" velocity_control="${velocity_control}"
+        ros2_control_plugin="${ros2_control_plugin}" ros2_control_params="${ros2_control_params}"
+        load_gazebo_plugin="${load_gazebo_plugin}" />
     </xacro:if>
     <xacro:if value="${add_vacuum_gripper}">
