Commit message: Refactor launch files for xArm configurations
- Removed unused LaunchConfiguration variables from xarm6 and xarm7 launch files to simplify the code.
- Updated the launch file paths for robot moveit gazebo launches to use the new naming convention.
- Added missing dependencies in package.xml files for xarm_moveit_config, xarm_msgs, and xarm_sdk.
- Introduced new message type MoveVelocity.msg for joint and cartesian velocity commands.
- Enhanced VacuumGripperCtrl.srv to include a sync parameter and hardware_version for better control.
- Enabled external program execution in RViz configuration files for improved functionality.
- Updated submodule reference for xarm_sdk/cxx to the latest commit.

File: xarm_description/urdf/common/common.link.xacro (robot description, xacro)
@@ -24,5 +24,5 @@
     </xacro:unless>
   </xacro:macro>
-  <xacro:macro name="common_link_visual" params="mesh_filename add_mesh_suffix:=true material_name:='White' origin_xyz:='0 0 0' origin_rpy:='0 0 0'">
+  <xacro:macro name="common_link_visual" params="mesh_filename add_mesh_suffix:=true material_name:='White' origin_xyz:='0 0 0' origin_rpy:='0 0 0' other_mesh_suffix:=''">
     <visual>
       <geometry>
@@ -31,5 +31,10 @@
         </xacro:if>
         <xacro:unless value="${add_mesh_suffix}">
-          <mesh filename="${mesh_path}/${mesh_filename}"/>
+          <xacro:if value="${other_mesh_suffix != ''}">
+            <mesh filename="${mesh_path}/${mesh_filename}.${other_mesh_suffix}"/>
+          </xacro:if>
+          <xacro:unless value="${other_mesh_suffix != ''}">
+            <mesh filename="${mesh_path}/${mesh_filename}"/>
+          </xacro:unless>
         </xacro:unless>
       </geometry>
@@ -38,5 +43,5 @@
     </visual>
   </xacro:macro>
-  <xacro:macro name="common_link_collision" params="mesh_filename add_mesh_suffix:=true origin_xyz:='0 0 0' origin_rpy:='0 0 0'">
+  <xacro:macro name="common_link_collision" params="mesh_filename add_mesh_suffix:=true origin_xyz:='0 0 0' origin_rpy:='0 0 0' other_mesh_suffix:=''">
     <collision>
       <geometry>
@@ -45,5 +50,10 @@
         </xacro:if>
         <xacro:unless value="${add_mesh_suffix}">
-          <mesh filename="${mesh_path}/${mesh_filename}"/>
+          <xacro:if value="${other_mesh_suffix != ''}">
+            <mesh filename="${mesh_path}/${mesh_filename}.${other_mesh_suffix}"/>
+          </xacro:if>
+          <xacro:unless value="${other_mesh_suffix != ''}">
+            <mesh filename="${mesh_path}/${mesh_filename}"/>
+          </xacro:unless>
         </xacro:unless>
       </geometry>
@@ -75,5 +85,10 @@
     <xacro:property name="mass_type" value="-1" />
     <xacro:property name="model_type" value="-1" />
-    <xacro:property name="_model1300" value="${model1300}" />
+    <xacro:if value="${model1300}">
+      <xacro:property name="model_num" value="1300" />
+    </xacro:if>
+    <xacro:unless value="${model1300}">
+      <xacro:property name="model_num" value="-1" />
+    </xacro:unless>
     <!-- parse model_type and mass_type from robot_sn -->
     <xacro:if value="${robot_sn_len >= 14 and (robot_sn[0] == 'X' or robot_sn[0] == 'L' or robot_sn[0] == 'F')}">
@@ -102,5 +117,4 @@
         </xacro:if>
       </xacro:if>
-      <!-- <xacro:property name="model_type" value="${9 if robot_sn[0] == 'L' else 5 if robot_sn[1] == 'F' else 6 if robot_sn[1] == 'I' else 7 if robot_sn[1] == 'S' else -1}" /> -->
       <xacro:property name="model_num" value="${int(robot_sn[2:6])}" />
       <xacro:if value="${model_num == 1250}">
@@ -112,7 +126,4 @@
         <xacro:property name="mass_type" value="1" />
       </xacro:if>
-      <xacro:if value="${model_num >= 1300}">
-        <xacro:property name="_model1300" value="true" />
-      </xacro:if>
       <xacro:property name="is_num" value="${robot_sn[8] == '0' or robot_sn[8] == '1' or robot_sn[8] == '2' or robot_sn[8] == '3' or robot_sn[8] == '4' or robot_sn[8] == '5' or robot_sn[8] == '6' or robot_sn[8] == '7' or robot_sn[8] == '8' or robot_sn[8] == '9'}" />
       <xacro:if value="${is_num}">
@@ -123,8 +134,8 @@
       </xacro:unless>
       <xacro:property name="date_int" value="${int(date_str)}" />
-      <xacro:if value="${robot_sn[11] == 'B' or robot_sn[11] == 'L' or robot_sn[11] == 'X' or robot_sn[11] == 'D'}">
+      <xacro:if value="${robot_sn[11] == 'B' or robot_sn[11] == 'L' or robot_sn[11] == 'X' or robot_sn[11] == 'D' or robot_sn[11] == 'A'}">
         <xacro:property name="hd_type" value="${robot_sn[11]}" />
       </xacro:if>
-      <xacro:unless value="${robot_sn[11] == 'B' or robot_sn[11] == 'L' or robot_sn[11] == 'X' or robot_sn[11] == 'D'}">
+      <xacro:unless value="${robot_sn[11] == 'B' or robot_sn[11] == 'L' or robot_sn[11] == 'X' or robot_sn[11] == 'D' or robot_sn[11] == 'A'}">
         <xacro:if value="${robot_sn_len >= 16 and robot_sn[14] == '_'}">
           <xacro:property name="hd_type" value="${robot_sn[15]}" />
@@ -134,5 +145,4 @@
         </xacro:unless>
       </xacro:unless>
-      <!-- <xacro:property name="hd_type" value="${robot_sn[11] if robot_sn[11] == 'B' or robot_sn[11] == 'L' or robot_sn[11] == 'X' or robot_sn[11] == 'D' else robot_sn[15] if robot_sn_len >= 16 and robot_sn[14] == '_' else ''}" /> -->
       <xacro:if value="${hd_type == 'B'}">
         <xacro:if value="${date_int >= 2004}">
@@ -142,5 +152,4 @@
           <xacro:property name="mass_type" value="1" />
         </xacro:unless>
-        <!-- <xacro:property name="mass_type" value="${11 if date_int >= 2004 else 1}" /> -->
       </xacro:if>
       <xacro:unless value="${hd_type == 'B'}">
@@ -149,5 +158,5 @@
           <xacro:property name="mass_type" value="2" />
         </xacro:if>
-        <xacro:if value="${hd_type == 'X'}">
+        <xacro:if value="${hd_type == 'A'}">
           <xacro:property name="mass_type" value="3" />
         </xacro:if>
@@ -155,74 +164,82 @@
           <xacro:property name="mass_type" value="4" />
         </xacro:if>
-        <!-- <xacro:property name="mass_type" value="${2 if hd_type == 'L' else 3 if hd_type == 'X' else 4 if hd_type == 'D' else 1}" /> -->
-      </xacro:unless>
-    </xacro:if>
-    <!-- update xarm5 inertia params filename -->
-    <xacro:if value="${dof == 5}">
-      <xacro:if value="${model_type == 5}">
-        <xacro:if value="${mass_type == 1}">
-          <xacro:property name="inertial_params_filename" value="xarm5_type5_HT_BR"/>
-        </xacro:if>
-        <xacro:if value="${mass_type == 2}">
-          <xacro:property name="inertial_params_filename" value="xarm5_type5_HT_LD"/>
-        </xacro:if>
-        <xacro:if value="${mass_type == 11}">
-          <xacro:property name="inertial_params_filename" value="xarm5_type5_HT_BR2"/>
-        </xacro:if>
-      </xacro:if>
-    </xacro:if>
-    <xacro:if value="${dof == 6}">
-      <!-- update uf850 inertia params filename -->
-      <xacro:if value="${robot_type == 'uf850'}">
-        <xacro:if value="${model_type == 12}">
-          <xacro:property name="inertial_params_filename" value="xarm6_type12_HT_LDBR2"/>
-        </xacro:if>
-      </xacro:if>
-      <!-- update lite6 inertia params filename -->
-      <xacro:if value="${robot_type == 'lite'}">
-        <xacro:if value="${model_type == 9}">
-          <xacro:property name="inertial_params_filename" value="xarm6_type9_HT_BR2"/>
-        </xacro:if>
-      </xacro:if>
-      <!-- update xarm6 inertia params filename -->
-      <xacro:unless value="${robot_type == 'lite' or robot_type == 'uf850'}">
-        <xacro:if value="${model_type == 6}">
+      </xacro:unless>
+      <!-- update xarm5 inertia params filename -->
+      <xacro:if value="${dof == 5}">
+        <xacro:if value="${model_type == 5}">
           <xacro:if value="${mass_type == 1}">
-            <xacro:property name="inertial_params_filename" value="xarm6_type6_HT_BR"/>
+            <xacro:property name="inertial_params_filename" value="xarm5_type5_HT_BR"/>
           </xacro:if>
           <xacro:if value="${mass_type == 2}">
-            <xacro:property name="inertial_params_filename" value="xarm6_type6_HT_LD"/>
+            <xacro:property name="inertial_params_filename" value="xarm5_type5_HT_LD"/>
+          </xacro:if>
+          <xacro:if value="${mass_type == 3}">
+            <xacro:property name="inertial_params_filename" value="xarm5_type5_UJ_BR_2403"/>
           </xacro:if>
           <xacro:if value="${mass_type == 11}">
-            <xacro:property name="inertial_params_filename" value="xarm6_type6_HT_BR2"/>
-          </xacro:if>
-        </xacro:if>
-        <xacro:if value="${model_type == 8}">
-          <xacro:property name="inertial_params_filename" value="xarm6_type8_HT2_BR2"/>
-        </xacro:if>
-        <xacro:if value="${model_type == 11}">
-          <xacro:property name="inertial_params_filename" value="xarm6_type11_HT_LD"/>
-        </xacro:if>
-      </xacro:unless>
-    </xacro:if>
-    <!-- update xarm7 inertia params filename -->
-    <xacro:unless value="${dof == 5 or dof == 6}">
-      <xacro:if value="${model_type == 3}">
-        <xacro:property name="inertial_params_filename" value="xarm7_type3_YT_SP"/>
-      </xacro:if>
-      <xacro:if value="${model_type == 7}">
-        <xacro:if value="${mass_type == 1}">
-          <xacro:property name="inertial_params_filename" value="xarm7_type7_HT_BR"/>
-        </xacro:if>
-        <xacro:if value="${mass_type == 2}">
-          <xacro:property name="inertial_params_filename" value="xarm7_type7_HT_LD"/>
-        </xacro:if>
-        <xacro:if value="${mass_type == 11}">
-          <xacro:property name="inertial_params_filename" value="xarm7_type7_HT_BR2"/>
-        </xacro:if>
-      </xacro:if>
-    </xacro:unless>
+            <xacro:property name="inertial_params_filename" value="xarm5_type5_HT_BR2"/>
+          </xacro:if>
+        </xacro:if>
+      </xacro:if>
+      <xacro:if value="${dof == 6}">
+        <!-- update uf850 inertia params filename -->
+        <xacro:if value="${robot_type == 'uf850'}">
+          <xacro:if value="${model_type == 12}">
+            <xacro:property name="inertial_params_filename" value="xarm6_type12_HT_LDBR2"/>
+          </xacro:if>
+        </xacro:if>
+        <!-- update lite6 inertia params filename -->
+        <xacro:if value="${robot_type == 'lite'}">
+          <xacro:if value="${model_type == 9}">
+            <xacro:property name="inertial_params_filename" value="xarm6_type9_HT_BR2"/>
+          </xacro:if>
+        </xacro:if>
+        <!-- update xarm6 inertia params filename -->
+        <xacro:unless value="${robot_type == 'lite' or robot_type == 'uf850'}">
+          <xacro:if value="${model_type == 6}">
+            <xacro:if value="${mass_type == 1}">
+              <xacro:property name="inertial_params_filename" value="xarm6_type6_HT_BR"/>
+            </xacro:if>
+            <xacro:if value="${mass_type == 2}">
+              <xacro:property name="inertial_params_filename" value="xarm6_type6_HT_LD"/>
+            </xacro:if>
+            <xacro:if value="${mass_type == 3}">
+              <xacro:property name="inertial_params_filename" value="xarm6_type6_UJ_BR_2403"/>
+            </xacro:if>
+            <xacro:if value="${mass_type == 11}">
+              <xacro:property name="inertial_params_filename" value="xarm6_type6_HT_BR2"/>
+            </xacro:if>
+          </xacro:if>
+          <xacro:if value="${model_type == 8}">
+            <xacro:property name="inertial_params_filename" value="xarm6_type8_HT2_BR2"/>
+          </xacro:if>
+          <xacro:if value="${model_type == 11}">
+            <xacro:property name="inertial_params_filename" value="xarm6_type11_HT_LD"/>
+          </xacro:if>
+        </xacro:unless>
+      </xacro:if>
+      <!-- update xarm7 inertia params filename -->
+      <xacro:unless value="${dof == 5 or dof == 6}">
+        <xacro:if value="${model_type == 3}">
+          <xacro:property name="inertial_params_filename" value="xarm7_type3_YT_SP"/>
+        </xacro:if>
+        <xacro:if value="${model_type == 7}">
+          <xacro:if value="${mass_type == 1}">
+            <xacro:property name="inertial_params_filename" value="xarm7_type7_HT_BR"/>
+          </xacro:if>
+          <xacro:if value="${mass_type == 2}">
+            <xacro:property name="inertial_params_filename" value="xarm7_type7_HT_LD"/>
+          </xacro:if>
+          <xacro:if value="${mass_type == 3}">
+            <xacro:property name="inertial_params_filename" value="xarm7_type7_UJ_BR_2403"/>
+          </xacro:if>
+          <xacro:if value="${mass_type == 11}">
+            <xacro:property name="inertial_params_filename" value="xarm7_type7_HT_BR2"/>
+          </xacro:if>
+        </xacro:if>
+      </xacro:unless>
+    </xacro:if>
     <xacro:property name="scope_parent_inertial_params_filename" value="${inertial_params_filename}" scope="parent"/>
-    <xacro:property name="scope_parent_model1300" value="${_model1300}" scope="parent"/>
+    <xacro:property name="scope_parent_model_num" value="${model_num}" scope="parent"/>
   </xacro:macro>
 </robot>

File: xarm_description/urdf/gripper/bio_gripper.ros2_control.xacro (robot description, xacro)
@@ -3,5 +3,5 @@
   <xacro:macro name="bio_gripper_ros2_control" params="prefix:=''
     ros2_control_plugin:='uf_robot_hardware/UFRobotFakeSystemHardware' ">
-    <ros2_control name="XArmGripperSystem" type="system">
+    <ros2_control name="${prefix}BioGripperSystem" type="system">
       <hardware>
         <plugin>${ros2_control_plugin}</plugin>

File: xarm_description/urdf/uf850/uf850.ros2_control.xacro (robot description, xacro)
@@ -36,4 +36,8 @@
       </hardware>
       <joint name="${prefix}joint1">
+        <command_interface name="position">
+          <param name="min">${joint1_lower_limit}</param>
+          <param name="max">${joint1_upper_limit}</param>
+        </command_interface>
         <command_interface name="velocity">
           <param name="min">-3.14</param>
@@ -42,8 +46,11 @@
         <state_interface name="position"/>
         <state_interface name="velocity"/>
-        <param name="sim_init">0.0140666039660573</param>
         <!-- <state_interface name="effort"/> -->
       </joint>
       <joint name="${prefix}joint2">
+        <command_interface name="position">
+          <param name="min">${joint2_lower_limit}</param>
+          <param name="max">${joint2_upper_limit}</param>
+        </command_interface>
         <command_interface name="velocity">
           <param name="min">-3.14</param>
@@ -52,8 +59,11 @@
         <state_interface name="position"/>
         <state_interface name="velocity"/>
-        <param name="sim_init">0.32001715898513794</param>
         <!-- <state_interface name="effort"/> -->
       </joint>
       <joint name="${prefix}joint3">
+        <command_interface name="position">
+          <param name="min">${joint3_lower_limit}</param>
+          <param name="max">${joint3_upper_limit}</param>
+        </command_interface>
         <command_interface name="velocity">
           <param name="min">-3.14</param>
@@ -62,8 +72,11 @@
         <state_interface name="position"/>
         <state_interface name="velocity"/>
-        <param name="sim_init">-0.7825928926467896</param>
         <!-- <state_interface name="effort"/> -->
       </joint>
       <joint name="${prefix}joint4">
+        <command_interface name="position">
+          <param name="min">${joint4_lower_limit}</param>
+          <param name="max">${joint4_upper_limit}</param>
+        </command_interface>
         <command_interface name="velocity">
           <param name="min">-3.14</param>
@@ -72,8 +85,11 @@
         <state_interface name="position"/>
         <state_interface name="velocity"/>
-        <param name="sim_init">-0.06832542270421982</param>
         <!-- <state_interface name="effort"/> -->
       </joint>
       <joint name="${prefix}joint5">
+        <command_interface name="position">
+          <param name="min">${joint5_lower_limit}</param>
+          <param name="max">${joint5_upper_limit}</param>
+        </command_interface>
         <command_interface name="velocity">
           <param name="min">-3.14</param>
@@ -82,8 +98,11 @@
         <state_interface name="position"/>
         <state_interface name="velocity"/>
-        <param name="sim_init">-1.0955243110656738</param>
         <!-- <state_interface name="effort"/> -->
       </joint>
       <joint name="${prefix}joint6">
+        <command_interface name="position">
+          <param name="min">${joint6_lower_limit}</param>
+          <param name="max">${joint6_upper_limit}</param>
+        </command_interface>
         <command_interface name="velocity">
           <param name="min">-3.14</param>
@@ -92,5 +111,4 @@
         <state_interface name="position"/>
         <state_interface name="velocity"/>
-        <param name="sim_init">2.342494010925293</param>
         <!-- <state_interface name="effort"/> -->
       </joint>

File: xarm_description/urdf/uf850/uf850_robot_macro.xacro (robot description, xacro)
@@ -13,5 +13,5 @@
     baud_checkset:='true'
     default_gripper_baud:=2000000
-    model1300:=false
+    model_num:=0
     inertial_params_filename:=''
     kinematics_params_filename:=''
@@ -38,5 +38,5 @@
           joint4_lower_limit="${-pi*0.99}" joint4_upper_limit="${pi*0.99}"
           joint5_lower_limit="${-2.1642}" joint5_upper_limit="${2.1642}"
-          joint6_lower_limit="${-pi*1.99}" joint6_upper_limit="${pi*1.99}"/>
+          joint6_lower_limit="${-pi*0.99}" joint6_upper_limit="${pi*0.99}"/>
       </xacro:if>
       <xacro:uf850_urdf prefix="${prefix}"
@@ -46,6 +46,6 @@
         joint4_lower_limit="${-pi*0.99}" joint4_upper_limit="${pi*0.99}"
         joint5_lower_limit="${-2.1642}" joint5_upper_limit="${2.1642}"
-        joint6_lower_limit="${-pi*1.99}" joint6_upper_limit="${pi*1.99}"
-        model1300="${model1300}"
+        joint6_lower_limit="${-pi*0.99}" joint6_upper_limit="${pi*0.99}"
+        model_num="${model_num}"
         inertial_params_filename="${inertial_params_filename}"
         kinematics_params_filename="${kinematics_params_filename}"/>
@@ -59,5 +59,5 @@
           baud_checkset="${baud_checkset}" default_gripper_baud="${default_gripper_baud}" />
       </xacro:if>
-      <xacro:uf850_urdf prefix="${prefix}" model1300="${model1300}"
+      <xacro:uf850_urdf prefix="${prefix}" model_num="${model_num}"
         inertial_params_filename="${inertial_params_filename}"
         kinematics_params_filename="${kinematics_params_filename}"/>
