Commit message: Refactor launch files for xArm configurations
- Removed unused LaunchConfiguration variables from xarm6 and xarm7 launch files to simplify the code.
- Updated the launch file paths for robot moveit gazebo launches to use the new naming convention.
- Added missing dependencies in package.xml files for xarm_moveit_config, xarm_msgs, and xarm_sdk.
- Introduced new message type MoveVelocity.msg for joint and cartesian velocity commands.
- Enhanced VacuumGripperCtrl.srv to include a sync parameter and hardware_version for better control.
- Enabled external program execution in RViz configuration files for improved functionality.
- Updated submodule reference for xarm_sdk/cxx to the latest commit.

File: xarm_description/urdf/xarm6/xarm6.urdf.xacro (robot description, xacro)
@@ -8,15 +8,29 @@
     joint5_lower_limit:=${-1.69297}  joint5_upper_limit:=${pi}
     joint6_lower_limit:=${-2.0*pi}  joint6_upper_limit:=${2.0*pi}
-    model1300:=false
+    model_num:=0
     inertial_params_filename:='' kinematics_params_filename:='' "
     >
     <!-- define property -->
-    <xacro:if value="${model1300}">
-      <xacro:property name="end_tool_visual_filename" value="end_tool/visual/end_tool_1300"/>
-      <xacro:property name="end_tool_collision_filename" value="end_tool/collision/end_tool_1300"/>
+    <xacro:if value="${model_num >= 1305 and model_num != 1380}">
+      <xacro:property name="visual_dir" value="xarm6_1305/visual"/>
+      <xacro:property name="collision_dir" value="xarm6_1305/collision"/>
+      <xacro:property name="add_mesh_suffix" value="false"/>
+      <xacro:property name="collison_mesh_suffix" value="obj"/>
+      <xacro:property name="link6_visual" value="xarm6_1305/visual/link6"/>
+      <xacro:property name="link6_collision" value="xarm6_1305/collision/link6"/>
     </xacro:if>
-    <xacro:unless value="${model1300}">
-      <xacro:property name="end_tool_visual_filename" value="xarm6/visual/link6"/>
-      <xacro:property name="end_tool_collision_filename" value="end_tool/collision/end_tool"/>
+    <xacro:unless value="${model_num >= 1305 and model_num != 1380}">
+      <xacro:property name="visual_dir" value="xarm6/visual"/>
+      <xacro:property name="collision_dir" value="xarm6/visual"/>
+      <xacro:property name="add_mesh_suffix" value="true"/>
+      <xacro:property name="collison_mesh_suffix" value="stl"/>
+      <xacro:if value="${model_num >= 1300}">
+        <xacro:property name="link6_visual" value="end_tool/visual/end_tool_1300"/>
+        <xacro:property name="link6_collision" value="end_tool/collision/end_tool_1300"/>
+      </xacro:if>
+      <xacro:unless value="${model_num >= 1300}">
+        <xacro:property name="link6_visual" value="xarm6/visual/link6"/>
+        <xacro:property name="link6_collision" value="end_tool/collision/end_tool"/>
+      </xacro:unless>
     </xacro:unless>
     <!-- load params and define property -->
@@ -46,10 +60,12 @@
       </inertial>
       <xacro:common_link_visual
-        mesh_filename="xarm6/visual/link_base"
-        origin_xyz="0 0 0"
-        origin_rpy="0 0 0"
-        material_name="${prefix}White" />
-      <xacro:common_link_collision
-        mesh_filename="xarm6/visual/link_base"
+        mesh_filename="${visual_dir}/link_base"
+        origin_xyz="0 0 0"
+        origin_rpy="0 0 0"
+        material_name="${prefix}White" />
+      <xacro:common_link_collision
+        mesh_filename="${collision_dir}/link_base"
+        add_mesh_suffix="${add_mesh_suffix}"
+        other_mesh_suffix="${collison_mesh_suffix}"
         origin_xyz="0 0 0"
         origin_rpy="0 0 0" />
@@ -60,10 +76,12 @@
         origin_rpy="0 0 0"/>
       <xacro:common_link_visual
-        mesh_filename="xarm6/visual/link1"
-        origin_xyz="0 0 0"
-        origin_rpy="0 0 0"
-        material_name="${prefix}White" />
-      <xacro:common_link_collision
-        mesh_filename="xarm6/visual/link1"
+        mesh_filename="${visual_dir}/link1"
+        origin_xyz="0 0 0"
+        origin_rpy="0 0 0"
+        material_name="${prefix}White" />
+      <xacro:common_link_collision
+        mesh_filename="${collision_dir}/link1"
+        add_mesh_suffix="${add_mesh_suffix}"
+        other_mesh_suffix="${collison_mesh_suffix}"
         origin_xyz="0 0 0"
         origin_rpy="0 0 0" />
@@ -87,11 +105,13 @@
         origin_rpy="0 0 0"/>
       <xacro:common_link_visual
-        mesh_filename="xarm6/visual/link2"
-        origin_xyz="0 0 ${-kinematics_params['joint2']['y']}"
-        origin_rpy="0 0 0"
-        material_name="${prefix}White" />
-      <xacro:common_link_collision
-        mesh_filename="xarm6/visual/link2"
-        origin_xyz="0 0 ${-kinematics_params['joint2']['y']}"
+        mesh_filename="${visual_dir}/link2"
+        origin_xyz="0 0 0"
+        origin_rpy="0 0 0"
+        material_name="${prefix}White" />
+      <xacro:common_link_collision
+        mesh_filename="${collision_dir}/link2"
+        add_mesh_suffix="${add_mesh_suffix}"
+        other_mesh_suffix="${collison_mesh_suffix}"
+        origin_xyz="0 0 0"
         origin_rpy="0 0 0" />
     </link>
@@ -114,10 +134,12 @@
         origin_rpy="0 0 0"/>
       <xacro:common_link_visual
-        mesh_filename="xarm6/visual/link3"
-        origin_xyz="0 0 0"
-        origin_rpy="0 0 0"
-        material_name="${prefix}White" />
-      <xacro:common_link_collision
-        mesh_filename="xarm6/visual/link3"
+        mesh_filename="${visual_dir}/link3"
+        origin_xyz="0 0 0"
+        origin_rpy="0 0 0"
+        material_name="${prefix}White" />
+      <xacro:common_link_collision
+        mesh_filename="${collision_dir}/link3"
+        add_mesh_suffix="${add_mesh_suffix}"
+        other_mesh_suffix="${collison_mesh_suffix}"
         origin_xyz="0 0 0"
         origin_rpy="0 0 0" />
@@ -141,10 +163,12 @@
         origin_rpy="0 0 0"/>
       <xacro:common_link_visual
-        mesh_filename="xarm6/visual/link4"
-        origin_xyz="0 0 0"
-        origin_rpy="0 0 0"
-        material_name="${prefix}White" />
-      <xacro:common_link_collision
-        mesh_filename="xarm6/visual/link4"
+        mesh_filename="${visual_dir}/link4"
+        origin_xyz="0 0 0"
+        origin_rpy="0 0 0"
+        material_name="${prefix}White" />
+      <xacro:common_link_collision
+        mesh_filename="${collision_dir}/link4"
+        add_mesh_suffix="${add_mesh_suffix}"
+        other_mesh_suffix="${collison_mesh_suffix}"
         origin_xyz="0 0 0"
         origin_rpy="0 0 0" />
@@ -168,10 +192,12 @@
         origin_rpy="0 0 0"/>
       <xacro:common_link_visual
-        mesh_filename="xarm6/visual/link5"
-        origin_xyz="0 0 0"
-        origin_rpy="0 0 0"
-        material_name="${prefix}White" />
-      <xacro:common_link_collision
-        mesh_filename="xarm6/visual/link5"
+        mesh_filename="${visual_dir}/link5"
+        origin_xyz="0 0 0"
+        origin_rpy="0 0 0"
+        material_name="${prefix}White" />
+      <xacro:common_link_collision
+        mesh_filename="${collision_dir}/link5"
+        add_mesh_suffix="${add_mesh_suffix}"
+        other_mesh_suffix="${collison_mesh_suffix}"
         origin_xyz="0 0 0"
         origin_rpy="0 0 0" />
@@ -194,10 +220,12 @@
         origin_rpy="0 0 0"/>
       <xacro:common_link_visual
-        mesh_filename="${end_tool_visual_filename}"
+        mesh_filename="${link6_visual}"
         origin_xyz="0 0 0"
         origin_rpy="0 0 0"
         material_name="${prefix}Silver" />
       <xacro:common_link_collision
-        mesh_filename="${end_tool_collision_filename}"
+        mesh_filename="${link6_collision}"
+        add_mesh_suffix="${add_mesh_suffix}"
+        other_mesh_suffix="${collison_mesh_suffix}"
         origin_xyz="0 0 0"
         origin_rpy="0 0 0" />

File: xarm_description/urdf/xarm6/xarm6_robot_macro.xacro (robot description, xacro)
@@ -13,5 +13,5 @@
     baud_checkset:='true'
     default_gripper_baud:=2000000
-    model1300:=false
+    model_num:=0
     inertial_params_filename:=''
     kinematics_params_filename:=''
@@ -35,17 +35,17 @@
           joint1_lower_limit="${-pi*0.99}" joint1_upper_limit="${pi*0.99}"
           joint2_lower_limit="${-2.059}" joint2_upper_limit="${2.0944}"
-          joint3_lower_limit="${-3.83972435}" joint3_upper_limit="${0.19198}"
+          joint3_lower_limit="${-pi*0.99}" joint3_upper_limit="${0.19198}"
           joint4_lower_limit="${-pi*0.99}" joint4_upper_limit="${pi*0.99}"
           joint5_lower_limit="${-1.69297}" joint5_upper_limit="${pi*0.99}"
-          joint6_lower_limit="${-2*pi*0.99}" joint6_upper_limit="${2*pi*0.99}"/>
+          joint6_lower_limit="${-pi*0.99}" joint6_upper_limit="${pi*0.99}"/>
       </xacro:if>
       <xacro:xarm6_urdf prefix="${prefix}"
         joint1_lower_limit="${-pi*0.99}" joint1_upper_limit="${pi*0.99}"
         joint2_lower_limit="${-2.059}" joint2_upper_limit="${2.0944}"
-        joint3_lower_limit="${-3.83972435}" joint3_upper_limit="${0.19198}"
+        joint3_lower_limit="${-pi*0.99}" joint3_upper_limit="${0.19198}"
         joint4_lower_limit="${-pi*0.99}" joint4_upper_limit="${pi*0.99}"
         joint5_lower_limit="${-1.69297}" joint5_upper_limit="${pi*0.99}"
-        joint6_lower_limit="${-2*pi*0.99}" joint6_upper_limit="${2*pi*0.99}"
-        model1300="${model1300}"
+        joint6_lower_limit="${-pi*0.99}" joint6_upper_limit="${pi*0.99}"
+        model_num="${model_num}"
         inertial_params_filename="${inertial_params_filename}"
         kinematics_params_filename="${kinematics_params_filename}"
@@ -60,5 +60,5 @@
           baud_checkset="${baud_checkset}" default_gripper_baud="${default_gripper_baud}" />
       </xacro:if>
-      <xacro:xarm6_urdf prefix="${prefix}" model1300="${model1300}"
+      <xacro:xarm6_urdf prefix="${prefix}" model_num="${model_num}"
         inertial_params_filename="${inertial_params_filename}"
         kinematics_params_filename="${kinematics_params_filename}"

File: xarm_description/urdf/xarm_device_macro.xacro (robot description, xacro)
@@ -52,9 +52,9 @@
     <!-- Specify Mesh file path -->
     <xacro:property name="mesh_suffix" value="${mesh_suffix}" scope="parent"/>
-    <xacro:if value="${ros2_control_plugin == 'gazebo_ros2_control/GazeboSystem' or ros2_control_plugin == 'ign_ros2_control/IgnitionSystem'}">
+    <xacro:if value="${ros2_control_plugin == 'gazebo_ros2_control/GazeboSystem' or ros2_control_plugin == 'ign_ros2_control/IgnitionSystem' or ros2_control_plugin == 'gz_ros2_control/GazeboSimSystem'}">
       <!-- gazebo use -->
       <xacro:property name="mesh_path" value="file://$(find xarm_description)/meshes" scope="parent"/>
     </xacro:if>
-    <xacro:unless value="${ros2_control_plugin == 'gazebo_ros2_control/GazeboSystem' or ros2_control_plugin == 'ign_ros2_control/IgnitionSystem'}">
+    <xacro:unless value="${ros2_control_plugin == 'gazebo_ros2_control/GazeboSystem' or ros2_control_plugin == 'ign_ros2_control/IgnitionSystem' or ros2_control_plugin == 'gz_ros2_control/GazeboSimSystem'}">
       <xacro:property name="mesh_path" value="package://xarm_description/meshes" scope="parent"/>
     </xacro:unless>
@@ -63,5 +63,6 @@
     <xacro:parse_link_inertial_filename dof="${dof}" robot_type="${robot_type}" robot_sn="${robot_sn}" model1300="${model1300}" />
     <xacro:property name="inertial_params_filename" value="${scope_parent_inertial_params_filename}"/>
-    <xacro:property name="new_model1300" value="${scope_parent_model1300}"/>
+    <xacro:property name="model_num" value="${scope_parent_model_num}"/>
+    <!-- Print the model number for debugging -->
     <!-- add one world link if no 'attach_to' specified  -->
     <xacro:if value="${attach_to == 'world' and create_attach_link}">
@@ -91,5 +92,5 @@
     </xacro:unless>
     <xacro:if value="${kinematics_suffix != ''}">
-      <xacro:property name="kinematics_params_filename" value="/shared/${robot_name}_kinematics_${kinematics_suffix}.yaml"/>
+      <xacro:property name="kinematics_params_filename" value="$(find xarm_description)/config/kinematics/user/${robot_name}_kinematics_${kinematics_suffix}.yaml"/>
     </xacro:if>
     <xacro:unless value="${kinematics_suffix != ''}">
@@ -108,5 +109,5 @@
         baud_checkset="${baud_checkset}"
         default_gripper_baud="${default_gripper_baud}"
-        model1300="${new_model1300}"
+        model_num="${model_num}"
         inertial_params_filename="${inertial_params_filename}"
         kinematics_params_filename="${kinematics_params_filename}"
@@ -126,5 +127,5 @@
           baud_checkset="${baud_checkset}"
           default_gripper_baud="${default_gripper_baud}"
-          model1300="${new_model1300}"
+          model_num="${model_num}"
           inertial_params_filename="${inertial_params_filename}"
           kinematics_params_filename="${kinematics_params_filename}"
@@ -142,4 +143,5 @@
           baud_checkset="${baud_checkset}"
           default_gripper_baud="${default_gripper_baud}"
+          model_num="${model_num}"
           inertial_params_filename="${inertial_params_filename}"
           kinematics_params_filename="${kinematics_params_filename}"
@@ -158,5 +160,5 @@
           baud_checkset="${baud_checkset}"
           default_gripper_baud="${default_gripper_baud}"
-          model1300="${new_model1300}"
+          model_num="${model_num}"
           inertial_params_filename="${inertial_params_filename}"
           kinematics_params_filename="${kinematics_params_filename}"
@@ -177,5 +179,5 @@
           baud_checkset="${baud_checkset}"
           default_gripper_baud="${default_gripper_baud}"
-          model1300="${new_model1300}"
+          model_num="${model_num}"
           inertial_params_filename="${inertial_params_filename}"
           kinematics_params_filename="${kinematics_params_filename}"
@@ -194,5 +196,5 @@
           baud_checkset="${baud_checkset}"
           default_gripper_baud="${default_gripper_baud}"
-          model1300="${new_model1300}"
+          model_num="${model_num}"
           inertial_params_filename="${inertial_params_filename}"
           kinematics_params_filename="${kinematics_params_filename}"
@@ -275,10 +277,13 @@
           <xacro:property name="new_ros2_control_params" value="${ros2_control_params}"/>
         </xacro:if>
+        <xacro:if value="${ros2_control_plugin == 'gz_ros2_control/GazeboSimSystem'}">
+          <xacro:gz_ros2_control_plugin ros2_control_params="${new_ros2_control_params}"/>
+        </xacro:if>
         <xacro:if value="${ros2_control_plugin == 'ign_ros2_control/IgnitionSystem'}">
           <xacro:ignition_ros2_control_plugin prefix="${prefix}" ros2_control_params="${new_ros2_control_params}"/>
         </xacro:if>
-        <xacro:unless value="${ros2_control_plugin == 'ign_ros2_control/IgnitionSystem'}">
+        <xacro:if value="${ros2_control_plugin == 'gazebo_ros2_control/GazeboSystem'}">
           <xacro:gazebo_ros2_control_plugin ros2_control_params="${new_ros2_control_params}"/>
-        </xacro:unless>
+        </xacro:if>
       </xacro:if>
       <xacro:unless value="${is_ros2}">
