Commit message: Feat: xarm_moveit_config/xarm_gazebo package support lite5
1. add parameter 'robot_type' to support lite6

File: xarm_moveit_config/srdf/dual_xarm.srdf.xacro (robot description, xacro)
@@ -6,4 +6,6 @@
   <xacro:arg name="dof_1" default="7" />
   <xacro:arg name="dof_2" default="7" />
+  <xacro:arg name="robot_type_1" default="xarm" />
+  <xacro:arg name="robot_type_2" default="xarm" />
   <xacro:arg name="add_gripper_1" default="false" />
   <xacro:arg name="add_gripper_2" default="false" />
@@ -13,7 +15,7 @@
   <xacro:arg name="add_other_geometry_2" default="false" />
   <xacro:include filename="$(find xarm_moveit_config)/srdf/xarm_macro.srdf.xacro" />
-  <xacro:xarm_macro_srdf prefix="$(arg prefix_1)" dof="$(arg dof_1)"
+  <xacro:xarm_macro_srdf prefix="$(arg prefix_1)" dof="$(arg dof_1)" robot_type="$(arg robot_type_1)"
     add_gripper="$(arg add_gripper_1)" add_vacuum_gripper="$(arg add_vacuum_gripper_1)" add_other_geometry="$(arg add_other_geometry_1)" />
-  <xacro:xarm_macro_srdf prefix="$(arg prefix_2)" dof="$(arg dof_2)"
+  <xacro:xarm_macro_srdf prefix="$(arg prefix_2)" dof="$(arg dof_2)" robot_type="$(arg robot_type_2)"
     add_gripper="$(arg add_gripper_2)" add_vacuum_gripper="$(arg add_vacuum_gripper_2)" add_other_geometry="$(arg add_other_geometry_2)" />
 </robot>

File: xarm_moveit_config/srdf/xarm.srdf.xacro (robot description, xacro)
@@ -1,12 +1,13 @@
 <?xml version="1.0" encoding="UTF-8"?>
-<robot xmlns:xacro="http://wiki.ros.org/xacro" name="xarm$(arg dof)">
+<robot xmlns:xacro="http://wiki.ros.org/xacro" name="$(arg robot_type)$(arg dof)">
   <!-- parameters -->
   <xacro:arg name="prefix" default="" />
   <xacro:arg name="dof" default="7" />
+  <xacro:arg name="robot_type" default="xarm" />
   <xacro:arg name="add_gripper" default="false"/>
   <xacro:arg name="add_vacuum_gripper" default="false" />
   <xacro:arg name="add_other_geometry" default="false" />
   <xacro:include filename="$(find xarm_moveit_config)/srdf/xarm_macro.srdf.xacro" />
-  <xacro:xarm_macro_srdf prefix="$(arg prefix)" dof="$(arg dof)"
+  <xacro:xarm_macro_srdf prefix="$(arg prefix)" dof="$(arg dof)" robot_type="$(arg robot_type)"
     add_gripper="$(arg add_gripper)" add_vacuum_gripper="$(arg add_vacuum_gripper)" add_other_geometry="$(arg add_other_geometry)" />
 </robot>

File: xarm_moveit_config/srdf/xarm_macro.srdf.xacro (robot description, xacro)
@@ -1,5 +1,5 @@
 <?xml version="1.0" encoding="UTF-8"?>
 <robot xmlns:xacro="http://wiki.ros.org/xacro" name="xarm_srdf">
-  <xacro:macro name="xarm_macro_srdf" params="prefix:='' dof:=7
+  <xacro:macro name="xarm_macro_srdf" params="prefix:='' dof:=7 robot_type:='xarm'
     add_gripper:='false' add_vacuum_gripper:='false' add_other_geometry:='false' ">
     <xacro:if value="${dof == 5}">
@@ -9,7 +9,14 @@
     </xacro:if>
     <xacro:if value="${dof == 6}">
-      <xacro:include filename="$(find xarm_moveit_config)/srdf/_xarm6_macro.srdf.xacro" />
-      <xacro:xarm6_macro_srdf prefix="${prefix}"
-        add_gripper="${add_gripper}" add_vacuum_gripper="${add_vacuum_gripper}" add_other_geometry="${add_other_geometry}"  />
+      <xacro:if value="${robot_type == 'lite'}">
+        <xacro:include filename="$(find xarm_moveit_config)/srdf/_lite6_macro.srdf.xacro" />
+        <xacro:lite6_macro_srdf prefix="${prefix}"
+          add_gripper="${add_gripper}" add_vacuum_gripper="${add_vacuum_gripper}" add_other_geometry="${add_other_geometry}"  />
+      </xacro:if>
+      <xacro:unless value="${robot_type == 'lite'}">
+        <xacro:include filename="$(find xarm_moveit_config)/srdf/_xarm6_macro.srdf.xacro" />
+        <xacro:xarm6_macro_srdf prefix="${prefix}"
+          add_gripper="${add_gripper}" add_vacuum_gripper="${add_vacuum_gripper}" add_other_geometry="${add_other_geometry}"  />
+      </xacro:unless>
     </xacro:if>
     <xacro:unless value="${dof == 5 or dof == 6}">
