Commit message: [fix] fix group hold-up of uf850

File: xarm_moveit_config/srdf/_uf850_macro.srdf.xacro (robot description, xacro)
@@ -52,5 +52,5 @@
       <joint name="${prefix}joint3" value="0" />
       <joint name="${prefix}joint4" value="0" />
-      <joint name="${prefix}joint5" value="-1.5708" />
+      <joint name="${prefix}joint5" value="1.5708" />
       <joint name="${prefix}joint6" value="0" />
     </group_state>
