Commit message: [Fix] fix ros2_control name

File: xarm_description/urdf/xarm6/xarm6.urdf.xacro (robot description, xacro)
@@ -37,13 +37,13 @@
       </collision>
       <inertial>
-      <origin xyz="0.0 0.0 0.09103" rpy="0 0 0" />
-      <mass value="2.7" />
-      <inertia
-        ixx="0.00494875"
-        ixy="-3.5E-06"
-        ixz="1.25E-05"
-        iyy="0.00494174"
-        iyz="1.67E-06"
-        izz="0.002219" />
+        <origin xyz="0.0 0.0 0.09103" rpy="0 0 0" />
+        <mass value="2.7" />
+        <inertia
+          ixx="0.00494875"
+          ixy="-3.5E-06"
+          ixz="1.25E-05"
+          iyy="0.00494174"
+          iyz="1.67E-06"
+          izz="0.002219" />
       </inertial>
     </link>

File: xarm_description/urdf/xarm7/xarm7.urdf.xacro (robot description, xacro)
@@ -22,38 +22,38 @@
     </material>
     <link
-    name="${prefix}link_base">
-    <inertial>
-      <origin
-        xyz="-0.021131 -0.0016302 0.056488"
-        rpy="0 0 0" />
-      <mass
-        value="0.88556" />
-      <inertia
-        ixx="0.0030595"
-        ixy="0.00012259"
-        ixz="-0.00062705"
-        iyy="0.0037783"
-        iyz="0.00027023"
-        izz="0.0020125" />
-    </inertial>
-    <visual>
-      <origin
-        xyz="0 0 0"
-        rpy="0 0 0" />
-      <geometry>
-        <!-- <mesh filename="package://xarm_description/meshes/xarm7/visual/link_base.STL" /> -->
-        <mesh filename="file:///$(find xarm_description)/meshes/xarm7/visual/link_base.STL"/>
-      </geometry>
-      <material name="${prefix}White" />
-    </visual>
-    <collision>
-      <origin
-        xyz="0 0 0"
-        rpy="0 0 0" />
-      <geometry>
-        <!-- <mesh filename="package://xarm_description/meshes/xarm7/visual/link_base.STL" /> -->
-        <mesh filename="file:///$(find xarm_description)/meshes/xarm7/visual/link_base.STL"/>
-      </geometry>
-    </collision>
+      name="${prefix}link_base">
+      <inertial>
+        <origin
+          xyz="-0.021131 -0.0016302 0.056488"
+          rpy="0 0 0" />
+        <mass
+          value="0.88556" />
+        <inertia
+          ixx="0.0030595"
+          ixy="0.00012259"
+          ixz="-0.00062705"
+          iyy="0.0037783"
+          iyz="0.00027023"
+          izz="0.0020125" />
+      </inertial>
+      <visual>
+        <origin
+          xyz="0 0 0"
+          rpy="0 0 0" />
+        <geometry>
+          <!-- <mesh filename="package://xarm_description/meshes/xarm7/visual/link_base.STL" /> -->
+          <mesh filename="file:///$(find xarm_description)/meshes/xarm7/visual/link_base.STL"/>
+        </geometry>
+        <material name="${prefix}White" />
+      </visual>
+      <collision>
+        <origin
+          xyz="0 0 0"
+          rpy="0 0 0" />
+        <geometry>
+          <!-- <mesh filename="package://xarm_description/meshes/xarm7/visual/link_base.STL" /> -->
+          <mesh filename="file:///$(find xarm_description)/meshes/xarm7/visual/link_base.STL"/>
+        </geometry>
+      </collision>
     </link>
     <link
