Commit message: [Feat] add the model of realsense D435i camera to the end
1. Support D435i simulation in gazebo
2. Integrate third-party plugin (realsense_gazebo_plugin)

File: xarm_description/urdf/dual_xarm_device.urdf.xacro (robot description, xacro)
@@ -17,4 +17,6 @@
   <xacro:arg name="ros2_control_plugin" default="uf_robot_hardware/UFRobotSystemHardware"/>
   <xacro:arg name="ros2_control_params" default="$(find xarm_controller)/config/xarm$(arg dof_1)_controllers.yaml"/>
+  <xacro:arg name="add_realsense_d435i_1" default="false"/>
+  <xacro:arg name="add_realsense_d435i_2" default="false"/>
   <xacro:arg name="add_other_geometry_1" default="false"/>
   <xacro:arg name="geometry_type_1" default="box"/>
@@ -61,4 +63,5 @@
     load_gazebo_plugin="false" ros2_control_params="$(arg ros2_control_params)"
     attach_to="ground" xyz="0 0 0" rpy="0 0 0"
+    add_realsense_d435i="$(arg add_realsense_d435i_1)"
     add_other_geometry="$(arg add_other_geometry_1)"
     geometry_type="$(arg geometry_type_1)" geometry_mass="$(arg geometry_mass_1)"
@@ -77,4 +80,5 @@
     load_gazebo_plugin="false" ros2_control_params="$(arg ros2_control_params)"
     attach_to="ground" xyz="0 1 0" rpy="0 0 0"
+    add_realsense_d435i="$(arg add_realsense_d435i_2)"
     add_other_geometry="$(arg add_other_geometry_2)"
     geometry_type="$(arg geometry_type_2)" geometry_mass="$(arg geometry_mass_2)"

File: xarm_description/urdf/lite6/lite6.urdf.xacro (robot description, xacro)
@@ -347,5 +347,5 @@
       <dynamics damping="1.0" friction="1.0"/>
     </joint>
-    <link name="${prefix}link_eef" />
+    <!-- <link name="${prefix}link_eef" />
     <joint
       name="${prefix}joint_eef"
@@ -358,5 +358,5 @@
       <child
         link="${prefix}link_eef" />
-    </joint>
+    </joint> -->
   </xacro:macro>
 </robot>

File: xarm_description/urdf/xarm5/xarm5.urdf.xacro (robot description, xacro)
@@ -340,16 +340,16 @@
         friction="1" />
     </joint>
-  <link name="${prefix}link_eef" />
-  <joint
-    name="${prefix}joint_eef"
-    type="fixed">
-    <origin
-      xyz="0 0 0"
-      rpy="0 0 0" />
-    <parent
-      link="${prefix}link5" />
-    <child
-      link="${prefix}link_eef" />
-  </joint>
+    <!-- <link name="${prefix}link_eef" />
+    <joint
+      name="${prefix}joint_eef"
+      type="fixed">
+      <origin
+        xyz="0 0 0"
+        rpy="0 0 0" />
+      <parent
+        link="${prefix}link5" />
+      <child
+        link="${prefix}link_eef" />
+    </joint> -->
   </xacro:macro>
 </robot>

File: xarm_description/urdf/xarm6/xarm6.urdf.xacro (robot description, xacro)
@@ -105,17 +105,17 @@
       </collision>
       <inertial>
-      <origin
-        xyz="0.03531 -0.21398 0.03386"
-        rpy="0 0 0" />
-      <mass
-        value="1.71" />
-      <inertia
-        ixx="0.0248674"
-        ixy="-0.00430651"
-        ixz="-0.00067797"
-        iyy="0.00485548"
-        iyz="0.00457245"
-        izz="0.02387827" />
-    </inertial>
+        <origin
+          xyz="0.03531 -0.21398 0.03386"
+          rpy="0 0 0" />
+        <mass
+          value="1.71" />
+        <inertia
+          ixx="0.0248674"
+          ixy="-0.00430651"
+          ixz="-0.00067797"
+          iyy="0.00485548"
+          iyz="0.00457245"
+          izz="0.02387827" />
+      </inertial>
     </link>
     <joint name="${prefix}joint2" type="revolute">
@@ -148,17 +148,17 @@
       </collision>
       <inertial>
-      <origin
-        xyz="0.06781 0.10749 0.01457"
-        rpy="0 0 0" />
-      <mass
-        value="1.384" />
-      <inertia
-        ixx="0.0053694"
-        ixy="0.0014185"
-        ixz="-0.00092094"
-        iyy="0.0032423"
-        iyz="-0.00169178"
-        izz="0.00501731" />
-    </inertial>
+        <origin
+          xyz="0.06781 0.10749 0.01457"
+          rpy="0 0 0" />
+        <mass
+          value="1.384" />
+        <inertia
+          ixx="0.0053694"
+          ixy="0.0014185"
+          ixz="-0.00092094"
+          iyy="0.0032423"
+          iyz="-0.00169178"
+          izz="0.00501731" />
+      </inertial>
     </link>
     <joint name="${prefix}joint3" type="revolute">
@@ -231,17 +231,17 @@
       </collision>
       <inertial>
-      <origin
-        xyz="0.05428 0.01781 0.00543"
-        rpy="0 0 0" />
-      <mass
-        value="1.275" />
-      <inertia
-        ixx="0.001202758"
-        ixy="0.000492428"
-        ixz="-0.00039147"
-        iyy="0.0022876"
-        iyz="-1.235E-04"
-        izz="0.0026866" />
-    </inertial>
+        <origin
+          xyz="0.05428 0.01781 0.00543"
+          rpy="0 0 0" />
+        <mass
+          value="1.275" />
+        <inertia
+          ixx="0.001202758"
+          ixy="0.000492428"
+          ixz="-0.00039147"
+          iyy="0.0022876"
+          iyz="-1.235E-04"
+          izz="0.0026866" />
+      </inertial>
     </link>
     <joint name="${prefix}joint5" type="revolute">
@@ -274,17 +274,17 @@
       </collision>
       <inertial>
-      <origin
-        xyz="0 0.00064 -0.00952"
-        rpy="0 0 0" />
-      <mass
-        value="0.1096" />
-      <inertia
-        ixx="4.5293E-05"
-        ixy="0"
-        ixz="0"
-        iyy="4.8111E-05"
-        iyz="0"
-        izz="7.9715E-05" />
-    </inertial>
+        <origin
+          xyz="0 0.00064 -0.00952"
+          rpy="0 0 0" />
+        <mass
+          value="0.1096" />
+        <inertia
+          ixx="4.5293E-05"
+          ixy="0"
+          ixz="0"
+          iyy="4.8111E-05"
+          iyz="0"
+          izz="7.9715E-05" />
+      </inertial>
     </link>
     <joint name="${prefix}joint6" type="revolute">
@@ -300,16 +300,16 @@
       <dynamics damping="1.0" friction="1.0"/>
     </joint>
-  <link name="${prefix}link_eef" />
-  <joint
-    name="${prefix}joint_eef"
-    type="fixed">
-    <origin
-      xyz="0 0 0"
-      rpy="0 0 0" />
-    <parent
-      link="${prefix}link6" />
-    <child
-      link="${prefix}link_eef" />
-  </joint>
+    <!-- <link name="${prefix}link_eef" />
+    <joint
+      name="${prefix}joint_eef"
+      type="fixed">
+      <origin
+        xyz="0 0 0"
+        rpy="0 0 0" />
+      <parent
+        link="${prefix}link6" />
+      <child
+        link="${prefix}link_eef" />
+    </joint> -->
   </xacro:macro>
 </robot>

File: xarm_description/urdf/xarm7/xarm7.urdf.xacro (robot description, xacro)
@@ -56,416 +56,416 @@
       </geometry>
     </collision>
-  </link>
-  <link
-    name="${prefix}link1">
-    <inertial>
-      <origin
-        xyz="-0.0042142 0.02821 -0.0087788"
+    </link>
+    <link
+      name="${prefix}link1">
+      <inertial>
+        <origin
+          xyz="-0.0042142 0.02821 -0.0087788"
+          rpy="0 0 0" />
+        <mass
+          value="0.42603" />
+        <inertia
+          ixx="0.0014243"
+          ixy="3.9946E-05"
+          ixz="4.7078E-06"
+          iyy="0.00123"
+          iyz="-0.00026073"
+          izz="0.00099229" />
+      </inertial>
+      <visual>
+        <origin
+          xyz="0 0 0"
+          rpy="0 0 0" />
+        <geometry>
+          <!-- <mesh filename="package://xarm_description/meshes/xarm7/visual/link1.STL" /> -->
+          <mesh filename="file:///$(find xarm_description)/meshes/xarm7/visual/link1.STL"/>
+        </geometry>
+        <material name="${prefix}White" />
+      </visual>
+      <collision>
+        <origin
+          xyz="0 0 0"
+          rpy="0 0 0" />
+        <geometry>
+          <!-- <mesh filename="package://xarm_description/meshes/xarm7/visual/link1.STL" /> -->
+          <mesh filename="file:///$(find xarm_description)/meshes/xarm7/visual/link1.STL"/>
+        </geometry>
+      </collision>
+    </link>
+    <joint
+      name="${prefix}joint1"
+      type="revolute">
+      <origin
+        xyz="0 0 0.267"
         rpy="0 0 0" />
-      <mass
-        value="0.42603" />
-      <inertia
-        ixx="0.0014243"
-        ixy="3.9946E-05"
-        ixz="4.7078E-06"
-        iyy="0.00123"
-        iyz="-0.00026073"
-        izz="0.00099229" />
-    </inertial>
-    <visual>
+      <parent
+        link="${prefix}link_base" />
+      <child
+        link="${prefix}link1" />
+      <axis
+        xyz="0 0 1" />
+      <limit
+        lower="${joint1_lower_limit}"
+        upper="${joint1_upper_limit}"
+        effort="50"
+        velocity="3.14" />
+      <dynamics
+        damping="10"
+        friction="1" />
+    </joint>
+    <link
+      name="${prefix}link2">
+      <inertial>
+        <origin
+          xyz="-3.3178E-05 -0.12849 0.026337"
+          rpy="0 0 0" />
+        <mass
+          value="0.56095" />
+        <inertia
+          ixx="0.0031915"
+          ixy="3.0892E-06"
+          ixz="2.8729E-06"
+          iyy="0.0017468"
+          iyz="-0.0010241"
+          izz="0.00235" />
+      </inertial>
+      <visual>
+        <origin
+          xyz="0 0 0"
+          rpy="0 0 0" />
+        <geometry>
+          <!-- <mesh filename="package://xarm_description/meshes/xarm7/visual/link2.STL" /> -->
+          <mesh filename="file:///$(find xarm_description)/meshes/xarm7/visual/link2.STL"/>
+        </geometry>
+        <material name="${prefix}White" />
+      </visual>
+      <collision>
+        <origin
+          xyz="0 0 0"
+          rpy="0 0 0" />
+        <geometry>
+          <!-- <mesh filename="package://xarm_description/meshes/xarm7/visual/link2.STL" /> -->
+          <mesh filename="file:///$(find xarm_description)/meshes/xarm7/visual/link2.STL"/>
+        </geometry>
+      </collision>
+    </link>
+    <joint
+      name="${prefix}joint2"
+      type="revolute">
+      <origin
+        xyz="0 0 0"
+        rpy="-1.5708 0 0" />
+      <parent
+        link="${prefix}link1" />
+      <child
+        link="${prefix}link2" />
+      <axis
+        xyz="0 0 1" />
+      <limit
+        lower="${joint2_lower_limit}"
+        upper="${joint2_upper_limit}"
+        effort="50"
+        velocity="3.14" />
+      <dynamics
+        damping="10"
+        friction="1" />
+    </joint>
+    <link
+      name="${prefix}link3">
+      <inertial>
+        <origin
+          xyz="0.04223 -0.023258 -0.0096674"
+          rpy="0 0 0" />
+        <mass
+          value="0.44463" />
+        <inertia
+          ixx="0.0011454"
+          ixy="0.0001654"
+          ixz="-0.0001951"
+          iyy="0.0010503"
+          iyz="0.00012027"
+          izz="0.0011083" />
+      </inertial>
+      <visual>
+        <origin
+          xyz="0 0 0"
+          rpy="0 0 0" />
+        <geometry>
+          <!-- <mesh filename="package://xarm_description/meshes/xarm7/visual/link3.STL" /> -->
+          <mesh filename="file:///$(find xarm_description)/meshes/xarm7/visual/link3.STL"/>
+        </geometry>
+        <material name="${prefix}White" />
+      </visual>
+      <collision>
+        <origin
+          xyz="0 0 0"
+          rpy="0 0 0" />
+        <geometry>
+          <!-- <mesh filename="package://xarm_description/meshes/xarm7/visual/link3.STL" /> -->
+          <mesh filename="file:///$(find xarm_description)/meshes/xarm7/visual/link3.STL"/>
+        </geometry>
+      </collision>
+    </link>
+    <joint
+      name="${prefix}joint3"
+      type="revolute">
+      <origin
+        xyz="0 -0.293 0"
+        rpy="1.5708 0 0" />
+      <parent
+        link="${prefix}link2" />
+      <child
+        link="${prefix}link3" />
+      <axis
+        xyz="0 0 1" />
+      <limit
+        lower="${joint3_lower_limit}"
+        upper="${joint3_upper_limit}"
+        effort="30"
+        velocity="3.14" />
+      <dynamics
+        damping="5"
+        friction="1" />
+    </joint>
+    <link
+      name="${prefix}link4">
+      <inertial>
+        <origin
+          xyz="0.067148 -0.10732 0.024479"
+          rpy="0 0 0" />
+        <mass
+          value="0.52387" />
+        <inertia
+          ixx="0.0026033"
+          ixy="0.00053379"
+          ixz="0.00036314"
+          iyy="0.0017649"
+          iyz="-0.00083253"
+          izz="0.0022431" />
+      </inertial>
+      <visual>
+        <origin
+          xyz="0 0 0"
+          rpy="0 0 0" />
+        <geometry>
+          <!-- <mesh filename="package://xarm_description/meshes/xarm7/visual/link4.STL" /> -->
+          <mesh filename="file:///$(find xarm_description)/meshes/xarm7/visual/link4.STL"/>
+        </geometry>
+        <material name="${prefix}White" />
+      </visual>
+      <collision>
+        <origin
+          xyz="0 0 0"
+          rpy="0 0 0" />
+        <geometry>
+          <!-- <mesh filename="package://xarm_description/meshes/xarm7/visual/link4.STL" /> -->
+          <mesh filename="file:///$(find xarm_description)/meshes/xarm7/visual/link4.STL"/>
+        </geometry>
+      </collision>
+    </link>
+    <joint
+      name="${prefix}joint4"
+      type="revolute">
+      <origin
+        xyz="0.0525 0 0"
+        rpy="1.5708 0 0" />
+      <parent
+        link="${prefix}link3" />
+      <child
+        link="${prefix}link4" />
+      <axis
+        xyz="0 0 1" />
+      <limit
+        lower="${joint4_lower_limit}"
+        upper="${joint4_upper_limit}"
+        effort="30"
+        velocity="3.14" />
+      <dynamics
+        damping="5"
+        friction="1" />
+    </joint>
+    <link
+      name="${prefix}link5">
+      <inertial>
+        <origin
+          xyz="-0.00023397 0.036705 -0.080064"
+          rpy="0 0 0" />
+        <mass
+          value="0.18554" />
+        <inertia
+          ixx="0.00099549"
+          ixy="8.9957E-07"
+          ixz="8.5285E-07"
+          iyy="0.0008853"
+          iyz="-0.00025682"
+          izz="0.00035048" />
+      </inertial>
+      <visual>
+        <origin
+          xyz="0 0 0"
+          rpy="0 0 0" />
+        <geometry>
+          <!-- <mesh filename="package://xarm_description/meshes/xarm7/visual/link5.STL" /> -->
+          <mesh filename="file:///$(find xarm_description)/meshes/xarm7/visual/link5.STL"/>
+        </geometry>
+        <material name="${prefix}White" />
+      </visual>
+      <collision>
+        <origin
+          xyz="0 0 0"
+          rpy="0 0 0" />
+        <geometry>
+          <!-- <mesh filename="package://xarm_description/meshes/xarm7/visual/link5.STL" /> -->
+          <mesh filename="file:///$(find xarm_description)/meshes/xarm7/visual/link5.STL"/>
+        </geometry>
+      </collision>
+    </link>
+    <joint
+      name="${prefix}joint5"
+      type="revolute">
+      <origin
+        xyz="0.0775 -0.3425 0"
+        rpy="1.5708 0 0" />
+      <parent
+        link="${prefix}link4" />
+      <child
+        link="${prefix}link5" />
+      <axis
+        xyz="0 0 1" />
+      <limit
+        lower="${joint5_lower_limit}"
+        upper="${joint5_upper_limit}"
+        effort="30"
+        velocity="3.14" />
+      <dynamics
+        damping="5"
+        friction="1" />
+    </joint>
+    <link
+      name="${prefix}link6">
+      <inertial>
+        <origin
+          xyz="0.058911 0.028469 0.0068428"
+          rpy="0 0 0" />
+        <mass
+          value="0.31344" />
+        <inertia
+          ixx="0.00052034"
+          ixy="-0.00014989"
+          ixz="0.00011658"
+          iyy="0.00067968"
+          iyz="6.116E-05"
+          izz="0.00078345" />
+      </inertial>
+      <visual>
+        <origin
+          xyz="0 0 0"
+          rpy="0 0 0" />
+        <geometry>
+          <!-- <mesh filename="package://xarm_description/meshes/xarm7/visual/link6.STL" /> -->
+          <mesh filename="file:///$(find xarm_description)/meshes/xarm7/visual/link6.STL"/>
+        </geometry>
+        <material name="${prefix}White" />
+      </visual>
+      <collision>
+        <origin
+          xyz="0 0 0"
+          rpy="0 0 0" />
+        <geometry>
+          <!-- <mesh filename="package://xarm_description/meshes/xarm7/visual/link6.STL" /> -->
+          <mesh filename="file:///$(find xarm_description)/meshes/xarm7/visual/link6.STL"/>
+        </geometry>
+      </collision>
+    </link>
+    <joint
+      name="${prefix}joint6"
+      type="revolute">
+      <origin
+        xyz="0 0 0"
+        rpy="1.5708 0 0" />
+      <parent
+        link="${prefix}link5" />
+      <child
+        link="${prefix}link6" />
+      <axis
+        xyz="0 0 1" />
+      <limit
+        lower="${joint6_lower_limit}"
+        upper="${joint6_upper_limit}"
+        effort="20"
+        velocity="3.14" />
+      <dynamics
+        damping="2"
+        friction="1" />
+    </joint>
+    <link
+      name="${prefix}link7">
+      <inertial>
+        <origin
+          xyz="-1.5846E-05 -0.0046377 -0.012705"
+          rpy="0 0 0" />
+        <mass
+          value="0.31468" />
+        <inertia
+          ixx="0.00016985"
+          ixy="1.1102E-07"
+          ixz="5.1075E-08"
+          iyy="0.00011924"
+          iyz="-2.1251E-06"
+          izz="0.00026032" />
+      </inertial>
+      <visual>
+        <origin
+          xyz="0 0 0"
+          rpy="0 0 0" />
+        <geometry>
+          <!-- <mesh filename="package://xarm_description/meshes/xarm7/visual/link7.STL" /> -->
+          <mesh filename="file:///$(find xarm_description)/meshes/xarm7/visual/link7.STL"/>
+        </geometry>
+        <material name="${prefix}Silver" />
+      </visual>
+      <collision>
+        <origin
+          xyz="0 0 0"
+          rpy="0 0 0" />
+        <geometry>
+          <!-- <mesh filename="package://xarm_description/meshes/xarm7/visual/link7.STL" /> -->
+          <mesh filename="file:///$(find xarm_description)/meshes/xarm7/visual/link7.STL"/>
+        </geometry>
+      </collision>
+    </link>
+    <joint
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
File: xarm_description/urdf/xarm_device.urdf.xacro (robot description, xacro)
@@ -12,4 +12,5 @@
   <xacro:arg name="ros2_control_plugin" default="uf_robot_hardware/UFRobotSystemHardware"/>
   <xacro:arg name="ros2_control_params" default="$(find xarm_controller)/config/xarm$(arg dof)_controllers.yaml"/>
+  <xacro:arg name="add_realsense_d435i" default="false"/>
   <xacro:arg name="add_other_geometry" default="false"/>
   <xacro:arg name="geometry_type" default="box"/>
@@ -38,4 +39,5 @@
     ros2_control_plugin="$(arg ros2_control_plugin)" robot_type="$(arg robot_type)"
     load_gazebo_plugin="false" ros2_control_params="$(arg ros2_control_params)"
+    add_realsense_d435i="$(arg add_realsense_d435i)"
     add_other_geometry="$(arg add_other_geometry)"
     geometry_type="$(arg geometry_type)" geometry_mass="$(arg geometry_mass)"

File: xarm_description/urdf/xarm_device_macro.xacro (robot description, xacro)
@@ -4,4 +4,5 @@
     velocity_control:='false' add_gripper:='false' add_vacuum_gripper:='false' dof:=7 robot_type:='xarm' ros2_control_plugin:='uf_robot_hardware/UFRobotSystemHardware'
     attach_to:='world' xyz:='0 0 0' rpy:='0 0 0' ros2_control_params:='' load_gazebo_plugin:='false'
+    add_realsense_d435i:='false'
     add_other_geometry:='false'
     geometry_type:='box' geometry_mass:='0.1'
@@ -78,4 +79,18 @@
         default_gripper_baud="${default_gripper_baud}" />
     </xacro:unless>
+    <xacro:if value="${robot_type != 'lite' and add_realsense_d435i}">
+      <xacro:include filename="$(find xarm_description)/urdf/camera/realsense_d435i.urdf.xacro" />
+      <xacro:d435i_urdf prefix="${prefix}"/>
+      <xacro:include filename="$(find xarm_description)/urdf/camera/realsense.gazebo.xacro" />
+      <xacro:realsense_gazebo prefix="$(arg prefix)" />
+    </xacro:if>
+    <xacro:unless value="${add_realsense_d435i}">
+      <link name="${prefix}link_eef"/>
+    </xacro:unless>
+    <joint name="${prefix}joint_eef" type="fixed">
+      <origin xyz="0 0 0" rpy="0 0 0" />
+      <parent link="${prefix}link${dof}" />
+      <child link="${prefix}link_eef" />
+    </joint>
     <xacro:if value="${add_gripper}">
       <xacro:if value="${robot_type == 'lite'}">
