Commit message: [feat] add launch parameter `model1300` to replace the end model
1. add launch parameter `model1300` to replace the model of the end of xarm robot arm with the 1300 series

File: xarm_description/urdf/dual_xarm_device.urdf.xacro (robot description, xacro)
@@ -51,4 +51,6 @@
   <xacro:arg name="default_gripper_baud_1" default="2000000"/>
   <xacro:arg name="default_gripper_baud_2" default="2000000"/>
+  <xacro:arg name="model1300_1" default="false"/>
+  <xacro:arg name="model1300_2" default="false"/>
   <!-- load xarm device -->
   <xacro:include filename="$(find xarm_description)/urdf/xarm_device_macro.xacro" />
@@ -73,5 +75,5 @@
     robot_ip="$(arg robot_ip_1)" report_type="$(arg report_type_1)"
     baud_checkset="$(arg baud_checkset_1)" default_gripper_baud="$(arg default_gripper_baud_1)"
-    />
+    model1300="$(arg model1300_1)"/>
   <xacro:xarm_device prefix="$(arg prefix_2)" namespace="$(arg hw_ns)" limited="$(arg limited)"
     effort_control="$(arg effort_control)" velocity_control="$(arg velocity_control)"
@@ -90,4 +92,4 @@
     robot_ip="$(arg robot_ip_2)" report_type="$(arg report_type_2)"
     baud_checkset="$(arg baud_checkset_2)" default_gripper_baud="$(arg default_gripper_baud_2)"
-    />
+    model1300="$(arg model1300_2)"/>
 </robot>

File: xarm_description/urdf/xarm5/xarm5.urdf.xacro (robot description, xacro)
@@ -6,5 +6,6 @@
     joint3_lower_limit:=${-3.927}  joint3_upper_limit:=${0.19198}
     joint4_lower_limit:=${-1.69297}  joint4_upper_limit:=${pi}
-    joint5_lower_limit:=${-2.0*pi}  joint5_upper_limit:=${2.0*pi}">
+    joint5_lower_limit:=${-2.0*pi}  joint5_upper_limit:=${2.0*pi}
+    model1300:=false">
     <material name="${prefix}Black">
       <color rgba="0.0 0.0 0.0 1.0"/>
@@ -305,5 +306,10 @@
         <geometry>
           <!-- <mesh filename="package://xarm_description/meshes/xarm5/visual/link5.STL" /> -->
-          <mesh filename="file:///$(find xarm_description)/meshes/xarm5/visual/link5.STL"/>
+          <xacro:if value="${model1300}">
+            <mesh filename="file:///$(find xarm_description)/meshes/end_tool/visual/end_tool_1300.STL"/>
+          </xacro:if>
+          <xacro:unless value="${model1300}">
+            <mesh filename="file:///$(find xarm_description)/meshes/xarm5/visual/link5.STL"/>
+          </xacro:unless>
         </geometry>
         <material name="${prefix}Silver" />
@@ -315,5 +321,10 @@
         <geometry>
           <!-- <mesh filename="package://xarm_description/meshes/xarm5/visual/link5.STL" /> -->
-          <mesh filename="file:///$(find xarm_description)/meshes/xarm5/visual/link5.STL"/>
+          <xacro:if value="${model1300}">
+            <mesh filename="file:///$(find xarm_description)/meshes/end_tool/collision/end_tool_1300.STL"/>
+          </xacro:if>
+          <xacro:unless value="${model1300}">
+            <mesh filename="file:///$(find xarm_description)/meshes/end_tool/collision/end_tool.STL"/>
+          </xacro:unless>
         </geometry>
       </collision>

File: xarm_description/urdf/xarm5/xarm5_robot_macro.xacro (robot description, xacro)
@@ -4,5 +4,6 @@
     velocity_control:='false' attach_to:='world' xyz:='0 0 0' rpy:='0 0 0' load_gazebo_plugin:='false'
     ros2_control_plugin:='uf_robot_hardware/UFRobotSystemHardware' ros2_control_params:='' add_gripper:='false'
-    robot_ip:='' report_type:='normal' baud_checkset:='true' default_gripper_baud:=2000000 ">
+    robot_ip:='' report_type:='normal' baud_checkset:='true' default_gripper_baud:=2000000
+    model1300:='false' ">
     <!-- include xarm5 relative macros: -->
     <xacro:include filename="$(find xarm_description)/urdf/xarm5/xarm5.ros2_control.xacro" />
@@ -41,5 +42,6 @@
         joint3_lower_limit="${-pi*0.99}" joint3_upper_limit="${0.19198}"
         joint4_lower_limit="${-1.69297}" joint4_upper_limit="${pi*0.99}"
-        joint5_lower_limit="${-pi*0.99}" joint5_upper_limit="${pi*0.99}"/>
+        joint5_lower_limit="${-pi*0.99}" joint5_upper_limit="${pi*0.99}"
+        model1300="${model1300}"/>
     </xacro:if>
     <xacro:unless value="${limited}">
@@ -49,5 +51,5 @@
         robot_ip="${robot_ip}" report_type="${report_type}"
         baud_checkset="${baud_checkset}" default_gripper_baud="${default_gripper_baud}" />
-      <xacro:xarm5_urdf prefix="${prefix}"/>
+      <xacro:xarm5_urdf prefix="${prefix}" model1300="${model1300}"/>
     </xacro:unless>
     <xacro:xarm5_transmission prefix="${prefix}" hard_interface="${'EffortJointInterface' if effort_control else 'VelocityJointInterface' if velocity_control else 'PositionJointInterface'}" />

File: xarm_description/urdf/xarm6/xarm6.urdf.xacro (robot description, xacro)
@@ -7,5 +7,6 @@
     joint4_lower_limit:=${-2.0*pi}  joint4_upper_limit:=${2.0*pi}
     joint5_lower_limit:=${-1.69297}  joint5_upper_limit:=${pi}
-    joint6_lower_limit:=${-2.0*pi}  joint6_upper_limit:=${2.0*pi}">
+    joint6_lower_limit:=${-2.0*pi}  joint6_upper_limit:=${2.0*pi}
+    model1300:=false">
     <material name="${prefix}Black">
       <color rgba="0.0 0.0 0.0 1.0"/>
@@ -261,5 +262,10 @@
         <geometry>
           <!-- <mesh filename="package://xarm_description/meshes/xarm6/visual/link6.stl"/> -->
-          <mesh filename="file:///$(find xarm_description)/meshes/xarm6/visual/link6.stl"/>
+          <xacro:if value="${model1300}">
+            <mesh filename="file:///$(find xarm_description)/meshes/end_tool/visual/end_tool_1300.STL"/>
+          </xacro:if>
+          <xacro:unless value="${model1300}">
+            <mesh filename="file:///$(find xarm_description)/meshes/xarm6/visual/link6.stl"/>
+          </xacro:unless>
         </geometry>
         <origin xyz="0 0 0" rpy="0 0 0"/>
@@ -269,5 +275,10 @@
         <geometry>
           <!-- <mesh filename="package://xarm_description/meshes/xarm6/visual/link6.stl"/> -->
-          <mesh filename="file:///$(find xarm_description)/meshes/xarm6/visual/link6.stl"/>
+          <xacro:if value="${model1300}">
+            <mesh filename="file:///$(find xarm_description)/meshes/end_tool/collision/end_tool_1300.STL"/>
+          </xacro:if>
+          <xacro:unless value="${model1300}">
+            <mesh filename="file:///$(find xarm_description)/meshes/end_tool/collision/end_tool.STL"/>
+          </xacro:unless>
         </geometry>
         <origin xyz="0 0 0" rpy="0 0 0"/>

File: xarm_description/urdf/xarm6/xarm6_robot_macro.xacro (robot description, xacro)
@@ -4,5 +4,6 @@
     velocity_control:='false' attach_to:='world' xyz:='0 0 0' rpy:='0 0 0' load_gazebo_plugin:='false'
     ros2_control_plugin:='uf_robot_hardware/UFRobotSystemHardware' ros2_control_params:='' add_gripper:='false'
-    robot_ip:='' report_type:='normal' baud_checkset:='true' default_gripper_baud:=2000000 ">
+    robot_ip:='' report_type:='normal' baud_checkset:='true' default_gripper_baud:=2000000
+    model1300:='false' ">
     <!-- include xarm6 relative macros: -->
     <xacro:include filename="$(find xarm_description)/urdf/xarm6/xarm6.ros2_control.xacro" />
@@ -43,5 +44,6 @@
         joint4_lower_limit="${-pi*0.99}" joint4_upper_limit="${pi*0.99}"
         joint5_lower_limit="${-1.69297}" joint5_upper_limit="${pi*0.99}"
-        joint6_lower_limit="${-pi*0.99}" joint6_upper_limit="${pi*0.99}"/>
+        joint6_lower_limit="${-pi*0.99}" joint6_upper_limit="${pi*0.99}"
+        model1300="${model1300}"/>
     </xacro:if>
     <xacro:unless value="${limited}">
@@ -51,5 +53,5 @@
         robot_ip="${robot_ip}" report_type="${report_type}"
         baud_checkset="${baud_checkset}" default_gripper_baud="${default_gripper_baud}" />
-      <xacro:xarm6_urdf prefix="${prefix}"/>
+      <xacro:xarm6_urdf prefix="${prefix}" model1300="${model1300}"/>
     </xacro:unless>
     <xacro:xarm6_transmission prefix="${prefix}" hard_interface="${'EffortJointInterface' if effort_control else 'VelocityJointInterface' if velocity_control else 'PositionJointInterface'}" />

File: xarm_description/urdf/xarm7/xarm7.urdf.xacro (robot description, xacro)
@@ -8,5 +8,6 @@
     joint5_lower_limit:=${-2.0*pi}  joint5_upper_limit:=${2.0*pi}
     joint6_lower_limit:=${-1.69297}  joint6_upper_limit:=${pi}
-    joint7_lower_limit:=${-2.0*pi}  joint7_upper_limit:=${2.0*pi}">
+    joint7_lower_limit:=${-2.0*pi}  joint7_upper_limit:=${2.0*pi}
+    model1300:=false">
     <material name="${prefix}Black">
       <color rgba="0.0 0.0 0.0 1.0"/>
@@ -421,5 +422,10 @@
         <geometry>
           <!-- <mesh filename="package://xarm_description/meshes/xarm7/visual/link7.STL" /> -->
-          <mesh filename="file:///$(find xarm_description)/meshes/xarm7/visual/link7.STL"/>
+          <xacro:if value="${model1300}">
+            <mesh filename="file:///$(find xarm_description)/meshes/end_tool/visual/end_tool_1300.STL"/>
+          </xacro:if>
+          <xacro:unless value="${model1300}">
+            <mesh filename="file:///$(find xarm_description)/meshes/xarm7/visual/link7.STL"/>
+          </xacro:unless>
         </geometry>
         <material name="${prefix}Silver" />
@@ -431,5 +437,10 @@
         <geometry>
           <!-- <mesh filename="package://xarm_description/meshes/xarm7/visual/link7.STL" /> -->
-          <mesh filename="file:///$(find xarm_description)/meshes/xarm7/visual/link7.STL"/>
+          <xacro:if value="${model1300}">
+            <mesh filename="file:///$(find xarm_description)/meshes/end_tool/collision/end_tool_1300.STL"/>
+          </xacro:if>
+          <xacro:unless value="${model1300}">
+            <mesh filename="file:///$(find xarm_description)/meshes/end_tool/collision/end_tool.STL"/>
+          </xacro:unless>
         </geometry>
       </collision>

File: xarm_description/urdf/xarm7/xarm7_robot_macro.xacro (robot description, xacro)
@@ -4,5 +4,6 @@
     velocity_control:='false' attach_to:='world' xyz:='0 0 0' rpy:='0 0 0' load_gazebo_plugin:='false'
     ros2_control_plugin:='uf_robot_hardware/UFRobotSystemHardware' ros2_control_params:='' add_gripper:='false'
-    robot_ip:='' report_type:='normal' baud_checkset:='true' default_gripper_baud:=2000000 ">
+    robot_ip:='' report_type:='normal' baud_checkset:='true' default_gripper_baud:=2000000
+    model1300:='false' ">
     <!-- xarm7 -->
     <xacro:include filename="$(find xarm_description)/urdf/xarm7/xarm7.ros2_control.xacro" />
@@ -45,5 +46,6 @@
         joint5_lower_limit="${-pi*0.99}" joint5_upper_limit="${pi*0.99}"
         joint6_lower_limit="${-1.75}" joint6_upper_limit="${pi*0.99}"
-        joint7_lower_limit="${-pi*0.99}" joint7_upper_limit="${pi*0.99}"/>
+        joint7_lower_limit="${-pi*0.99}" joint7_upper_limit="${pi*0.99}"
+        model1300="${model1300}"/>
     </xacro:if>
     <xacro:unless value="${limited}">
@@ -53,5 +55,5 @@
         robot_ip="${robot_ip}" report_type="${report_type}"
         baud_checkset="${baud_checkset}" default_gripper_baud="${default_gripper_baud}" />
-      <xacro:xarm7_urdf prefix="${prefix}"/>
+      <xacro:xarm7_urdf prefix="${prefix}" model1300="${model1300}"/>
     </xacro:unless>
     <xacro:xarm7_transmission prefix="${prefix}" hard_interface="${'EffortJointInterface' if effort_control else 'VelocityJointInterface' if velocity_control else 'PositionJointInterface'}" />

File: xarm_description/urdf/xarm_device.urdf.xacro (robot description, xacro)
@@ -29,4 +29,5 @@
   <xacro:arg name="baud_checkset" default="true"/>
   <xacro:arg name="default_gripper_baud" default="2000000"/>
+  <xacro:arg name="model1300" default="false"/>
   <!-- gazebo_plugin -->
   <xacro:include filename="$(find xarm_description)/urdf/common/common.gazebo.xacro" />
@@ -48,4 +49,5 @@
     geometry_mesh_tcp_xyz="$(arg geometry_mesh_tcp_xyz)" geometry_mesh_tcp_rpy="$(arg geometry_mesh_tcp_rpy)"
     robot_ip="$(arg robot_ip)" report_type="$(arg report_type)"
-    baud_checkset="$(arg baud_checkset)" default_gripper_baud="$(arg default_gripper_baud)"/>
+    baud_checkset="$(arg baud_checkset)" default_gripper_baud="$(arg default_gripper_baud)"
+    model1300="$(arg model1300)"/>
 </robot>

File: xarm_description/urdf/xarm_device_macro.xacro (robot description, xacro)
@@ -16,5 +16,6 @@
     robot_ip:='' report_type:='normal'
     baud_checkset:='true'
-    default_gripper_baud:=2000000 ">
+    default_gripper_baud:=2000000
+    model1300:='false'">
     <xacro:if value="${dof == 5}">
       <!-- Load XArm5 Robot Model URDF -->
@@ -30,5 +31,6 @@
         report_type="${report_type}"
         baud_checkset="${baud_checkset}"
-        default_gripper_baud="${default_gripper_baud}" />
+        default_gripper_baud="${default_gripper_baud}"
+        model1300="${model1300}" />
     </xacro:if>
     <xacro:if value="${dof == 6}">
@@ -61,5 +63,6 @@
           report_type="${report_type}"
           baud_checkset="${baud_checkset}"
-          default_gripper_baud="${default_gripper_baud}"/>
+          default_gripper_baud="${default_gripper_baud}"
+          model1300="${model1300}" />
       </xacro:unless>
     </xacro:if>
@@ -77,5 +80,6 @@
         report_type="${report_type}"
         baud_checkset="${baud_checkset}"
-        default_gripper_baud="${default_gripper_baud}" />
+        default_gripper_baud="${default_gripper_baud}"
+        model1300="${model1300}" />
     </xacro:unless>
     <xacro:if value="${robot_type != 'lite' and add_realsense_d435i}">

Commit message: [feat] add uf850 models

File: xarm_description/urdf/dual_xarm_device.urdf.xacro (robot description, xacro)
@@ -1,4 +1,4 @@
 <?xml version='1.0' encoding='utf-8'?>
-<robot xmlns:xacro="http://ros.org/wiki/xacro" name="dual_xarm">
+<robot xmlns:xacro="http://ros.org/wiki/xacro" name="DUAL_UF_ROBOT">
   <xacro:arg name="prefix_1" default="L_"/>
   <xacro:arg name="prefix_2" default="R_"/>
@@ -24,5 +24,5 @@
   <xacro:arg name="report_type_2" default="normal"/>
   <xacro:arg name="ros2_control_plugin" default="uf_robot_hardware/UFRobotSystemHardware"/>
-  <xacro:arg name="ros2_control_params" default="$(find xarm_controller)/config/xarm$(arg dof_1)_controllers.yaml"/>
+  <xacro:arg name="ros2_control_params" default=""/>
   <xacro:arg name="add_realsense_d435i_1" default="false"/>
   <xacro:arg name="add_realsense_d435i_2" default="false"/>
@@ -59,9 +59,4 @@
   <!-- load xarm device -->
   <xacro:include filename="$(find xarm_description)/urdf/xarm_device_macro.xacro" />
-  <link name="ground" />
-  <!-- gazebo_plugin -->
-  <xacro:include filename="$(find xarm_description)/urdf/common/common.gazebo.xacro" />
-  <!-- <xacro:gazebo_ros1_control_plugin namespace="$(arg hw_ns)"/> -->
-  <xacro:gazebo_ros2_control_plugin ros2_control_params="$(arg ros2_control_params)"/>
   <xacro:xarm_device prefix="$(arg prefix_1)" hw_ns="$(arg hw_ns)" limited="$(arg limited)"
     effort_control="$(arg effort_control)" velocity_control="$(arg velocity_control)"
@@ -69,5 +64,5 @@
     ros2_control_plugin="$(arg ros2_control_plugin)" robot_type="$(arg robot_type_1)"
     load_gazebo_plugin="false" ros2_control_params="$(arg ros2_control_params)"
-    attach_to="ground" attach_xyz="0 0 0" attach_rpy="0 0 0"
+    attach_to="world" attach_xyz="0 0 0" attach_rpy="0 0 0"
     add_realsense_d435i="$(arg add_realsense_d435i_1)"
     add_d435i_links="$(arg add_d435i_links_1)"
@@ -86,6 +81,6 @@
     add_gripper="$(arg add_gripper_2)" add_vacuum_gripper="$(arg add_vacuum_gripper_2)" dof="$(arg dof_2)"
     ros2_control_plugin="$(arg ros2_control_plugin)" robot_type="$(arg robot_type_2)"
-    load_gazebo_plugin="false" ros2_control_params="$(arg ros2_control_params)"
-    attach_to="ground" attach_xyz="0 1 0" attach_rpy="0 0 0"
+    load_gazebo_plugin="true" ros2_control_params="$(arg ros2_control_params)"
+    attach_to="world" attach_xyz="0 1 0" attach_rpy="0 0 0" create_attach_link="false"
     add_realsense_d435i="$(arg add_realsense_d435i_2)"
     add_d435i_links="$(arg add_d435i_links_2)"
