Commit message: update lite6 and its gripper/vacuum_gripper models and some launch files

File: xarm_description/urdf/xarm_device_macro.xacro (robot description, xacro)
@@ -52,12 +52,24 @@
     </xacro:unless>
     <xacro:if value="${add_gripper}">
-      <xacro:include filename="$(find xarm_description)/urdf/gripper/xarm_gripper_model.xacro" />
-      <xacro:load_gripper prefix="${prefix}" attach_to="${prefix}link_eef" effort_control="${effort_control}" velocity_control="${velocity_control}"
-        ros2_control_plugin="${ros2_control_plugin}" ros2_control_params="${ros2_control_params}"
-        load_gazebo_plugin="${load_gazebo_plugin}" />
+      <xacro:if value="${robot_type == 'xarm'}">
+        <xacro:include filename="$(find xarm_description)/urdf/gripper/xarm_gripper_model.xacro" />
+        <xacro:load_gripper prefix="${prefix}" attach_to="${prefix}link_eef" effort_control="${effort_control}" velocity_control="${velocity_control}"
+          ros2_control_plugin="${ros2_control_plugin}" ros2_control_params="${ros2_control_params}"
+          load_gazebo_plugin="${load_gazebo_plugin}" />
+      </xacro:if>
+      <xacro:if value="${robot_type == 'lite'}">
+        <xacro:include filename="$(find xarm_description)/urdf/gripper/lite_gripper.urdf.xacro" />
+        <xacro:uflite_gripper_urdf prefix="${prefix}" attach_to="${prefix}link_eef" />
+      </xacro:if>
     </xacro:if>
     <xacro:if value="${not add_gripper and add_vacuum_gripper}">
-      <xacro:include filename="$(find xarm_description)/urdf/vacuum_gripper/xarm_vacuum_gripper.urdf.xacro" />
-      <xacro:xarm_vacuum_gripper_urdf prefix="${prefix}" attach_to="${prefix}link_eef" effort_control="${effort_control}" velocity_control="${velocity_control}" />
+      <xacro:if value="${robot_type == 'xarm'}">
+        <xacro:include filename="$(find xarm_description)/urdf/vacuum_gripper/xarm_vacuum_gripper.urdf.xacro" />
+        <xacro:xarm_vacuum_gripper_urdf prefix="${prefix}" attach_to="${prefix}link_eef" effort_control="${effort_control}" velocity_control="${velocity_control}" />
+      </xacro:if>
+      <xacro:if value="${robot_type == 'lite'}">
+        <xacro:include filename="$(find xarm_description)/urdf/vacuum_gripper/lite_vacuum_gripper.urdf.xacro" />
+        <xacro:uflite_vacuum_gripper_urdf prefix="${prefix}" attach_to="${prefix}link_eef" />
+      </xacro:if>
     </xacro:if>
     <xacro:if value="${not add_gripper and not add_vacuum_gripper and add_other_geometry}">

File: xarm_moveit_config/srdf/_lite6_macro.srdf.xacro (robot description, xacro)
@@ -43,100 +43,40 @@
       <joint name="${prefix}joint6" value="0" />
     </group_state>
-    <group_state name="hold-up" group="${prefix}lite6">
-      <joint name="${prefix}joint1" value="0" />
-      <joint name="${prefix}joint2" value="0" />
-      <joint name="${prefix}joint3" value="0" />
-      <joint name="${prefix}joint4" value="0" />
-      <joint name="${prefix}joint5" value="-1.5708" />
-      <joint name="${prefix}joint6" value="0" />
-    </group_state>
     <!-- gripper -->
     <xacro:if value="${add_gripper}">
-      <group name="${prefix}xarm_gripper">
-        <link name="${prefix}xarm_gripper_base_link" />
-        <link name="${prefix}left_outer_knuckle" />
-        <link name="${prefix}left_finger" />
-        <link name="${prefix}left_inner_knuckle" />
-        <link name="${prefix}right_inner_knuckle" />
-        <link name="${prefix}right_outer_knuckle" />
-        <link name="${prefix}right_finger" />
-        <link name="${prefix}link_tcp" />
-        <joint name="${prefix}drive_joint" />
+      <group name="${prefix}lite_gripper">
+        <joint name="${prefix}gripper_fix" />
+        <joint name="${prefix}joint_tcp" />
       </group>
-      <group_state name="open" group="${prefix}xarm_gripper">
-        <joint name="${prefix}drive_joint" value="0" />
-      </group_state>
-      <group_state name="close" group="${prefix}xarm_gripper">
-        <joint name="${prefix}drive_joint" value="0.85" />
-      </group_state>
       <!-- END EFFECTOR, Purpose, Represent information about an end effector. -->
-      <end_effector name="${prefix}xarm_gripper" parent_link="${prefix}link_tcp" group="${prefix}xarm_gripper" />
+      <end_effector name="${prefix}lite_gripper" parent_link="${prefix}link_tcp" group="${prefix}lite_gripper" />
+      <passive_joint name="${prefix}gripper_fix" />
       <!--PASSIVE JOINT, Purpose, this element is used to mark joints that are not actuated-->
-      <passive_joint name="${prefix}left_finger_joint" />
-      <passive_joint name="${prefix}left_inner_knuckle_joint" />
-      <passive_joint name="${prefix}right_inner_knuckle_joint" />
-      <passive_joint name="${prefix}right_outer_knuckle_joint" />
-      <passive_joint name="${prefix}right_finger_joint" />
       <!-- DISABLE COLLISIONS, By default it is assumed that any link of the robot could potentially come into collision with any other link in the robot. This tag disables collision checking between a specified pair of links. -->
-      <disable_collisions link1="${prefix}left_finger" link2="${prefix}left_inner_knuckle" reason="Default" />
-      <disable_collisions link1="${prefix}left_finger" link2="${prefix}left_outer_knuckle" reason="Adjacent" />
-      <disable_collisions link1="${prefix}left_finger" link2="${prefix}link4" reason="Never" />
-      <disable_collisions link1="${prefix}left_finger" link2="${prefix}link5" reason="Never" />
-      <disable_collisions link1="${prefix}left_finger" link2="${prefix}link6" reason="Never" />
-      <disable_collisions link1="${prefix}left_finger" link2="${prefix}right_finger" reason="Never" />
-      <disable_collisions link1="${prefix}left_finger" link2="${prefix}right_inner_knuckle" reason="Never" />
-      <disable_collisions link1="${prefix}left_finger" link2="${prefix}right_outer_knuckle" reason="Never" />
-      <disable_collisions link1="${prefix}left_finger" link2="${prefix}xarm_gripper_base_link" reason="Never" />
-      <disable_collisions link1="${prefix}left_inner_knuckle" link2="${prefix}left_outer_knuckle" reason="Never" />
-      <disable_collisions link1="${prefix}left_inner_knuckle" link2="${prefix}link4" reason="Never" />
-      <disable_collisions link1="${prefix}left_inner_knuckle" link2="${prefix}link5" reason="Never" />
-      <disable_collisions link1="${prefix}left_inner_knuckle" link2="${prefix}link6" reason="Never" />
-      <disable_collisions link1="${prefix}left_inner_knuckle" link2="${prefix}right_finger" reason="Never" />
-      <disable_collisions link1="${prefix}left_inner_knuckle" link2="${prefix}right_inner_knuckle" reason="Never" />
-      <disable_collisions link1="${prefix}left_inner_knuckle" link2="${prefix}right_outer_knuckle" reason="Never" />
-      <disable_collisions link1="${prefix}left_inner_knuckle" link2="${prefix}xarm_gripper_base_link" reason="Adjacent" />
-      <disable_collisions link1="${prefix}left_outer_knuckle" link2="${prefix}link5" reason="Never" />
-      <disable_collisions link1="${prefix}left_outer_knuckle" link2="${prefix}link6" reason="Never" />
-      <disable_collisions link1="${prefix}left_outer_knuckle" link2="${prefix}right_finger" reason="Never" />
-      <disable_collisions link1="${prefix}left_outer_knuckle" link2="${prefix}right_inner_knuckle" reason="Never" />
-      <disable_collisions link1="${prefix}left_outer_knuckle" link2="${prefix}right_outer_knuckle" reason="Never" />
-      <disable_collisions link1="${prefix}left_outer_knuckle" link2="${prefix}xarm_gripper_base_link" reason="Adjacent" />
-      <disable_collisions link1="${prefix}link4" link2="${prefix}right_finger" reason="Never" />
-      <disable_collisions link1="${prefix}link4" link2="${prefix}right_inner_knuckle" reason="Never" />
-      <disable_collisions link1="${prefix}link5" link2="${prefix}link6" reason="Adjacent" />
-      <disable_collisions link1="${prefix}link5" link2="${prefix}right_finger" reason="Never" />
-      <disable_collisions link1="${prefix}link5" link2="${prefix}right_inner_knuckle" reason="Never" />
-      <disable_collisions link1="${prefix}link5" link2="${prefix}right_outer_knuckle" reason="Never" />
-      <disable_collisions link1="${prefix}link5" link2="${prefix}xarm_gripper_base_link" reason="Never" />
-      <disable_collisions link1="${prefix}link6" link2="${prefix}right_finger" reason="Never" />
-      <disable_collisions link1="${prefix}link6" link2="${prefix}right_inner_knuckle" reason="Never" />
-      <disable_collisions link1="${prefix}link6" link2="${prefix}right_outer_knuckle" reason="Never" />
-      <disable_collisions link1="${prefix}link6" link2="${prefix}xarm_gripper_base_link" reason="Adjacent" />
-      <disable_collisions link1="${prefix}right_finger" link2="${prefix}right_inner_knuckle" reason="Default" />
-      <disable_collisions link1="${prefix}right_finger" link2="${prefix}right_outer_knuckle" reason="Adjacent" />
-      <disable_collisions link1="${prefix}right_finger" link2="${prefix}xarm_gripper_base_link" reason="Never" />
-      <disable_collisions link1="${prefix}right_inner_knuckle" link2="${prefix}right_outer_knuckle" reason="Never" />
-      <disable_collisions link1="${prefix}right_inner_knuckle" link2="${prefix}xarm_gripper_base_link" reason="Adjacent" />
-      <disable_collisions link1="${prefix}right_outer_knuckle" link2="${prefix}xarm_gripper_base_link" reason="Adjacent" />
+      <disable_collisions link1="${prefix}link5" link2="${prefix}uflite_gripper_link" reason="Never" />
+      <disable_collisions link1="${prefix}link6" link2="${prefix}uflite_gripper_link" reason="Never" />
+      <disable_collisions link1="${prefix}link_eef" link2="${prefix}uflite_gripper_link" reason="Adjacent" />
     </xacro:if>
     <!-- vacuum gripper -->
     <xacro:if value="${not add_gripper and add_vacuum_gripper}">
-      <!-- <group name="${prefix}vacuum_gripper">
+      <group name="${prefix}vacuum_gripper">
         <joint name="${prefix}vacuum_gripper_fix" />
-      </group> -->
-      <!-- <end_effector name="${prefix}vacuum_gripper" parent_link="${prefix}link_tcp" group="${prefix}vacuum_gripper" /> -->
+      </group>
+      <end_effector name="${prefix}vacuum_gripper" parent_link="${prefix}link_tcp" group="${prefix}vacuum_gripper" />
       <passive_joint name="${prefix}vacuum_gripper_fix" />
-      <disable_collisions link1="${prefix}link5" link2="${prefix}xarm_vacuum_gripper_link" reason="Never" />
-      <disable_collisions link1="${prefix}link6" link2="${prefix}xarm_vacuum_gripper_link" reason="Adjacent" />
+      <disable_collisions link1="${prefix}link5" link2="${prefix}uflite_vacuum_gripper_link" reason="Never" />
+      <disable_collisions link1="${prefix}link6" link2="${prefix}uflite_vacuum_gripper_link" reason="Never" />
+      <disable_collisions link1="${prefix}link_eef" link2="${prefix}uflite_vacuum_gripper_link" reason="Adjacent" />
     </xacro:if>
     <!-- other box -->
     <xacro:if value="${not add_gripper and not add_vacuum_gripper and add_other_geometry}">
-      <!-- <group name="${prefix}other_geometry">
+      <group name="${prefix}other_geometry">
         <joint name="${prefix}other_geometry_fix" />
-      </group> -->
-      <!-- <end_effector name="${prefix}other_geometry" parent_link="${prefix}link_tcp" group="${prefix}other_geometry" /> -->
+      </group>
+      <end_effector name="${prefix}other_geometry" parent_link="${prefix}link_tcp" group="${prefix}other_geometry" />
       <passive_joint name="${prefix}other_geometry_fix" />
       <disable_collisions link1="${prefix}link5" link2="${prefix}other_geometry_link" reason="Never" />
-      <disable_collisions link1="${prefix}link6" link2="${prefix}other_geometry_link" reason="Adjacent" />
+      <disable_collisions link1="${prefix}link6" link2="${prefix}other_geometry_link" reason="Never" />
+      <disable_collisions link1="${prefix}link_eef" link2="${prefix}other_geometry_link" reason="Adjacent" />
     </xacro:if>
     <disable_collisions link1="${prefix}link1" link2="${prefix}link2" reason="Adjacent" />
@@ -152,4 +92,7 @@
     <disable_collisions link1="${prefix}link4" link2="${prefix}link6" reason="Never" />
     <disable_collisions link1="${prefix}link5" link2="${prefix}link6" reason="Adjacent" />
+    <disable_collisions link1="${prefix}link3" link2="${prefix}link_eef" reason="Never" />
+    <disable_collisions link1="${prefix}link5" link2="${prefix}link_eef" reason="Never" />
+    <disable_collisions link1="${prefix}link6" link2="${prefix}link_eef" reason="Adjacent" />
   </xacro:macro>
 </robot>

Commit message: update kinematics_params_filename path to use shared directory

File: xarm_description/urdf/xarm_device_macro.xacro (robot description, xacro)
@@ -91,5 +91,5 @@
     </xacro:unless>
     <xacro:if value="${kinematics_suffix != ''}">
-      <xacro:property name="kinematics_params_filename" value="$(find xarm_description)/config/kinematics/user/${robot_name}_kinematics_${kinematics_suffix}.yaml"/>
+      <xacro:property name="kinematics_params_filename" value="/shared/${robot_name}_kinematics_${kinematics_suffix}.yaml"/>
     </xacro:if>
     <xacro:unless value="${kinematics_suffix != ''}">

Commit message: Update kinematics_params_filename path for improved configuration management

File: xarm_description/urdf/xarm_device_macro.xacro (robot description, xacro)
@@ -92,5 +92,5 @@
     </xacro:unless>
     <xacro:if value="${kinematics_suffix != ''}">
-      <xacro:property name="kinematics_params_filename" value="$(find xarm_description)/config/kinematics/user/${robot_name}_kinematics_${kinematics_suffix}.yaml"/>
+      <xacro:property name="kinematics_params_filename" value="/shared/${robot_name}_kinematics_${kinematics_suffix}.yaml"/>
     </xacro:if>
     <xacro:unless value="${kinematics_suffix != ''}">
