Commit message: [feat] support bio gripper
1. add `add_bio_gripper` parameter to support bio gripper
2. Lite6 is not support bio gripper

File: xarm_description/urdf/xarm7_mirror/xarm7_mirror.ros2_control.xacro (robot description, xacro)
@@ -4,5 +4,5 @@
     velocity_control:='false'
     ros2_control_plugin:='uf_robot_hardware/UFRobotSystemHardware'
-    hw_ns:='xarm' add_gripper:='false'
+    hw_ns:='xarm' add_gripper:='false' add_bio_gripper:='false'
     robot_ip:='' report_type:='normal' baud_checkset:='true' default_gripper_baud:=2000000
     joint1_lower_limit:=${-2.0*pi}  joint1_upper_limit:=${2.0*pi}
@@ -27,4 +27,5 @@
           <param name="robot_type">xarm</param>
           <param name="add_gripper">${add_gripper}</param>
+          <param name="add_bio_gripper">${add_bio_gripper}</param>
         </xacro:if>
       </hardware>

File: xarm_description/urdf/xarm7_mirror/xarm7_mirror_robot_macro.xacro (robot description, xacro)
@@ -7,4 +7,5 @@
     velocity_control:=false
     add_gripper:=false
+    add_bio_gripper:=false
     ros2_control_plugin:='uf_robot_hardware/UFRobotSystemHardware'
     robot_ip:=''
@@ -29,5 +30,5 @@
           velocity_control="${velocity_control}"
           ros2_control_plugin="${ros2_control_plugin}"
-          hw_ns="${hw_ns}" add_gripper="${add_gripper}"
+          hw_ns="${hw_ns}" add_gripper="${add_gripper}" add_bio_gripper="${add_bio_gripper}"
           robot_ip="${robot_ip}" report_type="${report_type}"
           baud_checkset="${baud_checkset}" default_gripper_baud="${default_gripper_baud}"
@@ -57,5 +58,5 @@
         <xacro:xarm7_mirror_ros2_control prefix="${prefix}" velocity_control="${velocity_control}"
           ros2_control_plugin="${ros2_control_plugin}"
-          hw_ns="${hw_ns}" add_gripper="${add_gripper}"
+          hw_ns="${hw_ns}" add_gripper="${add_gripper}" add_bio_gripper="${add_bio_gripper}"
           robot_ip="${robot_ip}" report_type="${report_type}"
           baud_checkset="${baud_checkset}" default_gripper_baud="${default_gripper_baud}" />

File: xarm_description/urdf/xarm_device_macro.xacro (robot description, xacro)
@@ -9,4 +9,5 @@
     add_gripper:=false
     add_vacuum_gripper:=false
+    add_bio_gripper:=false
     dof:=7
     robot_type:='xarm'
@@ -102,4 +103,5 @@
         ros2_control_plugin="${ros2_control_plugin}"
         add_gripper="${add_gripper}"
+        add_bio_gripper="${add_bio_gripper}"
         robot_ip="${robot_ip}"
         report_type="${report_type}"
@@ -119,4 +121,5 @@
           ros2_control_plugin="${ros2_control_plugin}"
           add_gripper="${add_gripper}"
+          add_bio_gripper="${add_bio_gripper}"
           robot_ip="${robot_ip}"
           report_type="${report_type}"
@@ -150,4 +153,5 @@
           ros2_control_plugin="${ros2_control_plugin}"
           add_gripper="${add_gripper}"
+          add_bio_gripper="${add_bio_gripper}"
           robot_ip="${robot_ip}"
           report_type="${report_type}"
@@ -168,4 +172,5 @@
           ros2_control_plugin="${ros2_control_plugin}"
           add_gripper="${add_gripper}"
+          add_bio_gripper="${add_bio_gripper}"
           robot_ip="${robot_ip}"
           report_type="${report_type}"
@@ -184,4 +189,5 @@
           ros2_control_plugin="${ros2_control_plugin}"
           add_gripper="${add_gripper}"
+          add_bio_gripper="${add_bio_gripper}"
           robot_ip="${robot_ip}"
           report_type="${report_type}"
@@ -224,5 +230,13 @@
       </xacro:unless>
     </xacro:if>
-    <xacro:if value="${not add_gripper and add_vacuum_gripper}">
+    <xacro:if value="${not add_gripper and add_bio_gripper}">
+      <xacro:unless value="${robot_type == 'lite'}">
+        <!-- Load BIO Gripper Model URDF -->
+        <xacro:include filename="$(find xarm_description)/urdf/gripper/bio_gripper_macro.xacro" />
+        <xacro:bio_gripper_macro prefix="${prefix}" attach_to="${prefix}link_eef"
+          ros2_control_plugin="${ros2_control_plugin}" dof="${dof}" hard_interface="${hard_interface}" />
+      </xacro:unless>
+    </xacro:if>
+    <xacro:if value="${not add_gripper and not add_bio_gripper and add_vacuum_gripper}">
       <xacro:if value="${robot_type == 'lite'}">
         <!-- Load Lite Vacuum Gripper Model URDF -->

File: xarm_moveit_config/srdf/_uf850_macro.srdf.xacro (robot description, xacro)
@@ -10,5 +10,5 @@
   <!-- SUBGROUPS: Groups can also be formed by referencing to already defined group names -->
   <xacro:macro name="uf850_macro_srdf" params="prefix=''
-    add_gripper='false' add_vacuum_gripper='false' add_other_geometry='false' ">
+    add_gripper='false' add_vacuum_gripper='false' add_bio_gripper='false' add_other_geometry='false' ">
     <group name="${prefix}uf850">
       <joint name="${prefix}world_joint" />
@@ -25,9 +25,13 @@
         <joint name="${prefix}joint_tcp" />
       </xacro:if>
-      <xacro:if value="${not add_gripper and add_vacuum_gripper}">
+      <xacro:if value="${not add_gripper and add_bio_gripper}">
+        <joint name="${prefix}bio_gripper_fix" />
+        <joint name="${prefix}joint_tcp" />
+      </xacro:if>
+      <xacro:if value="${not add_gripper and not add_bio_gripper and add_vacuum_gripper}">
         <joint name="${prefix}vacuum_gripper_fix" />
         <joint name="${prefix}joint_tcp" />
       </xacro:if>
-      <xacro:if value="${not add_gripper and not add_vacuum_gripper and add_other_geometry}">
+      <xacro:if value="${not add_gripper and not add_bio_gripper and not add_vacuum_gripper and add_other_geometry}">
         <joint name="${prefix}other_geometry_fix" />
         <joint name="${prefix}joint_tcp" />
@@ -127,6 +131,42 @@
       <disable_collisions link1="${prefix}link_eef" link2="${prefix}xarm_gripper_base_link" reason="Adjacent" />
     </xacro:if>
+    <!-- bio gripper -->
+    <xacro:if value="${not add_gripper and add_bio_gripper}">
+      <group name="${prefix}bio_gripper">
+        <link name="${prefix}bio_gripper_base_link" />
+        <link name="${prefix}bio_gripper_left_finger" />
+        <link name="${prefix}bio_gripper_right_finger" />
+        <link name="${prefix}link_tcp" />
+        <joint name="${prefix}left_finger_joint" />
+        <joint name="${prefix}right_finger_joint" />
+      </group>
+      <group_state name="open" group="${prefix}bio_gripper">
+        <joint name="${prefix}left_finger_joint" value="-0.04" />
+        <joint name="${prefix}right_finger_joint" value="0.04" />
+      </group_state>
+      <group_state name="close" group="${prefix}bio_gripper">
+        <joint name="${prefix}left_finger_joint" value="0" />
+        <joint name="${prefix}right_finger_joint" value="0" />
+      </group_state>
+      <!-- END EFFECTOR, Purpose, Represent information about an end effector. -->
+      <end_effector name="${prefix}bio_gripper" parent_link="${prefix}link_tcp" group="${prefix}bio_gripper" />
+      <!-- DISABLE COLLISIONS, By default it is assumed that any link of the robot could potentially come into collision with any other link in the robot. This tag disables collision checking between a specified pair of links. -->
+      <disable_collisions link1="${prefix}bio_gripper_left_finger" link2="${prefix}bio_gripper_base_link" reason="Adjacent" />
+      <disable_collisions link1="${prefix}bio_gripper_right_finger" link2="${prefix}bio_gripper_base_link" reason="Adjacent" />
+      <disable_collisions link1="${prefix}bio_gripper_left_finger" link2="${prefix}bio_gripper_right_finger" reason="Never" />
+      <disable_collisions link1="${prefix}bio_gripper_left_finger" link2="${prefix}link4" reason="Never" />
+      <disable_collisions link1="${prefix}bio_gripper_left_finger" link2="${prefix}link5" reason="Never" />
+      <disable_collisions link1="${prefix}bio_gripper_left_finger" link2="${prefix}link6" reason="Never" />
+      <disable_collisions link1="${prefix}bio_gripper_right_finger" link2="${prefix}link4" reason="Never" />
+      <disable_collisions link1="${prefix}bio_gripper_right_finger" link2="${prefix}link5" reason="Never" />
+      <disable_collisions link1="${prefix}bio_gripper_right_finger" link2="${prefix}link6" reason="Never" />
+      <disable_collisions link1="${prefix}link6" link2="${prefix}bio_gripper_base_link" reason="Adjacent" />
+      <disable_collisions link1="${prefix}link5" link2="${prefix}bio_gripper_base_link" reason="Never" />
+      <disable_collisions link1="${prefix}link_eef" link2="${prefix}bio_gripper_left_finger" reason="Never" />
+      <disable_collisions link1="${prefix}link_eef" link2="${prefix}bio_gripper_left_finger" reason="Never" />
+      <disable_collisions link1="${prefix}link_eef" link2="${prefix}bio_gripper_base_link" reason="Adjacent" />
+    </xacro:if>
     <!-- vacuum gripper -->
-    <xacro:if value="${not add_gripper and add_vacuum_gripper}">
+    <xacro:if value="${not add_gripper and not add_bio_gripper and add_vacuum_gripper}">
       <!-- <group name="${prefix}vacuum_gripper">
         <joint name="${prefix}vacuum_gripper_fix" />
@@ -139,5 +179,5 @@
     </xacro:if>
     <!-- other box -->
-    <xacro:if value="${not add_gripper and not add_vacuum_gripper and add_other_geometry}">
+    <xacro:if value="${not add_gripper and not add_bio_gripper and not add_vacuum_gripper and add_other_geometry}">
       <!-- <group name="${prefix}other_geometry">
         <joint name="${prefix}other_geometry_fix" />

File: xarm_moveit_config/srdf/_xarm7_mirror_macro.srdf.xacro (robot description, xacro)
@@ -10,5 +10,5 @@
   <!-- SUBGROUPS: Groups can also be formed by referencing to already defined group names -->
   <xacro:macro name="xarm7_mirror_macro_srdf" params="prefix=''
-    add_gripper='false' add_vacuum_gripper='false' add_other_geometry='false' ">
+    add_gripper='false' add_vacuum_gripper='false' add_bio_gripper='false' add_other_geometry='false' ">
     <group name="${prefix}xarm7_mirror">
       <joint name="${prefix}world_joint" />
@@ -26,9 +26,13 @@
         <joint name="${prefix}joint_tcp" />
       </xacro:if>
-      <xacro:if value="${not add_gripper and add_vacuum_gripper}">
+      <xacro:if value="${not add_gripper and add_bio_gripper}">
+        <joint name="${prefix}bio_gripper_fix" />
+        <joint name="${prefix}joint_tcp" />
+      </xacro:if>
+      <xacro:if value="${not add_gripper and not add_bio_gripper and add_vacuum_gripper}">
         <joint name="${prefix}vacuum_gripper_fix" />
         <joint name="${prefix}joint_tcp" />
       </xacro:if>
-      <xacro:if value="${not add_gripper and not add_vacuum_gripper and add_other_geometry}">
+      <xacro:if value="${not add_gripper and not add_bio_gripper and not add_vacuum_gripper and add_other_geometry}">
         <joint name="${prefix}other_geometry_fix" />
         <joint name="${prefix}joint_tcp" />
@@ -135,6 +139,43 @@
       <disable_collisions link1="${prefix}link_eef" link2="${prefix}xarm_gripper_base_link" reason="Adjacent" />
     </xacro:if>
+    <!-- bio gripper -->
+    <xacro:if value="${not add_gripper and add_bio_gripper}">
+      <group name="${prefix}bio_gripper">
+        <link name="${prefix}bio_gripper_base_link" />
+        <link name="${prefix}bio_gripper_left_finger" />
+        <link name="${prefix}bio_gripper_right_finger" />
+        <link name="${prefix}link_tcp" />
+        <joint name="${prefix}left_finger_joint" />
+        <joint name="${prefix}right_finger_joint" />
+      </group>
+      <group_state name="open" group="${prefix}bio_gripper">
+        <joint name="${prefix}left_finger_joint" value="-0.04" />
+        <joint name="${prefix}right_finger_joint" value="0.04" />
+      </group_state>
+      <group_state name="close" group="${prefix}bio_gripper">
+        <joint name="${prefix}left_finger_joint" value="0" />
+        <joint name="${prefix}right_finger_joint" value="0" />
+      </group_state>
+      <!-- END EFFECTOR, Purpose, Represent information about an end effector. -->
+      <end_effector name="${prefix}bio_gripper" parent_link="${prefix}link_tcp" group="${prefix}bio_gripper" />
+      <!-- DISABLE COLLISIONS, By default it is assumed that any link of the robot could potentially come into collision with any other link in the robot. This tag disables collision checking between a specified pair of links. -->
+      <disable_collisions link1="${prefix}bio_gripper_left_finger" link2="${prefix}bio_gripper_base_link" reason="Adjacent" />
+      <disable_collisions link1="${prefix}bio_gripper_right_finger" link2="${prefix}bio_gripper_base_link" reason="Adjacent" />
+      <disable_collisions link1="${prefix}bio_gripper_left_finger" link2="${prefix}bio_gripper_right_finger" reason="Never" />
+      <disable_collisions link1="${prefix}bio_gripper_left_finger" link2="${prefix}link5" reason="Never" />
+      <disable_collisions link1="${prefix}bio_gripper_left_finger" link2="${prefix}link6" reason="Never" />
+      <disable_collisions link1="${prefix}bio_gripper_left_finger" link2="${prefix}link7" reason="Never" />
+      <disable_collisions link1="${prefix}bio_gripper_right_finger" link2="${prefix}link5" reason="Never" />
+      <disable_collisions link1="${prefix}bio_gripper_right_finger" link2="${prefix}link6" reason="Never" />
+      <disable_collisions link1="${prefix}bio_gripper_right_finger" link2="${prefix}link7" reason="Never" />
+      <disable_collisions link1="${prefix}link7" link2="${prefix}bio_gripper_base_link" reason="Adjacent" />
+      <disable_collisions link1="${prefix}link6" link2="${prefix}bio_gripper_base_link" reason="Never" />
+      <disable_collisions link1="${prefix}link3" link2="${prefix}bio_gripper_base_link" reason="Never" />
+      <disable_collisions link1="${prefix}link_eef" link2="${prefix}bio_gripper_left_finger" reason="Never" />
+      <disable_collisions link1="${prefix}link_eef" link2="${prefix}bio_gripper_left_finger" reason="Never" />
+      <disable_collisions link1="${prefix}link_eef" link2="${prefix}bio_gripper_base_link" reason="Adjacent" />
+    </xacro:if>
     <!-- vacuum gripper -->
-    <xacro:if value="${not add_gripper and add_vacuum_gripper}">
+    <xacro:if value="${not add_gripper and not add_bio_gripper and add_vacuum_gripper}">
       <!-- <group name="${prefix}vacuum_gripper">
         <joint name="${prefix}vacuum_gripper_fix" />
@@ -148,5 +189,5 @@
     </xacro:if>
     <!-- other box -->
-    <xacro:if value="${not add_gripper and not add_vacuum_gripper and add_other_geometry}">
+    <xacro:if value="${not add_gripper and not add_bio_gripper and not add_vacuum_gripper and add_other_geometry}">
       <!-- <group name="${prefix}other_geometry">
         <joint name="${prefix}other_geometry_fix" />

File: xarm_moveit_config/srdf/xarm_macro.srdf.xacro (robot description, xacro)
@@ -2,9 +2,9 @@
 <robot xmlns:xacro="http://wiki.ros.org/xacro" name="xarm_srdf">
   <xacro:macro name="xarm_macro_srdf" params="prefix:='' dof:=7 robot_type:='xarm'
-    add_gripper:='false' add_vacuum_gripper:='false' add_other_geometry:='false' ">
+    add_gripper:='false' add_vacuum_gripper:='false' add_bio_gripper:='false' add_other_geometry:='false' ">
     <xacro:if value="${dof == 5}">
       <xacro:include filename="$(find xarm_moveit_config)/srdf/_xarm5_macro.srdf.xacro" />
       <xacro:xarm5_macro_srdf prefix="${prefix}"
-        add_gripper="${add_gripper}" add_vacuum_gripper="${add_vacuum_gripper}" add_other_geometry="${add_other_geometry}" />
+        add_gripper="${add_gripper}" add_vacuum_gripper="${add_vacuum_gripper}" add_bio_gripper="${add_bio_gripper}" add_other_geometry="${add_other_geometry}" />
     </xacro:if>
     <xacro:if value="${dof == 6}">
@@ -12,5 +12,5 @@
         <xacro:include filename="$(find xarm_moveit_config)/srdf/_uf850_macro.srdf.xacro" />
         <xacro:uf850_macro_srdf prefix="${prefix}"
-          add_gripper="${add_gripper}" add_vacuum_gripper="${add_vacuum_gripper}" add_other_geometry="${add_other_geometry}"  />
+          add_gripper="${add_gripper}" add_vacuum_gripper="${add_vacuum_gripper}" add_bio_gripper="${add_bio_gripper}" add_other_geometry="${add_other_geometry}"  />
       </xacro:if>
       <xacro:if value="${robot_type == 'lite'}">
@@ -22,5 +22,5 @@
         <xacro:include filename="$(find xarm_moveit_config)/srdf/_xarm6_macro.srdf.xacro" />
         <xacro:xarm6_macro_srdf prefix="${prefix}"
-          add_gripper="${add_gripper}" add_vacuum_gripper="${add_vacuum_gripper}" add_other_geometry="${add_other_geometry}"  />
+          add_gripper="${add_gripper}" add_vacuum_gripper="${add_vacuum_gripper}" add_bio_gripper="${add_bio_gripper}" add_other_geometry="${add_other_geometry}"  />
       </xacro:unless>
     </xacro:if>
@@ -29,10 +29,10 @@
         <xacro:include filename="$(find xarm_moveit_config)/srdf/_xarm7_mirror_macro.srdf.xacro" />
         <xacro:xarm7_mirror_macro_srdf prefix="${prefix}"
-          add_gripper="${add_gripper}" add_vacuum_gripper="${add_vacuum_gripper}" add_other_geometry="${add_other_geometry}"  />
+          add_gripper="${add_gripper}" add_vacuum_gripper="${add_vacuum_gripper}" add_bio_gripper="${add_bio_gripper}" add_other_geometry="${add_other_geometry}"  />
       </xacro:if>
       <xacro:unless value="${robot_type == 'xarm7_mirror'}">
         <xacro:include filename="$(find xarm_moveit_config)/srdf/_xarm7_macro.srdf.xacro" />
         <xacro:xarm7_macro_srdf prefix="${prefix}"
-          add_gripper="${add_gripper}" add_vacuum_gripper="${add_vacuum_gripper}" add_other_geometry="${add_other_geometry}"  />
+          add_gripper="${add_gripper}" add_vacuum_gripper="${add_vacuum_gripper}" add_bio_gripper="${add_bio_gripper}" add_other_geometry="${add_other_geometry}"  />
       </xacro:unless>
     </xacro:unless>
