Commit message: updated xarm_ros2 package to work internally

File: xarm_description/urdf/camera/camera.gazebo.xacro (robot description, xacro)
@@ -42,5 +42,5 @@
             <width>640</width>
             <height>480</height>
-            <format>B8G8R8</format>
+            <foramt>B8G8R8</foramt>
           </image>
           <clip>

File: xarm_description/urdf/camera/realsense.gazebo.xacro (robot description, xacro)
@@ -1,8 +1,8 @@
 <?xml version="1.0"?>
 <robot xmlns:xacro="http://ros.org/wiki/xacro">
-  <xacro:macro name="realsense_gazebo" params="prefix:=''">
-    <gazebo reference="${prefix}camera_depth_frame">
-      <sensor name="${prefix}cameradepth" type="depth">
-        <camera name="${prefix}camera">
+  <xacro:macro name="realsense_gazebo" params="prefix:='' ">
+    <!-- <gazebo reference="${prefix}camera_depth_frame">
+      <sensor name="cameradepth" type="depth">
+        <camera name="camera">
           <horizontal_fov>1.57</horizontal_fov>
           <image>
@@ -26,6 +26,6 @@
     </gazebo>
     <gazebo reference="${prefix}camera_color_frame">
-      <sensor name="${prefix}cameracolor" type="camera">
-        <camera name="${prefix}camera">
+      <sensor name="cameracolor" type="camera">
+        <camera name="camera">
           <horizontal_fov>1.57</horizontal_fov>
           <image>
@@ -50,6 +50,6 @@
     </gazebo>
     <gazebo reference="${prefix}camera_left_ir_frame">
-      <sensor name="${prefix}cameraired1" type="camera">
-        <camera name="${prefix}camera">
+      <sensor name="cameraired1" type="camera">
+        <camera name="camera">
           <horizontal_fov>1.57</horizontal_fov>
           <image>
@@ -74,6 +74,6 @@
     </gazebo>
     <gazebo reference="${prefix}camera_right_ir_frame">
-      <sensor name="${prefix}cameraired2" type="camera">
-        <camera name="${prefix}camera">
+      <sensor name="cameraired2" type="camera">
+        <camera name="camera">
           <horizontal_fov>1.57</horizontal_fov>
           <image>
@@ -99,270 +99,85 @@
     <gazebo>
       <plugin name="realsense_gazebo_camera" filename="librealsense_gazebo_plugin.so">
-        <prefix>${prefix}camera</prefix>
+        <prefix>camera</prefix>
         <depthUpdateRate>30.0</depthUpdateRate>
         <colorUpdateRate>30.0</colorUpdateRate>
         <infraredUpdateRate>30.0</infraredUpdateRate>
-        <depthTopicName>${prefix}aligned_depth_to_color/image_raw</depthTopicName>
-        <depthCameraInfoTopicName>${prefix}depth/camera_info</depthCameraInfoTopicName>
-        <colorTopicName>${prefix}color/image_raw</colorTopicName>
-        <colorCameraInfoTopicName>${prefix}color/camera_info</colorCameraInfoTopicName>
-        <infrared1TopicName>${prefix}infra1/image_raw</infrared1TopicName>
-        <infrared1CameraInfoTopicName>${prefix}infra1/camera_info</infrared1CameraInfoTopicName>
-        <infrared2TopicName>${prefix}infra2/image_raw</infrared2TopicName>
-        <infrared2CameraInfoTopicName>${prefix}infra2/camera_info</infrared2CameraInfoTopicName>
-        <colorOpticalframeName>${prefix}camera_color_optical_frame</colorOpticalframeName>
-        <depthOpticalframeName>${prefix}camera_depth_optical_frame</depthOpticalframeName>
-        <infrared1OpticalframeName>${prefix}camera_left_ir_optical_frame</infrared1OpticalframeName>
-        <infrared2OpticalframeName>${prefix}camera_right_ir_optical_frame</infrared2OpticalframeName>
+        <depthTopicName>aligned_depth_to_color/image_raw</depthTopicName>
+        <depthCameraInfoTopicName>depth/camera_info</depthCameraInfoTopicName>
+        <colorTopicName>color/image_raw</colorTopicName>
+        <colorCameraInfoTopicName>color/camera_info</colorCameraInfoTopicName>
+        <infrared1TopicName>infra1/image_raw</infrared1TopicName>
+        <infrared1CameraInfoTopicName>infra1/camera_info</infrared1CameraInfoTopicName>
+        <infrared2TopicName>infra2/image_raw</infrared2TopicName>
+        <infrared2CameraInfoTopicName>infra2/camera_info</infrared2CameraInfoTopicName>
+        <colorOpticalframeName>camera_color_optical_frame</colorOpticalframeName>
+        <depthOpticalframeName>camera_depth_optical_frame</depthOpticalframeName>
+        <infrared1OpticalframeName>camera_left_ir_optical_frame</infrared1OpticalframeName>
+        <infrared2OpticalframeName>camera_right_ir_optical_frame</infrared2OpticalframeName>
         <rangeMinDepth>0.3</rangeMinDepth>
         <rangeMaxDepth>3.0</rangeMaxDepth>
         <pointCloud>true</pointCloud>
-        <pointCloudTopicName>${prefix}depth/color/points</pointCloudTopicName>
+        <pointCloudTopicName>depth/color/points</pointCloudTopicName>
         <pointCloudCutoff>0.3</pointCloudCutoff>
       </plugin>
-    </gazebo>
-  </xacro:macro>
-  <xacro:macro name="realsense_ignition" params="prefix:=''">
-    <gazebo reference="${prefix}camera_depth_frame">
-      <sensor name="${prefix}cameradepth" type="rgbd_camera">
-        <camera name="${prefix}camera">
-          <horizontal_fov>1.57</horizontal_fov>
+    </gazebo> -->
+    <gazebo reference="${prefix}camera_color_frame">
+      <sensor name="${prefix}_rgbd_sensor" type="rgbd_camera">
+        <camera>
+          <horizontal_fov>1.047</horizontal_fov>
           <image>
-            <width>1280</width>
-            <height>720</height>
-            <format>L8</format>
-          </image>
-          <clip>
-            <near>0.1</near>
-            <far>100</far>
-          </clip>
-          <depth_camera>
-            <clip>
-              <near>0.1</near>
-              <far>10</far>
-            </clip>
-          </depth_camera>
-          <noise>
-            <type>gaussian</type>
-            <mean>0.0</mean>
-            <stddev>0.100</stddev>
-          </noise>
-           <!-- <camera_info_topic>${prefix}camera/depth/camera_info</camera_info_topic> -->
-        </camera>
-        <always_on>1</always_on>
-        <update_rate>30</update_rate>
-        <visualize>0</visualize>
-        <topic>${prefix}camera/depth</topic>
-      </sensor>
-    </gazebo>
-    <gazebo reference="${prefix}camera_color_frame">
-      <sensor name="${prefix}cameracolor" type="camera">
-        <!-- <ignition_frame_id>${prefix}camera_color_frame</ignition_frame_id>
-        <optical_frame_id>${prefix}camera_color_frame</optical_frame_id> -->
-        <camera name="${prefix}camera">
-          <horizontal_fov>1.57</horizontal_fov>
-          <image>
-            <width>1280</width>
-            <height>720</height>
+            <width>640</width>
+            <height>480</height>
             <format>RGB_INT8</format>
           </image>
           <clip>
             <near>0.1</near>
-            <far>100</far>
+            <far>5</far>
           </clip>
+          <distortion>
+            <k1>0.0</k1>
+            <k2>0.0</k2>
+            <k3>0.0</k3>
+            <p1>0.0</p1>
+            <p2>0.0</p2>
+            <center>0.5 0.5</center>
+          </distortion>
+          <lens>
+            <intrinsics>
+              <fx>554.25469</fx>
+              <fy>554.25469</fy>
+              <cx>320.5</cx>
+              <cy>240.5</cy>
+              <s>0</s>
+            </intrinsics>
+            <projection>
+              <p_fx>554.25469</p_fx>
+              <p_fy>554.25469</p_fy>
+              <p_cx>320.5</p_cx>
+              <p_cy>240.5</p_cy>
+              <tx>0</tx>
+              <ty>0</ty>
+            </projection>
+          </lens>
           <noise>
             <type>gaussian</type>
-            <mean>0.0</mean>
-            <stddev>0.007</stddev>
+            <mean>0</mean>
+            <stddev>0.00</stddev>
           </noise>
-          <camera_info_topic>${prefix}camera/color/camera_info</camera_info_topic>
-        </camera>
-        <always_on>1</always_on>
-        <update_rate>30</update_rate>
-        <visualize>1</visualize>
-        <topic>${prefix}camera/color/image_raw</topic>
-        <enable_metrics>true</enable_metrics>
-      </sensor>
-    </gazebo>
-    <gazebo reference="${prefix}camera_left_ir_frame">
-      <sensor name="${prefix}cameraired1" type="camera">
-        <camera name="${prefix}camera">
-          <horizontal_fov>1.57</horizontal_fov>
-          <image>
-            <width>1280</width>
-            <height>720</height>
-            <format>L_INT8</format>
-          </image>
-          <clip>
-            <near>0.1</near>
-            <far>100</far>
-          </clip>
-          <noise>
-            <type>gaussian</type>
-            <mean>0.0</mean>
-            <stddev>0.05</stddev>
-          </noise>
-           <camera_info_topic>${prefix}camera/infra1/camera_info</camera_info_topic>
-        </camera>
-        <always_on>1</always_on>
-        <update_rate>30</update_rate>
-        <visualize>0</visualize>
-        <topic>${prefix}camera/infra1/image_raw</topic>
-      </sensor>
-    </gazebo>
-    <gazebo reference="${prefix}camera_right_ir_frame">
-      <sensor name="${prefix}cameraired2" type="camera">
-        <camera name="${prefix}camera">
-          <horizontal_fov>1.57</horizontal_fov>
-          <image>
-            <width>1280</width>
-            <height>720</height>
-            <format>L_INT8</format>
-          </image>
-          <clip>
-            <near>0.1</near>
-            <far>100</far>
-          </clip>
-          <noise>
-            <type>gaussian</type>
-            <mean>0.0</mean>
-            <stddev>0.05</stddev>
-          </noise>
-          <camera_info_topic>${prefix}camera/infra2/camera_info</camera_info_topic>
-        </camera>
-        <always_on>1</always_on>
-        <update_rate>30</update_rate>
-        <visualize>0</visualize>
-        <topic>${prefix}camera/infra2/image_raw</topic>
-      </sensor>
-    </gazebo>
-    <gazebo>
-      <plugin
-        filename="libignition-gazebo-sensors-system.so"
-        name="ignition::gazebo::systems::Sensors">
-        <render_engine>ogre2</render_engine>
-      </plugin>
-    </gazebo>
-  </xacro:macro>
-  <xacro:macro name="realsense_gz" params="prefix:=''">
-    <gazebo reference="${prefix}camera_depth_frame">
-      <sensor name="${prefix}cameradepth" type="rgbd_camera">
-        <camera name="${prefix}camera">
-          <horizontal_fov>1.57</horizontal_fov>
-          <image>
-            <width>1280</width>
-            <height>720</height>
-            <format>L8</format>
-          </image>
-          <clip>
-            <near>0.1</near>
-            <far>100</far>
-          </clip>
           <depth_camera>
             <clip>
-              <near>0.1</near>
-              <far>10</far>
+              <near>0.25</near>
+              <far>5</far>
             </clip>
           </depth_camera>
-          <noise>
-            <type>gaussian</type>
-            <mean>0.0</mean>
-            <stddev>0.100</stddev>
-          </noise>
-           <!-- <camera_info_topic>${prefix}camera/depth/camera_info</camera_info_topic> -->
+          <optical_frame_id>${prefix}camera_color_optical_frame</optical_frame_id>
         </camera>
+        <ignition_frame_id>${prefix}camera_color_frame</ignition_frame_id>
         <always_on>1</always_on>
-        <update_rate>30</update_rate>
-        <visualize>0</visualize>
-        <topic>${prefix}camera/depth</topic>
+        <update_rate>10.0</update_rate>
+        <visualize>false</visualize>
+        <topic>wrist_mounted_camera</topic>
+        <enable_metrics>false</enable_metrics>
       </sensor>
-    </gazebo>
-    <gazebo reference="${prefix}camera_color_frame">
-      <sensor name="${prefix}cameracolor" type="camera">
-        <!-- <ignition_frame_id>${prefix}camera_color_frame</ignition_frame_id>
-        <optical_frame_id>${prefix}camera_color_frame</optical_frame_id> -->
-        <camera name="${prefix}camera">
-          <horizontal_fov>1.57</horizontal_fov>
-          <image>
-            <width>1280</width>
-            <height>720</height>
-            <format>RGB_INT8</format>
-          </image>
-          <clip>
-            <near>0.1</near>
-            <far>100</far>
-          </clip>
-          <noise>
-            <type>gaussian</type>
-            <mean>0.0</mean>
-            <stddev>0.007</stddev>
-          </noise>
-          <camera_info_topic>${prefix}camera/color/camera_info</camera_info_topic>
-        </camera>
-        <always_on>1</always_on>
-        <update_rate>30</update_rate>
-        <visualize>1</visualize>
-        <topic>${prefix}camera/color/image_raw</topic>
-        <enable_metrics>true</enable_metrics>
-      </sensor>
-    </gazebo>
-    <gazebo reference="${prefix}camera_left_ir_frame">
-      <sensor name="${prefix}cameraired1" type="camera">
-        <camera name="${prefix}camera">
-          <horizontal_fov>1.57</horizontal_fov>
-          <image>
-            <width>1280</width>
-            <height>720</height>
-            <format>L_INT8</format>
-          </image>
-          <clip>
-            <near>0.1</near>
-            <far>100</far>
-          </clip>
-          <noise>
-            <type>gaussian</type>
-            <mean>0.0</mean>
-            <stddev>0.05</stddev>
-          </noise>
-           <camera_info_topic>${prefix}camera/infra1/camera_info</camera_info_topic>
-        </camera>
-        <always_on>1</always_on>
-        <update_rate>30</update_rate>
-        <visualize>0</visualize>
-        <topic>${prefix}camera/infra1/image_raw</topic>
-      </sensor>
-    </gazebo>
-    <gazebo reference="${prefix}camera_right_ir_frame">
-      <sensor name="${prefix}cameraired2" type="camera">
-        <camera name="${prefix}camera">
-          <horizontal_fov>1.57</horizontal_fov>
-          <image>
-            <width>1280</width>
-            <height>720</height>
-            <format>L_INT8</format>
-          </image>
-          <clip>
-            <near>0.1</near>
-            <far>100</far>
-          </clip>
-          <noise>
-            <type>gaussian</type>
-            <mean>0.0</mean>
-            <stddev>0.05</stddev>
-          </noise>
-          <camera_info_topic>${prefix}camera/infra2/camera_info</camera_info_topic>
-        </camera>
-        <always_on>1</always_on>
-        <update_rate>30</update_rate>
-        <visualize>0</visualize>
-        <topic>${prefix}camera/infra2/image_raw</topic>
-      </sensor>
-    </gazebo>
-    <gazebo>
-      <plugin
-        filename="libgz-sim-sensors-system.so"
-        name="gz::sim::systems::Sensors">
-        <render_engine>ogre2</render_engine>
-      </plugin>
     </gazebo>
   </xacro:macro>

File: xarm_description/urdf/gripper/xarm_gripper_macro.xacro (robot description, xacro)
@@ -20,17 +20,17 @@
     <xacro:mimic_joint_plugin_gazebo name_prefix="${prefix}left_finger_joint"
       following_joint="${prefix}drive_joint" mimic_joint="${prefix}left_finger_joint"
-      has_pid="${is_ros2}" multiplier="1.0" max_effort="10.0" ros2_control_plugin="${ros2_control_plugin}"/>
+      has_pid="${is_ros2}" multiplier="1.0" max_effort="10.0" />
     <xacro:mimic_joint_plugin_gazebo name_prefix="${prefix}left_inner_knuckle_joint"
       following_joint="${prefix}drive_joint" mimic_joint="${prefix}left_inner_knuckle_joint"
-      has_pid="${is_ros2}" multiplier="1.0" max_effort="10.0" ros2_control_plugin="${ros2_control_plugin}"/>
+      has_pid="${is_ros2}" multiplier="1.0" max_effort="10.0" />
     <xacro:mimic_joint_plugin_gazebo name_prefix="${prefix}right_outer_knuckle_joint"
       following_joint="${prefix}drive_joint" mimic_joint="${prefix}right_outer_knuckle_joint"
-      has_pid="${is_ros2}" multiplier="1.0" max_effort="10.0" ros2_control_plugin="${ros2_control_plugin}"/>
+      has_pid="${is_ros2}" multiplier="1.0" max_effort="10.0" />
     <xacro:mimic_joint_plugin_gazebo name_prefix="${prefix}right_finger_joint"
       following_joint="${prefix}drive_joint" mimic_joint="${prefix}right_finger_joint"
-      has_pid="${is_ros2}" multiplier="1.0" max_effort="10.0" ros2_control_plugin="${ros2_control_plugin}"/>
+      has_pid="${is_ros2}" multiplier="1.0" max_effort="10.0" />
     <xacro:mimic_joint_plugin_gazebo name_prefix="${prefix}right_inner_knuckle_joint"
       following_joint="${prefix}drive_joint" mimic_joint="${prefix}right_inner_knuckle_joint"
-      has_pid="${is_ros2}" multiplier="1.0" max_effort="10.0" ros2_control_plugin="${ros2_control_plugin}"/>
+      has_pid="${is_ros2}" multiplier="1.0" max_effort="10.0" />
   </xacro:macro>
 </robot>

File: xarm_description/urdf/uf850/uf850.ros2_control.xacro (robot description, xacro)
@@ -44,6 +44,10 @@
           <param name="max">3.14</param>
         </command_interface>
-        <state_interface name="position"/>
-        <state_interface name="velocity"/>
+        <state_interface name="position">
+          <param name="initial_value">0.0</param>
+        </state_interface>
+        <state_interface name="velocity">
+          <param name="initial_value">0.0</param>
+        </state_interface>
         <!-- <state_interface name="effort"/> -->
       </joint>
@@ -57,6 +61,10 @@
           <param name="max">3.14</param>
         </command_interface>
-        <state_interface name="position"/>
-        <state_interface name="velocity"/>
+        <state_interface name="position">
+          <param name="initial_value">0.3</param>
+        </state_interface>
+        <state_interface name="velocity">
+          <param name="initial_value">0.0</param>
+        </state_interface>
         <!-- <state_interface name="effort"/> -->
       </joint>
@@ -70,6 +78,10 @@
           <param name="max">3.14</param>
         </command_interface>
-        <state_interface name="position"/>
-        <state_interface name="velocity"/>
+        <state_interface name="position">
+          <param name="initial_value">-0.0</param>
+        </state_interface>
+        <state_interface name="velocity">
+          <param name="initial_value">0.0</param>
+        </state_interface>
         <!-- <state_interface name="effort"/> -->
       </joint>
@@ -83,6 +95,10 @@
           <param name="max">3.14</param>
         </command_interface>
-        <state_interface name="position"/>
-        <state_interface name="velocity"/>
+        <state_interface name="position">
+          <param name="initial_value">-0.0</param>
+        </state_interface>
+        <state_interface name="velocity">
+          <param name="initial_value">0.0</param>
+        </state_interface>
         <!-- <state_interface name="effort"/> -->
       </joint>
@@ -96,6 +112,10 @@
           <param name="max">3.14</param>
         </command_interface>
-        <state_interface name="position"/>
-        <state_interface name="velocity"/>
+        <state_interface name="position">
+          <param name="initial_value">-0.0</param>
+        </state_interface>
+        <state_interface name="velocity">
+          <param name="initial_value">0.0</param>
+        </state_interface>
         <!-- <state_interface name="effort"/> -->
       </joint>
@@ -109,6 +129,10 @@
           <param name="max">3.14</param>
         </command_interface>
-        <state_interface name="position"/>
-        <state_interface name="velocity"/>
+        <state_interface name="position">
+          <param name="initial_value">0.0</param>
+        </state_interface>
+        <state_interface name="velocity">
+          <param name="initial_value">0.0</param>
+        </state_interface>
         <!-- <state_interface name="effort"/> -->
       </joint>

File: xarm_description/urdf/xarm7/xarm7.ros2_control.xacro (robot description, xacro)
@@ -39,6 +39,10 @@
           <param name="max">3.14</param>
         </command_interface>
-        <state_interface name="position"/>
-        <state_interface name="velocity"/>
+        <state_interface name="position">
+          <param name="initial_value">0.0</param>
+        </state_interface>
+        <state_interface name="velocity">
+          <param name="initial_value">0.0</param>
+        </state_interface>
         <!-- <state_interface name="effort"/> -->
       </joint>
@@ -52,6 +56,10 @@
           <param name="max">3.14</param>
         </command_interface>
-        <state_interface name="position"/>
-        <state_interface name="velocity"/>
+        <state_interface name="position">
+          <param name="initial_value">-1.186786</param>
+        </state_interface>
+        <state_interface name="velocity">
+          <param name="initial_value">0.0</param>
+        </state_interface>
         <!-- <state_interface name="effort"/> -->
       </joint>
@@ -65,6 +73,10 @@
           <param name="max">3.14</param>
         </command_interface>
-        <state_interface name="position"/>
-        <state_interface name="velocity"/>
+        <state_interface name="position">
+          <param name="initial_value">0.0</param>
+        </state_interface>
+        <state_interface name="velocity">
+          <param name="initial_value">0.0</param>
+        </state_interface>
         <!-- <state_interface name="effort"/> -->
       </joint>
@@ -78,6 +90,10 @@
           <param name="max">3.14</param>
         </command_interface>
-        <state_interface name="position"/>
-        <state_interface name="velocity"/>
+        <state_interface name="position">
+          <param name="initial_value">0.878955</param>
+        </state_interface>
+        <state_interface name="velocity">
+          <param name="initial_value">0.0</param>
+        </state_interface>
         <!-- <state_interface name="effort"/> -->
       </joint>
@@ -91,6 +107,10 @@
           <param name="max">3.14</param>
         </command_interface>
-        <state_interface name="position"/>
-        <state_interface name="velocity"/>
+        <state_interface name="position">
+          <param name="initial_value">0.0</param>
+        </state_interface>
+        <state_interface name="velocity">
+          <param name="initial_value">0.0</param>
+        </state_interface>
         <!-- <state_interface name="effort"/> -->
       </joint>
@@ -104,6 +124,10 @@
           <param name="max">3.14</param>
         </command_interface>
-        <state_interface name="position"/>
-        <state_interface name="velocity"/>
+        <state_interface name="position">
+          <param name="initial_value">1.449496</param>
+        </state_interface>
+        <state_interface name="velocity">
+          <param name="initial_value">0.0</param>
+        </state_interface>
         <!-- <state_interface name="effort"/> -->
       </joint>
@@ -117,6 +141,10 @@
           <param name="max">3.14</param>
         </command_interface>
-        <state_interface name="position"/>
-        <state_interface name="velocity"/>
+        <state_interface name="position">
+          <param name="initial_value">0.0</param>
+        </state_interface>
+        <state_interface name="velocity">
+          <param name="initial_value">0.0</param>
+        </state_interface>
         <!-- <state_interface name="effort"/> -->
       </joint>
