Commit message: updated xarm_ros2 package to work internally

File: xarm_description/urdf/xarm_device.urdf.xacro (robot description, xacro)
@@ -20,4 +20,5 @@
   <xacro:arg name="add_d435i_links" default="true"/>
   <xacro:arg name="use_gazebo_camera" default="false"/>
+  <xacro:arg name="add_depthai_camera" default="false"/>
   <xacro:arg name="add_other_geometry" default="false"/>
   <xacro:arg name="geometry_type" default="box"/>
@@ -49,4 +50,5 @@
     add_realsense_d435i="$(arg add_realsense_d435i)"
     add_d435i_links="$(arg add_d435i_links)"
+    add_depthai_camera="$(arg add_depthai_camera)"
     add_other_geometry="$(arg add_other_geometry)"
     geometry_type="$(arg geometry_type)" geometry_mass="$(arg geometry_mass)"

File: xarm_description/urdf/xarm_device_macro.xacro (robot description, xacro)
@@ -21,4 +21,5 @@
     add_realsense_d435i:=false
     add_d435i_links:=true
+    add_depthai_camera:=false
     use_gazebo_camera:=false
     add_other_geometry:=false
@@ -52,9 +53,9 @@
     <!-- Specify Mesh file path -->
     <xacro:property name="mesh_suffix" value="${mesh_suffix}" scope="parent"/>
-    <xacro:if value="${ros2_control_plugin == 'gazebo_ros2_control/GazeboSystem' or ros2_control_plugin == 'ign_ros2_control/IgnitionSystem' or ros2_control_plugin == 'gz_ros2_control/GazeboSimSystem'}">
+    <xacro:if value="${ros2_control_plugin == 'gazebo_ros2_control/GazeboSystem' or ros2_control_plugin == 'ign_ros2_control/IgnitionSystem'}">
       <!-- gazebo use -->
       <xacro:property name="mesh_path" value="file://$(find xarm_description)/meshes" scope="parent"/>
     </xacro:if>
-    <xacro:unless value="${ros2_control_plugin == 'gazebo_ros2_control/GazeboSystem' or ros2_control_plugin == 'ign_ros2_control/IgnitionSystem' or ros2_control_plugin == 'gz_ros2_control/GazeboSimSystem'}">
+    <xacro:unless value="${ros2_control_plugin == 'gazebo_ros2_control/GazeboSystem' or ros2_control_plugin == 'ign_ros2_control/IgnitionSystem'}">
       <xacro:property name="mesh_path" value="package://xarm_description/meshes" scope="parent"/>
     </xacro:unless>
@@ -207,17 +208,18 @@
       <xacro:if value="${add_d435i_links}">
         <xacro:include filename="$(find xarm_description)/urdf/camera/realsense.gazebo.xacro" />
-        <xacro:if value="${ros2_control_plugin == 'gz_ros2_control/GazeboSimSystem'}">
-          <xacro:realsense_gz prefix="${prefix}" />
-        </xacro:if>
-        <xacro:if value="${ros2_control_plugin == 'ign_ros2_control/IgnitionSystem'}">
-          <xacro:realsense_ignition prefix="${prefix}" />
-        </xacro:if>
-        <xacro:if value="${ros2_control_plugin == 'gazebo_ros2_control/GazeboSystem'}">
-          <xacro:realsense_gazebo prefix="${prefix}" />
-        </xacro:if>
+        <xacro:realsense_gazebo prefix="${prefix}" />
       </xacro:if>
     </xacro:if>
     <xacro:unless value="${add_realsense_d435i}">
-      <link name="${prefix}link_eef"/>
+      <!-- Add depthai camera  -->
+      <!-- TODO: check how to start depthai camera simulation. -->
+      <!-- probably use use_gazebo_camera or add an arg to start simulation -->
+      <xacro:if value="${add_depthai_camera}">
+        <xacro:include filename="$(find abluo_description)/description/camera.urdf.xacro" />
+        <xacro:depthai_camera prefix="${prefix}"  />
+      </xacro:if>
+      <xacro:unless value="${add_depthai_camera}">
+        <link name="${prefix}link_eef"/>
+      </xacro:unless>
     </xacro:unless>
     <joint name="${prefix}joint_eef" type="fixed">
@@ -284,13 +286,10 @@
           <xacro:property name="new_ros2_control_params" value="${ros2_control_params}"/>
         </xacro:if>
-        <xacro:if value="${ros2_control_plugin == 'gz_ros2_control/GazeboSimSystem'}">
-          <xacro:gz_ros2_control_plugin ros2_control_params="${new_ros2_control_params}"/>
-        </xacro:if>
         <xacro:if value="${ros2_control_plugin == 'ign_ros2_control/IgnitionSystem'}">
           <xacro:ignition_ros2_control_plugin prefix="${prefix}" ros2_control_params="${new_ros2_control_params}"/>
         </xacro:if>
-        <xacro:if value="${ros2_control_plugin == 'gazebo_ros2_control/GazeboSystem'}">
+        <xacro:unless value="${ros2_control_plugin == 'ign_ros2_control/IgnitionSystem'}">
           <xacro:gazebo_ros2_control_plugin ros2_control_params="${new_ros2_control_params}"/>
-        </xacro:if>
+        </xacro:unless>
       </xacro:if>
       <xacro:unless value="${is_ros2}">
